Commit message: Clean up and get Jacobian working.

File: assets/urdf/mm.urdf (robot description, URDF)
Before this commit: robot Thing, 30 links, 29 joints
Links:
- link thing_tool: geometry visual sphere radius=0.03
- link ur10_arm_tool0: geometry collision cylinder length=0.290 radius=0.01; visual cylinder length=0.290 radius=0.01
Joints:
- joint front_left_wheel: type continuous -> fixed
- joint front_right_wheel: type continuous -> fixed
- joint front_rocker: type revolute -> fixed
- joint rear_left_wheel: type continuous -> fixed
- joint rear_right_wheel: type continuous -> fixed
- joint tool0_tcp_fixed_joint: origin xyz=0.0 0.0 0.29 rpy=1.5707963 0.0 0.26179939 -> xyz=0.0 0.0 0.290 rpy=0.0 0.0 0.0

Commit message: Add "tray balancing" EE.

File: assets/urdf/mm.urdf (robot description, URDF)
Before this commit: robot Thing, 30 links, 29 joints
Links:
- link thing_tool: mass None -> 0.1; geometry collision sphere radius=0.03; collision sphere radius=0.03
