Commit message: Implement dynamic obstacle avoidance with multiple body points.

File: tray_balance_ocs2/urdf/mm_pyb.urdf (robot description, URDF)
Before this commit: robot Thing, 32 links, 31 joints
Links:
- removed link balanced_object_collision_link
- removed link base_collision_link
- removed link elbow_collision_link
- removed link forearm_collision_link
- removed link wrist_collision_link
Joints:
- removed joint balanced_object_collision_joint
- removed joint base_collision_joint
- removed joint elbow_collision_joint
- removed joint forearm_collision_joint
- removed joint wrist_collision_joint
