Commit message: Re-enable basic collision checking.

File: tray_balance_ocs2/urdf/mm.urdf (robot description, URDF)
Before this commit: robot Thing, 30 links, 29 joints
Links:
- link chassis_link: geometry collision box size=1.0 0.8 0.3; visual box size=1.0 0.8 0.3

Commit message: Simulation with multiple objects

File: tray_balance_ocs2/urdf/mm.urdf (robot description, URDF)
Before this commit: robot Thing, 30 links, 29 joints
Links:
- link chassis_link: geometry collision box size=1.0 0.8 0.3; visual mesh filename=file:///home/adam/phd/code/mm/ocs2_noetic/catkin_ws/src/ocs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

File: tray_balance_ocs2/urdf/obstacles.urdf (robot description, URDF)
Before this commit: robot Obstacles, 1 links, 0 joints
Links:
- added link obstacle2_link; collision cylinder length=0.5 radius=0.5; visual cylinder length=0.5 radius=0.5
- added link obstacle3_link; collision cylinder length=0.5 radius=0.5; visual cylinder length=0.5 radius=0.5
- added link obstacle_base_link
- link obstacle1_link: geometry collision cylinder length=0.5 radius=0.5; visual cylinder length=0.5 radius=0.5
Joints:
- added joint obstacle1_link_joint: type fixed, parent obstacle_base_link, child obstacle1_link, origin xyz=0 0 0 rpy=0 0 0
- added joint obstacle2_link_joint: type fixed, parent obstacle_base_link, child obstacle2_link, origin xyz=0 0 0 rpy=0 0 0
- added joint obstacle3_link_joint: type fixed, parent obstacle_base_link, child obstacle3_link, origin xyz=0 0 0 rpy=0 0 0

Commit message: Fix EE orientation.
Now has zero rotation wrt world frame at starting location. This makes
some assumptions with the inertia matrix calculations valid.

File: tray_balance_ocs2/urdf/mm.urdf (robot description, URDF)
Before this commit: robot Thing, 30 links, 29 joints
Joints:
- joint tool0_tcp_fixed_joint: origin xyz=0.0 0.0 0.290 rpy=0.0 0.0 0.0 -> xyz=0.0 0.0 0.290 rpy=0.0 0.0 3.14159

Commit message: Fix/clean up the pybullet-only URDF.

File: tray_balance_ocs2/urdf/mm.urdf (robot description, URDF)
Before this commit: robot Thing, 30 links, 29 joints
Joints:
- joint base_link_joint: origin xyz=0 0 0 rpy=0 0 0 -> xyz=0 0 0.01 rpy=0 0 0

File: tray_balance_ocs2/urdf/mm_pyb.urdf (robot description, URDF)
Before this commit: robot Thing, 33 links, 32 joints
Links:
- removed link front_left_wheel_link
- removed link front_right_wheel_link
- removed link front_rocker_link
- removed link rear_left_wheel_link
- removed link rear_right_wheel_link
- removed link rear_rocker_link
Joints:
- removed joint front_left_wheel
- removed joint front_right_wheel
- removed joint front_rocker
- removed joint rear_left_wheel
- removed joint rear_right_wheel
- removed joint rear_rocker
- joint base_to_y_joint: origin xyz=0 0 0.1 rpy=0 0 0 -> xyz=0 0 0.01 rpy=0 0 0

Commit message: Debugging ZMP mismatch between Python and C++

File: tray_balance_ocs2/urdf/mm.urdf (robot description, URDF)
Before this commit: robot Thing, 30 links, 29 joints
Links:
- added link balanced_object_collision_link; collision cylinder length=0.1 radius=0.25; visual cylinder length=0.1 radius=0.25
- added link elbow_collision_link; collision sphere radius=0.15; visual sphere radius=0.15
- added link forearm_collision_link; collision cylinder length=0.6 radius=0.06; visual cylinder length=0.6 radius=0.06
- added link shoulder_collision_link; collision sphere radius=0.15; visual sphere radius=0.15
- added link upper_arm_collision_link; collision cylinder length=0.65 radius=0.06; visual cylinder length=0.65 radius=0.06
- added link wrist_collision_link; collision sphere radius=0.15; visual sphere radius=0.15
- link thing_tool: geometry collision sphere radius=0.02; collision sphere radius=0.02
Joints:
- added joint balanced_object_collision_joint: type fixed, parent thing_tool, child balanced_object_collision_link, origin xyz=0 0 0 rpy=0 0 0
- added joint elbow_collision_joint: type fixed, parent ur10_arm_forearm_link, child elbow_collision_link, origin xyz=0 0 0 rpy=0 0 0
- added joint forearm_collision_joint: type fixed, parent ur10_arm_forearm_link, child forearm_collision_link, origin xyz=0 0 0 rpy=0 0 0
- added joint shoulder_collision_joint: type fixed, parent ur10_arm_upper_arm_link, child shoulder_collision_link, origin xyz=0 0 0 rpy=0 0 0
- added joint upper_arm_collision_joint: type fixed, parent ur10_arm_upper_arm_link, child upper_arm_collision_link, origin xyz=0 0 0 rpy=0 0 0
- added joint wrist_collision_joint: type fixed, parent ur10_arm_wrist_3_link, child wrist_collision_link, origin xyz=0 0 0 rpy=0 0 0

File: tray_balance_ocs2/urdf/mm_pyb.urdf (robot description, URDF)
Before this commit: robot Thing, 27 links, 26 joints
Links:
- link thing_tool: geometry collision sphere radius=0.02; collision sphere radius=0.02

Commit message: Configure static obstacle "cafe" environment.

File: tray_balance_ocs2/urdf/mm.urdf (robot description, URDF)
Before this commit: robot Thing, 36 links, 35 joints
Links:
- added link base_collision_link; collision box size=1.0 0.8 0.3; visual box size=1.0 0.8 0.3
- link balanced_object_collision_link: geometry collision cylinder length=0.2 radius=0.25; visual cylinder length=0.2 radius=0.25
Joints:
- added joint base_collision_joint: type fixed, parent base_link, child base_collision_link, origin xyz=0 0 0.01 rpy=0 0 0

File: tray_balance_ocs2/urdf/mm_pyb.urdf (robot description, URDF)
Before this commit: robot Thing, 27 links, 26 joints
Links:
- added link balanced_object_collision_link; visual cylinder length=0.2 radius=0.25
- added link base_collision_link; visual box size=1.0 0.8 0.3
- added link elbow_collision_link; visual sphere radius=0.15
- added link forearm_collision_link; visual cylinder length=0.6 radius=0.06
- added link wrist_collision_link; visual sphere radius=0.15
Joints:
- added joint balanced_object_collision_joint: type fixed, parent thing_tool, child balanced_object_collision_link, origin xyz=0 0 0 rpy=0 0 0
- added joint base_collision_joint: type fixed, parent base_link, child base_collision_link, origin xyz=0 0 0.01 rpy=0 0 0
- added joint elbow_collision_joint: type fixed, parent ur10_arm_forearm_link, child elbow_collision_link, origin xyz=0 0 0 rpy=0 0 0
- added joint forearm_collision_joint: type fixed, parent ur10_arm_forearm_link, child forearm_collision_link, origin xyz=0 0 0 rpy=0 0 0
- added joint wrist_collision_joint: type fixed, parent ur10_arm_wrist_3_link, child wrist_collision_link, origin xyz=0 0 0 rpy=0 0 0

File: tray_balance_ocs2/urdf/obstacles.urdf (robot description, URDF)
Before this commit: robot Obstacles, 4 links, 3 joints
Links:
- removed link obstacle1_link
- removed link obstacle2_link
- removed link obstacle3_link
- added link chair1_1_link; collision cylinder length=0.45 radius=0.2; visual cylinder length=0.45 radius=0.2
- added link chair1_2_link; collision cylinder length=0.45 radius=0.2; visual cylinder length=0.45 radius=0.2
- added link chair2_1_link; collision cylinder length=1.35 radius=0.2; visual cylinder length=1.35 radius=0.2
- added link chair3_1_link; collision cylinder length=1.35 radius=0.2; visual cylinder length=1.35 radius=0.2
- added link chair3_2_link; collision cylinder length=0.45 radius=0.2; visual cylinder length=0.45 radius=0.2
- added link chair4_1_link; collision cylinder length=0.45 radius=0.2; visual cylinder length=0.45 radius=0.2
- added link chair4_2_link; collision cylinder length=1.35 radius=0.2; visual cylinder length=1.35 radius=0.2
- added link table1_link; collision cylinder length=0.75 radius=0.5; visual cylinder length=0.75 radius=0.5
- added link table2_link; collision cylinder length=0.75 radius=0.5; visual cylinder length=0.75 radius=0.5
- added link table3_link; collision cylinder length=0.75 radius=0.5; visual cylinder length=0.75 radius=0.5
- added link table4_link; collision cylinder length=0.75 radius=0.5; visual cylinder length=0.75 radius=0.5
- added link table5_link; collision cylinder length=0.75 radius=0.5; visual cylinder length=0.75 radius=0.5
Joints:
- removed joint obstacle1_link_joint
- removed joint obstacle2_link_joint
- removed joint obstacle3_link_joint
- added joint chair1_1_link_joint: type fixed, parent obstacle_base_link, child chair1_1_link, origin xyz=0 0 0 rpy=0 0 0
- added joint chair1_2_link_joint: type fixed, parent obstacle_base_link, child chair1_2_link, origin xyz=0 0 0 rpy=0 0 0
- added joint chair2_1_link_joint: type fixed, parent obstacle_base_link, child chair2_1_link, origin xyz=0 0 0 rpy=0 0 0
- added joint chair3_1_link_joint: type fixed, parent obstacle_base_link, child chair3_1_link, origin xyz=0 0 0 rpy=0 0 0
- added joint chair3_2_link_joint: type fixed, parent obstacle_base_link, child chair3_2_link, origin xyz=0 0 0 rpy=0 0 0
- added joint chair4_1_link_joint: type fixed, parent obstacle_base_link, child chair4_1_link, origin xyz=0 0 0 rpy=0 0 0
- added joint chair4_2_link_joint: type fixed, parent obstacle_base_link, child chair4_2_link, origin xyz=0 0 0 rpy=0 0 0
- added joint table1_link_joint: type fixed, parent obstacle_base_link, child table1_link, origin xyz=0 0 0 rpy=0 0 0
- added joint table2_link_joint: type fixed, parent obstacle_base_link, child table2_link, origin xyz=0 0 0 rpy=0 0 0
- added joint table3_link_joint: type fixed, parent obstacle_base_link, child table3_link, origin xyz=0 0 0 rpy=0 0 0
- added joint table4_link_joint: type fixed, parent obstacle_base_link, child table4_link, origin xyz=0 0 0 rpy=0 0 0
- added joint table5_link_joint: type fixed, parent obstacle_base_link, child table5_link, origin xyz=0 0 0 rpy=0 0 0

Commit message: Update obstacle colours.

File: tray_balance_ocs2/urdf/mm.urdf (robot description, URDF)
Before this commit: robot Thing, 37 links, 36 joints
Links:
- link balanced_object_collision_link: geometry collision cylinder length=0.25 radius=0.25; visual cylinder length=0.25 radius=0.25

File: tray_balance_ocs2/urdf/mm_pyb.urdf (robot description, URDF)
Before this commit: robot Thing, 32 links, 31 joints
Links:
- link balanced_object_collision_link: geometry visual cylinder length=0.25 radius=0.25

Commit message: Configuration for collecting dynamic obstacle data.

File: tray_balance_ocs2/urdf/mm.urdf (robot description, URDF)
Before this commit: robot Thing, 37 links, 36 joints
Links:
- added link forearm_collision_sphere_link; collision sphere radius=0.15; visual sphere radius=0.15
Joints:
- added joint forearm_collision_sphere_joint: type fixed, parent ur10_arm_forearm_link, child forearm_collision_sphere_link, origin xyz=0 0 0.34 rpy=0 0 0
- joint forearm_collision_joint: origin xyz=0 0 0 rpy=0 0 0 -> xyz=0 0 0.3 rpy=0 0 0

File: tray_balance_ocs2/urdf/mm_pyb.urdf (robot description, URDF)
Before this commit: robot Thing, 27 links, 26 joints
Links:
- added link balanced_object_collision_link; visual cylinder length=0.25 radius=0.25
- added link balanced_object_collision_sphere_link; visual sphere radius=0.25
- added link base_collision_link; visual box size=1.0 0.8 0.3
- added link elbow_collision_link; visual sphere radius=0.15
- added link forearm_collision_link; visual cylinder length=0.6 radius=0.06
- added link forearm_collision_sphere_link; visual sphere radius=0.15
- added link wrist_collision_link; visual sphere radius=0.15
Joints:
- added joint balanced_object_collision_joint: type fixed, parent thing_tool, child balanced_object_collision_link, origin xyz=0 0 0 rpy=0 0 0
- added joint balanced_object_collision_sphere_joint: type fixed, parent thing_tool, child balanced_object_collision_sphere_link, origin xyz=0 0 0 rpy=0 0 0
- added joint base_collision_joint: type fixed, parent base_link, child base_collision_link, origin xyz=0 0 0.01 rpy=0 0 0
- added joint elbow_collision_joint: type fixed, parent ur10_arm_forearm_link, child elbow_collision_link, origin xyz=0 0 0 rpy=0 0 0
- added joint forearm_collision_joint: type fixed, parent ur10_arm_forearm_link, child forearm_collision_link, origin xyz=0 0 0.3 rpy=0 0 0
- added joint forearm_collision_sphere_joint: type fixed, parent ur10_arm_forearm_link, child forearm_collision_sphere_link, origin xyz=0 0 0.34 rpy=0 0 0
- added joint wrist_collision_joint: type fixed, parent ur10_arm_wrist_3_link, child wrist_collision_link, origin xyz=0 0 0 rpy=0 0 0

Commit message: Recollecting computation time data

File: tray_balance_ocs2/urdf/mm.urdf (robot description, URDF)
Before this commit: robot Thing, 38 links, 37 joints
Links:
- removed link forearm_collision_sphere_link
- link balanced_object_collision_link: geometry collision cylinder length=0.1 radius=0.25; visual cylinder length=0.1 radius=0.25
Joints:
- removed joint forearm_collision_sphere_joint
- joint forearm_collision_joint: origin xyz=0 0 0.3 rpy=0 0 0 -> xyz=0 0 0 rpy=0 0 0

File: tray_balance_ocs2/urdf/mm_pyb.urdf (robot description, URDF)
Before this commit: robot Thing, 34 links, 33 joints
Links:
- removed link balanced_object_collision_sphere_link
- removed link base_collision_link
- removed link forearm_collision_sphere_link
- link balanced_object_collision_link: geometry visual cylinder length=0.1 radius=0.25
Joints:
- removed joint balanced_object_collision_sphere_joint
- removed joint base_collision_joint
- removed joint forearm_collision_sphere_joint
- joint forearm_collision_joint: origin xyz=0 0 0.3 rpy=0 0 0 -> xyz=0 0 0 rpy=0 0 0

Commit message: ICRA-22 submission

File: tray_balance_ocs2/urdf/mm.urdf (robot description, URDF)
Before this commit: robot Thing, 37 links, 36 joints
Links:
- link balanced_object_collision_link: geometry collision cylinder length=0.25 radius=0.25; visual cylinder length=0.25 radius=0.25

File: tray_balance_ocs2/urdf/mm_pyb.urdf (robot description, URDF)
Before this commit: robot Thing, 31 links, 30 joints
Links:
- removed link balanced_object_collision_link
- removed link elbow_collision_link
- removed link forearm_collision_link
- removed link wrist_collision_link
Joints:
- removed joint balanced_object_collision_joint
- removed joint elbow_collision_joint
- removed joint forearm_collision_joint
- removed joint wrist_collision_joint

Commit message: Video recordings.

File: tray_balance_ocs2/urdf/mm.urdf (robot description, URDF)
Before this commit: robot Thing, 37 links, 36 joints
Links:
- added link forearm_collision_sphere_link1; collision sphere radius=0.15; visual sphere radius=0.15
- added link forearm_collision_sphere_link2; collision sphere radius=0.15; visual sphere radius=0.15
- link balanced_object_collision_link: geometry collision cylinder length=0.1 radius=0.25; visual cylinder length=0.1 radius=0.25
Joints:
- added joint forearm_collision_sphere_joint1: type fixed, parent ur10_arm_forearm_link, child forearm_collision_sphere_link1, origin xyz=0 0 0.2 rpy=0 0 0
- added joint forearm_collision_sphere_joint2: type fixed, parent ur10_arm_forearm_link, child forearm_collision_sphere_link2, origin xyz=0 0 0.4 rpy=0 0 0

Commit message: Change name to tray_balance_ocs2

File: tray_balance_ocs2/urdf/mm.urdf (robot description, URDF)
Before this commit: robot Thing, 39 links, 38 joints
Links:
- link arch_link: geometry visual mesh filename=file:///home/adam/phd/code/mm/ocs2_noetic/catkin_ws/src/tra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
- link axle_link: geometry visual mesh filename=file:///home/adam/phd/code/mm/ocs2_noetic/catkin_ws/src/tra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
- link chassis_link: geometry collision box size=1.0 0.8 0.3; visual mesh filename=file:///home/adam/phd/code/mm/ocs2_noetic/catkin_ws/src/tra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
- link front_cover_link: geometry visual mesh filename=file:///home/adam/phd/code/mm/ocs2_noetic/catkin_ws/src/tra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
- link front_left_wheel_link: geometry collision cylinder length=0.079 radius=0.0759; visual mesh filename=file:///home/adam/phd/code/mm/ocs2_noetic/catkin_ws/src/tra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
- link front_lights_link: geometry visual mesh filename=file:///home/adam/phd/code/mm/ocs2_noetic/catkin_ws/src/tra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
- link front_right_wheel_link: geometry collision cylinder length=0.079 radius=0.0759; visual mesh filename=file:///home/adam/phd/code/mm/ocs2_noetic/catkin_ws/src/tra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
- link front_rocker_link: geometry visual mesh filename=file:///home/adam/phd/code/mm/ocs2_noetic/catkin_ws/src/tra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
- link left_side_cover_link: geometry visual mesh filename=file:///home/adam/phd/code/mm/ocs2_noetic/catkin_ws/src/tra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
- link rear_cover_link: geometry visual mesh filename=file:///home/adam/phd/code/mm/ocs2_noetic/catkin_ws/src/tra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
- link rear_left_wheel_link: geometry collision cylinder length=0.079 radius=0.0759; visual mesh filename=file:///home/adam/phd/code/mm/ocs2_noetic/catkin_ws/src/tra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
- link rear_lights_link: geometry visual mesh filename=file:///home/adam/phd/code/mm/ocs2_noetic/catkin_ws/src/tra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
- link rear_right_wheel_link: geometry collision cylinder length=0.079 radius=0.0759; visual mesh filename=file:///home/adam/phd/code/mm/ocs2_noetic/catkin_ws/src/tra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
- link rear_rocker_link: geometry visual mesh filename=file:///home/adam/phd/code/mm/ocs2_noetic/catkin_ws/src/tra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
- link right_side_cover_link: geometry visual mesh filename=file:///home/adam/phd/code/mm/ocs2_noetic/catkin_ws/src/tra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
- link top_link: geometry collision mesh filename=file:///home/adam/phd/code/mm/ocs2_noetic/catkin_ws/src/tra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; visual mesh filename=file:///home/adam/phd/code/mm/ocs2_noetic/catkin_ws/src/tra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
- link ur10_arm_base_link: geometry collision mesh filename=file:///home/adam/phd/code/mm/ocs2_noetic/catkin_ws/src/tra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; visual mesh filename=file:///home/adam/phd/code/mm/ocs2_noetic/catkin_ws/src/tra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
- link ur10_arm_forearm_link: geometry collision mesh filename=file:///home/adam/phd/code/mm/ocs2_noetic/catkin_ws/src/tra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; visual mesh filename=file:///home/adam/phd/code/mm/ocs2_noetic/catkin_ws/src/tra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
- link ur10_arm_shoulder_link: geometry collision mesh filename=file:///home/adam/phd/code/mm/ocs2_noetic/catkin_ws/src/tra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; visual mesh filename=file:///home/adam/phd/code/mm/ocs2_noetic/catkin_ws/src/tra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
- link ur10_arm_upper_arm_link: geometry collision mesh filename=file:///home/adam/phd/code/mm/ocs2_noetic/catkin_ws/src/tra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; visual mesh filename=file:///home/adam/phd/code/mm/ocs2_noetic/catkin_ws/src/tra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
- link ur10_arm_wrist_1_link: geometry collision mesh filename=file:///home/adam/phd/code/mm/ocs2_noetic/catkin_ws/src/tra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; visual mesh filename=file:///home/adam/phd/code/mm/ocs2_noetic/catkin_ws/src/tra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
- link ur10_arm_wrist_2_link: geometry collision mesh filename=file:///home/adam/phd/code/mm/ocs2_noetic/catkin_ws/src/tra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; visual mesh filename=file:///home/adam/phd/code/mm/ocs2_noetic/catkin_ws/src/tra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
- link ur10_arm_wrist_3_link: geometry collision mesh filename=file:///home/adam/phd/code/mm/ocs2_noetic/catkin_ws/src/tra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; visual mesh filename=file:///home/adam/phd/code/mm/ocs2_noetic/catkin_ws/src/tra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

File: tray_balance_ocs2/urdf/mm_pyb.urdf (robot description, URDF)
Before this commit: robot Thing, 27 links, 26 joints
Links:
- link arch_link: geometry visual mesh filename=file:///home/adam/phd/code/mm/ocs2_noetic/catkin_ws/src/tra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
- link axle_link: geometry visual mesh filename=file:///home/adam/phd/code/mm/ocs2_noetic/catkin_ws/src/tra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
- link chassis_link: geometry collision box size=1.0 0.8 0.3; visual mesh filename=file:///home/adam/phd/code/mm/ocs2_noetic/catkin_ws/src/tra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
- link front_cover_link: geometry visual mesh filename=file:///home/adam/phd/code/mm/ocs2_noetic/catkin_ws/src/tra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
- link front_lights_link: geometry visual mesh filename=file:///home/adam/phd/code/mm/ocs2_noetic/catkin_ws/src/tra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
- link left_side_cover_link: geometry visual mesh filename=file:///home/adam/phd/code/mm/ocs2_noetic/catkin_ws/src/tra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
- link rear_cover_link: geometry visual mesh filename=file:///home/adam/phd/code/mm/ocs2_noetic/catkin_ws/src/tra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
- link rear_lights_link: geometry visual mesh filename=file:///home/adam/phd/code/mm/ocs2_noetic/catkin_ws/src/tra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
- link right_side_cover_link: geometry visual mesh filename=file:///home/adam/phd/code/mm/ocs2_noetic/catkin_ws/src/tra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
- link top_link: geometry collision mesh filename=file:///home/adam/phd/code/mm/ocs2_noetic/catkin_ws/src/tra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; visual mesh filename=file:///home/adam/phd/code/mm/ocs2_noetic/catkin_ws/src/tra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
- link ur10_arm_base_link: geometry collision mesh filename=file:///home/adam/phd/code/mm/ocs2_noetic/catkin_ws/src/tra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; visual mesh filename=file:///home/adam/phd/code/mm/ocs2_noetic/catkin_ws/src/tra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
- link ur10_arm_forearm_link: geometry collision mesh filename=file:///home/adam/phd/code/mm/ocs2_noetic/catkin_ws/src/tra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; visual mesh filename=file:///home/adam/phd/code/mm/ocs2_noetic/catkin_ws/src/tra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
- link ur10_arm_shoulder_link: geometry collision mesh filename=file:///home/adam/phd/code/mm/ocs2_noetic/catkin_ws/src/tra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; visual mesh filename=file:///home/adam/phd/code/mm/ocs2_noetic/catkin_ws/src/tra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
- link ur10_arm_upper_arm_link: geometry collision mesh filename=file:///home/adam/phd/code/mm/ocs2_noetic/catkin_ws/src/tra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; visual mesh filename=file:///home/adam/phd/code/mm/ocs2_noetic/catkin_ws/src/tra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
- link ur10_arm_wrist_1_link: geometry collision mesh filename=file:///home/adam/phd/code/mm/ocs2_noetic/catkin_ws/src/tra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; visual mesh filename=file:///home/adam/phd/code/mm/ocs2_noetic/catkin_ws/src/tra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
- link ur10_arm_wrist_2_link: geometry collision mesh filename=file:///home/adam/phd/code/mm/ocs2_noetic/catkin_ws/src/tra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; visual mesh filename=file:///home/adam/phd/code/mm/ocs2_noetic/catkin_ws/src/tra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
- link ur10_arm_wrist_3_link: geometry collision mesh filename=file:///home/adam/phd/code/mm/ocs2_noetic/catkin_ws/src/tra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; visual mesh filename=file:///home/adam/phd/code/mm/ocs2_noetic/catkin_ws/src/tra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
