Commit message: Rename mm_pybullet_sim -> tray_balance_sim

File: tray_balance_sim/assets/urdf/mm.urdf (robot description, URDF)
Before this commit: robot Thing, 30 links, 29 joints
Links:
- removed link front_left_wheel_link
- removed link front_right_wheel_link
- removed link front_rocker_link
- removed link rear_left_wheel_link
- removed link rear_right_wheel_link
- removed link rear_rocker_link
- added link world_link, mass 0
- added link x_prismatic_link, mass 0.01
- added link y_prismatic_link, mass 0.01
- link arch_link: geometry visual mesh filename=file:///home/adam/phd/code/mm/ocs2_noetic/catkin_ws/src/tra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
- link axle_link: geometry visual mesh filename=file:///home/adam/phd/code/mm/ocs2_noetic/catkin_ws/src/tra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
- link base_link: mass None -> 0.01
- link chassis_link: geometry collision box size=1.0 0.8 0.3; visual mesh filename=file:///home/adam/phd/code/mm/ocs2_noetic/catkin_ws/src/tra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
- link front_cover_link: geometry visual mesh filename=file:///home/adam/phd/code/mm/ocs2_noetic/catkin_ws/src/tra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
- link front_lights_link: geometry visual mesh filename=file:///home/adam/phd/code/mm/ocs2_noetic/catkin_ws/src/tra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
- link left_side_cover_link: geometry visual mesh filename=file:///home/adam/phd/code/mm/ocs2_noetic/catkin_ws/src/tra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
- link rear_cover_link: geometry visual mesh filename=file:///home/adam/phd/code/mm/ocs2_noetic/catkin_ws/src/tra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
- link rear_lights_link: geometry visual mesh filename=file:///home/adam/phd/code/mm/ocs2_noetic/catkin_ws/src/tra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
- link right_side_cover_link: geometry visual mesh filename=file:///home/adam/phd/code/mm/ocs2_noetic/catkin_ws/src/tra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
- link thing_tool: geometry collision sphere radius=0.02; collision sphere radius=0.02
- link top_link: geometry collision mesh filename=file:///home/adam/phd/code/mm/ocs2_noetic/catkin_ws/src/tra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; visual mesh filename=file:///home/adam/phd/code/mm/ocs2_noetic/catkin_ws/src/tra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
- link ur10_arm_base_link: geometry collision mesh filename=file:///home/adam/phd/code/mm/ocs2_noetic/catkin_ws/src/tra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; visual mesh filename=file:///home/adam/phd/code/mm/ocs2_noetic/catkin_ws/src/tra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
- link ur10_arm_forearm_link: geometry collision mesh filename=file:///home/adam/phd/code/mm/ocs2_noetic/catkin_ws/src/tra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; visual mesh filename=file:///home/adam/phd/code/mm/ocs2_noetic/catkin_ws/src/tra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
- link ur10_arm_shoulder_link: geometry collision mesh filename=file:///home/adam/phd/code/mm/ocs2_noetic/catkin_ws/src/tra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; visual mesh filename=file:///home/adam/phd/code/mm/ocs2_noetic/catkin_ws/src/tra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
- link ur10_arm_upper_arm_link: geometry collision mesh filename=file:///home/adam/phd/code/mm/ocs2_noetic/catkin_ws/src/tra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; visual mesh filename=file:///home/adam/phd/code/mm/ocs2_noetic/catkin_ws/src/tra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
- link ur10_arm_wrist_1_link: geometry collision mesh filename=file:///home/adam/phd/code/mm/ocs2_noetic/catkin_ws/src/tra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; visual mesh filename=file:///home/adam/phd/code/mm/ocs2_noetic/catkin_ws/src/tra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
- link ur10_arm_wrist_2_link: geometry collision mesh filename=file:///home/adam/phd/code/mm/ocs2_noetic/catkin_ws/src/tra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; visual mesh filename=file:///home/adam/phd/code/mm/ocs2_noetic/catkin_ws/src/tra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
- link ur10_arm_wrist_3_link: geometry collision mesh filename=file:///home/adam/phd/code/mm/ocs2_noetic/catkin_ws/src/tra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; visual mesh filename=file:///home/adam/phd/code/mm/ocs2_noetic/catkin_ws/src/tra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
Joints:
- removed joint front_left_wheel
- removed joint front_right_wheel
- removed joint front_rocker
- removed joint rear_left_wheel
- removed joint rear_right_wheel
- removed joint rear_rocker
- added joint base_to_y_joint: type continuous, parent y_prismatic_link, child base_link, origin xyz=0 0 0.01 rpy=0 0 0, axis 0 0 1
- added joint x_to_world_joint: type prismatic, parent world_link, child x_prismatic_link, origin xyz=0 0 0 rpy=0 0 0, axis 1 0 0, limit effort=0.0 velocity=1000.0
- added joint y_to_x_joint: type prismatic, parent x_prismatic_link, child y_prismatic_link, origin xyz=0 0 0 rpy=0 0 0, axis 0 1 0, limit effort=0.0 velocity=1000.0
- joint tool0_tcp_fixed_joint: origin xyz=0.0 0.0 0.290 rpy=0.0 0.0 0.0 -> xyz=0.0 0.0 0.290 rpy=0.0 0.0 3.14159
