Commit message: Make tor11 mesh light gray

File: tray_balance_assets/urdf/mm_pyb.urdf.xacro (robot description, xacro)
@@ -247,4 +247,7 @@
         <mesh filename="file://$(find tray_balance_assets)/meshes/tor11_mech.dae"/>
       </geometry>
+      <material name="LightGrey">
+        <color rgba="0.7 0.7 0.7 1.0"/>
+      </material>
     </visual>
     <!-- <collision> -->
