Commit message: Add visualization of spheres; fix max_radius implementation.

File: tray_balance_assets/urdf/mm_pyb.urdf (robot description, URDF)
Before this commit: robot Thing, 27 links, 26 joints
Links:
- added link robust_sphere1_link; visual sphere radius=0.12
- added link robust_sphere2_link; visual sphere radius=0.12
Joints:
- added joint robust_sphere1_joint: type fixed, parent thing_tool, child robust_sphere1_link, origin xyz=0 0 0 rpy=0 0 0
- added joint robust_sphere2_joint: type fixed, parent thing_tool, child robust_sphere2_link, origin xyz=0 0 0 rpy=0 0 0

File: tray_balance_assets/urdf/mm_pyb.urdf.xacro (robot description, xacro)
@@ -20,5 +20,5 @@
   </material>
   <material name="seethrough">
-    <color rgba="0.0 1.0 0.0 0.25"/>
+    <color rgba="0.0 0.0 0.0 0.25"/>
   </material>
   <link name="world_link">
@@ -568,4 +568,32 @@
     </inertial>
   </link>
+  <link name="robust_sphere1_link">
+    <visual>
+      <origin rpy="0 0 0" xyz="0 0 0.1"/>
+      <geometry>
+        <sphere radius="0.12"/>
+      </geometry>
+      <material name="seethrough"/>
+    </visual>
+  </link>
+  <joint name="robust_sphere1_joint" type="fixed">
+    <origin rpy="0 0 0" xyz="0 0 0"/>
+    <parent link="thing_tool"/>
+    <child link="robust_sphere1_link"/>
+  </joint>
+  <link name="robust_sphere2_link">
+    <visual>
+      <origin rpy="0 0 0" xyz="0 0 0.3"/>
+      <geometry>
+        <sphere radius="0.12"/>
+      </geometry>
+      <material name="seethrough"/>
+    </visual>
+  </link>
+  <joint name="robust_sphere2_joint" type="fixed">
+    <origin rpy="0 0 0" xyz="0 0 0"/>
+    <parent link="thing_tool"/>
+    <child link="robust_sphere2_link"/>
+  </joint>
   <!-- Collision element to protect the balanced objects -->
   <!-- <link name="balanced_object_collision_link"> -->

Commit message: Basic dynamic obstacle avoidance with robust constraints and flat configuration.

File: tray_balance_assets/urdf/mm_pyb.urdf (robot description, URDF)
Before this commit: robot Thing, 29 links, 28 joints
Links:
- removed link robust_sphere2_link
- link robust_sphere1_link: geometry visual sphere radius=0.1
Joints:
- removed joint robust_sphere2_joint

Commit message: Experiment with mapping depth map -> world points

File: tray_balance_assets/urdf/mm_pyb.urdf (robot description, URDF)
Before this commit: robot Thing, 28 links, 27 joints
Links:
- removed link robust_sphere1_link
Joints:
- removed joint robust_sphere1_joint

Commit message: Bring in GhostSpheres from pyb_utils.

File: tray_balance_assets/urdf/mm_pyb.urdf (robot description, URDF)
Before this commit: robot Thing, 27 links, 26 joints
Links:
- added link elbow_collision_link
Joints:
- added joint elbow_collision_joint: type fixed, parent ur10_arm_forearm_link, child elbow_collision_link, origin xyz=0 0 0 rpy=0 0 0

Commit message: Use pyb_utils GhostSpheres to show collision spheres.

File: tray_balance_assets/urdf/mm_pyb.urdf (robot description, URDF)
Before this commit: robot Thing, 28 links, 27 joints
Links:
- removed link elbow_collision_link
Joints:
- removed joint elbow_collision_joint

Commit message: Static obstacle experiments.

File: tray_balance_assets/urdf/mm_pyb.urdf (robot description, URDF)
Before this commit: robot Thing, 27 links, 26 joints
Links:
- added link base_collision_link; visual box size=1.0 0.8 0.3
- added link elbow_collision_link; visual sphere radius=0.15
- added link forearm_collision_link; visual cylinder length=0.6 radius=0.06
- added link shoulder_collision_link; visual sphere radius=0.15
- added link wrist_collision_link; visual sphere radius=0.15
Joints:
- added joint base_collision_joint: type fixed, parent base_link, child base_collision_link, origin xyz=0 0 0.01 rpy=0 0 0
- added joint elbow_collision_joint: type fixed, parent ur10_arm_forearm_link, child elbow_collision_link, origin xyz=0 0 0 rpy=0 0 0
- added joint forearm_collision_joint: type fixed, parent ur10_arm_forearm_link, child forearm_collision_link, origin xyz=0 0 0 rpy=0 0 0
- added joint shoulder_collision_joint: type fixed, parent ur10_arm_upper_arm_link, child shoulder_collision_link, origin xyz=0 0 0 rpy=0 0 0
- added joint wrist_collision_joint: type fixed, parent ur10_arm_wrist_3_link, child wrist_collision_link, origin xyz=0 0 0 rpy=0 0 0

Commit message: Taking pictures for eye candy image.

File: tray_balance_assets/urdf/mm_pyb.urdf (robot description, URDF)
Before this commit: robot Thing, 32 links, 31 joints
Links:
- removed link base_collision_link
- removed link elbow_collision_link
- removed link forearm_collision_link
- removed link shoulder_collision_link
- removed link wrist_collision_link
Joints:
- removed joint base_collision_joint
- removed joint elbow_collision_joint
- removed joint forearm_collision_joint
- removed joint shoulder_collision_joint
- removed joint wrist_collision_joint
