Commit message: Move assets to a separate ROS package.
Some clean up in older scripts.

File: tray_balance_assets/urdf/mm_ocs2.urdf (robot description, URDF)
Before this commit: robot Thing, 27 links, 26 joints
Links:
- removed link world_link
- removed link x_prismatic_link
- removed link y_prismatic_link
- added link balanced_object_collision_link; collision cylinder length=0.1 radius=0.25; visual cylinder length=0.1 radius=0.25
- added link base_collision_link; collision box size=1.0 0.8 0.3; visual box size=1.0 0.8 0.3
- added link elbow_collision_link; collision sphere radius=0.15; visual sphere radius=0.15
- added link forearm_collision_link; collision cylinder length=0.6 radius=0.06; visual cylinder length=0.6 radius=0.06
- added link forearm_collision_sphere_link1; collision sphere radius=0.15; visual sphere radius=0.15
- added link forearm_collision_sphere_link2; collision sphere radius=0.15; visual sphere radius=0.15
- added link front_left_wheel_link, mass 2.3; collision cylinder length=0.079 radius=0.0759; visual mesh filename=package://tray_balance_assets/meshes/ridgeback/wheel.stl
- added link front_right_wheel_link, mass 2.3; collision cylinder length=0.079 radius=0.0759; visual mesh filename=package://tray_balance_assets/meshes/ridgeback/wheel.stl
- added link front_rocker_link, mass 10.267; visual mesh filename=package://tray_balance_assets/meshes/ridgeback/rocker.stl
- added link rear_left_wheel_link, mass 2.3; collision cylinder length=0.079 radius=0.0759; visual mesh filename=package://tray_balance_assets/meshes/ridgeback/wheel.stl
- added link rear_right_wheel_link, mass 2.3; collision cylinder length=0.079 radius=0.0759; visual mesh filename=package://tray_balance_assets/meshes/ridgeback/wheel.stl
- added link rear_rocker_link, mass 10.267; visual mesh filename=package://tray_balance_assets/meshes/ridgeback/rocker.stl
- added link shoulder_collision_link; collision sphere radius=0.15; visual sphere radius=0.15
- added link upper_arm_collision_link; collision cylinder length=0.65 radius=0.06; visual cylinder length=0.65 radius=0.06
- added link wrist_collision_link; collision sphere radius=0.15; visual sphere radius=0.15
- link arch_link: geometry visual mesh filename=package://tray_balance_assets/meshes/tor11_mech.dae
- link axle_link: geometry visual mesh filename=package://tray_balance_assets/meshes/ridgeback/axle.stl
- link base_link: mass 0.01 -> None
- link chassis_link: geometry collision box size=1.0 0.8 0.3; visual mesh filename=package://tray_balance_assets/meshes/ridgeback/body.stl
- link front_cover_link: geometry visual mesh filename=package://tray_balance_assets/meshes/ridgeback/end-cover.stl
- link front_lights_link: geometry visual mesh filename=package://tray_balance_assets/meshes/ridgeback/lights.stl
- link left_side_cover_link: geometry visual mesh filename=package://tray_balance_assets/meshes/ridgeback/side-cover.s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
- link rear_cover_link: geometry visual mesh filename=package://tray_balance_assets/meshes/ridgeback/end-cover.stl
- link rear_lights_link: geometry visual mesh filename=package://tray_balance_assets/meshes/ridgeback/lights.stl
- link right_side_cover_link: geometry visual mesh filename=package://tray_balance_assets/meshes/ridgeback/side-cover.s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
- link top_link: geometry collision mesh filename=package://tray_balance_assets/meshes/ridgeback/top.stl; visual mesh filename=package://tray_balance_assets/meshes/ridgeback/top.stl
- link ur10_arm_base_link: geometry collision mesh filename=package://tray_balance_assets/meshes/ur10/collision/base.stl; visual mesh filename=package://tray_balance_assets/meshes/ur10/visual/base.dae
- link ur10_arm_forearm_link: geometry collision mesh filename=package://tray_balance_assets/meshes/ur10/collision/forearm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; visual mesh filename=package://tray_balance_assets/meshes/ur10/visual/forearm.dae
- link ur10_arm_shoulder_link: geometry collision mesh filename=package://tray_balance_assets/meshes/ur10/collision/shoulde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; visual mesh filename=package://tray_balance_assets/meshes/ur10/visual/shoulder.d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
- link ur10_arm_upper_arm_link: geometry collision mesh filename=package://tray_balance_assets/meshes/ur10/collision/upperar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; visual mesh filename=package://tray_balance_assets/meshes/ur10/visual/upperarm.d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
- link ur10_arm_wrist_1_link: geometry collision mesh filename=package://tray_balance_assets/meshes/ur10/collision/wrist1.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; visual mesh filename=package://tray_balance_assets/meshes/ur10/visual/wrist1.dae
- link ur10_arm_wrist_2_link: geometry collision mesh filename=package://tray_balance_assets/meshes/ur10/collision/wrist2.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; visual mesh filename=package://tray_balance_assets/meshes/ur10/visual/wrist2.dae
- link ur10_arm_wrist_3_link: geometry collision mesh filename=package://tray_balance_assets/meshes/ur10/collision/wrist3.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; visual mesh filename=package://tray_balance_assets/meshes/ur10/visual/wrist3.dae
Joints:
- removed joint base_to_y_joint
- removed joint x_to_world_joint
- removed joint y_to_x_joint
- added joint balanced_object_collision_joint: type fixed, parent thing_tool, child balanced_object_collision_link, origin xyz=0 0 0 rpy=0 0 0
- added joint base_collision_joint: type fixed, parent base_link, child base_collision_link, origin xyz=0 0 0.01 rpy=0 0 0
- added joint elbow_collision_joint: type fixed, parent ur10_arm_forearm_link, child elbow_collision_link, origin xyz=0 0 0 rpy=0 0 0
- added joint forearm_collision_joint: type fixed, parent ur10_arm_forearm_link, child forearm_collision_link, origin xyz=0 0 0 rpy=0 0 0
- added joint forearm_collision_sphere_joint1: type fixed, parent ur10_arm_forearm_link, child forearm_collision_sphere_link1, origin xyz=0 0 0.2 rpy=0 0 0
- added joint forearm_collision_sphere_joint2: type fixed, parent ur10_arm_forearm_link, child forearm_collision_sphere_link2, origin xyz=0 0 0.4 rpy=0 0 0
- added joint front_left_wheel: type fixed, parent front_rocker_link, child front_left_wheel_link, origin xyz=0 0.2755 0 rpy=0 0 0, axis 0 1 0
- added joint front_right_wheel: type fixed, parent front_rocker_link, child front_right_wheel_link, origin xyz=0 -0.2755 0 rpy=0 0 0, axis 0 1 0
- added joint front_rocker: type fixed, parent axle_link, child front_rocker_link, origin xyz=0.319 0 0 rpy=0 0 0, axis 1 0 0, limit lower=-0.08726 upper=0.08726 effort=0 velocity=0
- added joint rear_left_wheel: type fixed, parent rear_rocker_link, child rear_left_wheel_link, origin xyz=0 0.2755 0 rpy=0 0 0, axis 0 1 0
- added joint rear_right_wheel: type fixed, parent rear_rocker_link, child rear_right_wheel_link, origin xyz=0 -0.2755 0 rpy=0 0 0, axis 0 1 0
- added joint rear_rocker: type fixed, parent axle_link, child rear_rocker_link, origin xyz=-0.319 0 0 rpy=0 0 0, axis 1 0 0, limit effort=0 velocity=0
- added joint shoulder_collision_joint: type fixed, parent ur10_arm_upper_arm_link, child shoulder_collision_link, origin xyz=0 0 0 rpy=0 0 0
- added joint upper_arm_collision_joint: type fixed, parent ur10_arm_upper_arm_link, child upper_arm_collision_link, origin xyz=0 0 0 rpy=0 0 0
- added joint wrist_collision_joint: type fixed, parent ur10_arm_wrist_3_link, child wrist_collision_link, origin xyz=0 0 0 rpy=0 0 0
- joint base_link_joint: origin xyz=0 0 0 rpy=0 0 0 -> xyz=0 0 0.01 rpy=0 0 0
