Commit message: xacro URDF files to resolve ROS package paths

File: tray_balance_assets/urdf/mm_ocs2.urdf (robot description, URDF)
Before this commit: robot Thing, 39 links, 38 joints
Links:
- link arch_link: geometry visual mesh filename=file:///home/adam/phd/code/mm/tray_balance/catkin_ws/src/tr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
- link axle_link: geometry visual mesh filename=file:///home/adam/phd/code/mm/tray_balance/catkin_ws/src/tr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
- link chassis_link: geometry collision box size=1.0 0.8 0.3; visual mesh filename=file:///home/adam/phd/code/mm/tray_balance/catkin_ws/src/tr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
- link front_cover_link: geometry visual mesh filename=file:///home/adam/phd/code/mm/tray_balance/catkin_ws/src/tr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
- link front_left_wheel_link: geometry collision cylinder length=0.079 radius=0.0759; visual mesh filename=file:///home/adam/phd/code/mm/tray_balance/catkin_ws/src/tr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
- link front_lights_link: geometry visual mesh filename=file:///home/adam/phd/code/mm/tray_balance/catkin_ws/src/tr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
- link front_right_wheel_link: geometry collision cylinder length=0.079 radius=0.0759; visual mesh filename=file:///home/adam/phd/code/mm/tray_balance/catkin_ws/src/tr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
- link front_rocker_link: geometry visual mesh filename=file:///home/adam/phd/code/mm/tray_balance/catkin_ws/src/tr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
- link left_side_cover_link: geometry visual mesh filename=file:///home/adam/phd/code/mm/tray_balance/catkin_ws/src/tr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
- link rear_cover_link: geometry visual mesh filename=file:///home/adam/phd/code/mm/tray_balance/catkin_ws/src/tr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
- link rear_left_wheel_link: geometry collision cylinder length=0.079 radius=0.0759; visual mesh filename=file:///home/adam/phd/code/mm/tray_balance/catkin_ws/src/tr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
- link rear_lights_link: geometry visual mesh filename=file:///home/adam/phd/code/mm/tray_balance/catkin_ws/src/tr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
- link rear_right_wheel_link: geometry collision cylinder length=0.079 radius=0.0759; visual mesh filename=file:///home/adam/phd/code/mm/tray_balance/catkin_ws/src/tr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
- link rear_rocker_link: geometry visual mesh filename=file:///home/adam/phd/code/mm/tray_balance/catkin_ws/src/tr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
- link right_side_cover_link: geometry visual mesh filename=file:///home/adam/phd/code/mm/tray_balance/catkin_ws/src/tr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
- link top_link: geometry collision mesh filename=file:///home/adam/phd/code/mm/tray_balance/catkin_ws/src/tr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; visual mesh filename=file:///home/adam/phd/code/mm/tray_balance/catkin_ws/src/tr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
- link ur10_arm_base_link: geometry collision mesh filename=file:///home/adam/phd/code/mm/tray_balance/catkin_ws/src/tr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; visual mesh filename=file:///home/adam/phd/code/mm/tray_balance/catkin_ws/src/tr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
- link ur10_arm_forearm_link: geometry collision mesh filename=file:///home/adam/phd/code/mm/tray_balance/catkin_ws/src/tr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; visual mesh filename=file:///home/adam/phd/code/mm/tray_balance/catkin_ws/src/tr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
- link ur10_arm_shoulder_link: geometry collision mesh filename=file:///home/adam/phd/code/mm/tray_balance/catkin_ws/src/tr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; visual mesh filename=file:///home/adam/phd/code/mm/tray_balance/catkin_ws/src/tr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
- link ur10_arm_upper_arm_link: geometry collision mesh filename=file:///home/adam/phd/code/mm/tray_balance/catkin_ws/src/tr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; visual mesh filename=file:///home/adam/phd/code/mm/tray_balance/catkin_ws/src/tr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
- link ur10_arm_wrist_1_link: geometry collision mesh filename=file:///home/adam/phd/code/mm/tray_balance/catkin_ws/src/tr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; visual mesh filename=file:///home/adam/phd/code/mm/tray_balance/catkin_ws/src/tr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
- link ur10_arm_wrist_2_link: geometry collision mesh filename=file:///home/adam/phd/code/mm/tray_balance/catkin_ws/src/tr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; visual mesh filename=file:///home/adam/phd/code/mm/tray_balance/catkin_ws/src/tr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
- link ur10_arm_wrist_3_link: geometry collision mesh filename=file:///home/adam/phd/code/mm/tray_balance/catkin_ws/src/tr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; visual mesh filename=file:///home/adam/phd/code/mm/tray_balance/catkin_ws/src/tr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

File: tray_balance_assets/urdf/mm_ocs2.urdf.xacro (robot description, xacro)
@@ -1,7 +1,3 @@
-<?xml version="1.0" ?>
-<!-- =================================================================================== -->
-<!-- |    This document was autogenerated by xacro from mm_pyb.urdf.xacro              | -->
-<!-- |    EDITING THIS FILE BY HAND IS NOT RECOMMENDED                                 | -->
-<!-- =================================================================================== -->
+<?xml version="1.0" encoding="utf-8"?>
 <robot name="Thing">
   <material name="dark_grey">
@@ -24,57 +20,156 @@
   </material>
   <material name="seethrough">
-    <color rgba="0.0 1.0 0.0 0.25"/>
+    <color rgba="1.0 0.0 0.0 0.5"/>
   </material>
-  <link name="world_link">
-    <inertial>
-      <mass value="0"/>
-      <inertia ixx="0.2125" ixy="-0.005" ixz="0.0225" iyy="0.205" iyz="0.045" izz="0.0125"/>
-      <origin rpy="0 0 0" xyz="0 0 0"/>
-    </inertial>
-  </link>
-  <link name="x_prismatic_link">
-    <inertial>
-      <mass value="0.01"/>
-      <inertia ixx="0.01" ixy="0" ixz="0" iyy="0.01" iyz="0" izz="0.01"/>
-      <origin rpy="0 0 0" xyz="0 0 0"/>
-    </inertial>
-  </link>
-  <joint name="x_to_world_joint" type="prismatic">
-    <parent link="world_link"/>
-    <child link="x_prismatic_link"/>
+  <link name="front_rocker_link">
+    <visual>
+      <origin rpy="1.57079632679 0 1.57079632679" xyz="0 0 0"/>
+      <geometry>
+        <mesh filename="file://$(find tray_balance_assets)/meshes/ridgeback/rocker.stl"/>
+      </geometry>
+      <material name="black"/>
+    </visual>
+    <inertial>
+      <origin rpy="1.57079632679 0 1.57079632679" xyz="0 0 0"/>
+      <mass value="10.267"/>
+      <inertia ixx="0.0288" ixy="2.20484e-6" ixz="-1.3145e-5" iyy="0.4324" iyz="1.8944e-3" izz="0.4130"/>
+    </inertial>
+  </link>
+  <joint name="front_rocker" type="fixed">
+    <parent link="axle_link"/>
+    <child link="front_rocker_link"/>
+    <origin rpy="0 0 0" xyz="0.319 0 0"/>
     <axis xyz="1 0 0"/>
-    <origin rpy="0 0 0" xyz="0 0 0"/>
-    <limit effort="0.0" velocity="1000.0"/>
-  </joint>
-  <link name="y_prismatic_link">
-    <inertial>
-      <mass value="0.01"/>
-      <inertia ixx="0.01" ixy="0" ixz="0" iyy="0.01" iyz="0" izz="0.01"/>
-      <origin rpy="0 0 0" xyz="0 0 0"/>
-    </inertial>
-  </link>
-  <joint name="y_to_x_joint" type="prismatic">
-    <parent link="x_prismatic_link"/>
-    <child link="y_prismatic_link"/>
+    <limit effort="0" lower="-0.08726" upper="0.08726" velocity="0"/>
+  </joint>
+  <link name="front_left_wheel_link">
+    <visual>
+      <origin rpy="1.57079632679 0 0" xyz="0 0 0"/>
+      <geometry>
+        <mesh filename="file://$(find tray_balance_assets)/meshes/ridgeback/wheel.stl"/>
+      </geometry>
+      <material name="black"/>
+    </visual>
+    <collision>
+      <origin rpy="1.57079632679 0 0" xyz="0 0 0"/>
+      <geometry>
+        <cylinder length="0.079" radius="0.0759"/>
+      </geometry>
+    </collision>
+    <inertial>
+      <origin rpy="0 0 0" xyz="0 0 0"/>
+      <mass value="2.3"/>
+      <inertia ixx="3.3212e-3" ixy="0" ixz="0" iyy="6.6424e-3" iyz="0" izz="3.3212e-3"/>
+    </inertial>
+  </link>
+  <joint name="front_left_wheel" type="fixed">
+    <parent link="front_rocker_link"/>
+    <child link="front_left_wheel_link"/>
+    <origin rpy="0 0 0" xyz="0 0.2755 0"/>
     <axis xyz="0 1 0"/>
-    <origin rpy="0 0 0" xyz="0 0 0"/>
-    <limit effort="0.0" velocity="1000.0"/>
-  </joint>
-  <!-- Note the z-offset to raise the base off the ground, to avoid collision issues. Without this, there are vibrations and other artifacts from resolving the ground collision that result in significant error in the balanced object. -->
-  <joint name="base_to_y_joint" type="continuous">
-    <parent link="y_prismatic_link"/>
-    <child link="base_link"/>
-    <axis xyz="0 0 1"/>
+  </joint>
+  <link name="front_right_wheel_link">
+    <visual>
+      <origin rpy="1.57079632679 0 0" xyz="0 0 0"/>
+      <geometry>
+        <mesh filename="file://$(find tray_balance_assets)/meshes/ridgeback/wheel.stl"/>
+      </geometry>
+      <material name="black"/>
+    </visual>
+    <collision>
+      <origin rpy="1.57079632679 0 0" xyz="0 0 0"/>
+      <geometry>
+        <cylinder length="0.079" radius="0.0759"/>
+      </geometry>
+    </collision>
+    <inertial>
+      <origin rpy="0 0 0" xyz="0 0 0"/>
+      <mass value="2.3"/>
+      <inertia ixx="3.3212e-3" ixy="0" ixz="0" iyy="6.6424e-3" iyz="0" izz="3.3212e-3"/>
+    </inertial>
+  </link>
+  <joint name="front_right_wheel" type="fixed">
+    <parent link="front_rocker_link"/>
+    <child link="front_right_wheel_link"/>
+    <origin rpy="0 0 0" xyz="0 -0.2755 0"/>
+    <axis xyz="0 1 0"/>
+  </joint>
+  <link name="rear_rocker_link">
+    <visual>
+      <origin rpy="1.57079632679 0 1.57079632679" xyz="0 0 0"/>
+      <geometry>
+        <mesh filename="file://$(find tray_balance_assets)/meshes/ridgeback/rocker.stl"/>
+      </geometry>
+      <material name="black"/>
+    </visual>
+    <inertial>
+      <origin rpy="1.57079632679 0 1.57079632679" xyz="0 0 0"/>
+      <mass value="10.267"/>
+      <inertia ixx="0.0288" ixy="2.20484e-6" ixz="-1.3145e-5" iyy="0.4324" iyz="1.8944e-3" izz="0.4130"/>
+    </inertial>
+  </link>
+  <joint name="rear_rocker" type="fixed">
+    <parent link="axle_link"/>
+    <child link="rear_rocker_link"/>
+    <origin rpy="0 0 0" xyz="-0.319 0 0"/>
+    <axis xyz="1 0 0"/>
+    <limit effort="0" velocity="0"/>
+  </joint>
+  <link name="rear_left_wheel_link">
+    <visual>
+      <origin rpy="1.57079632679 0 0" xyz="0 0 0"/>
+      <geometry>
+        <mesh filename="file://$(find tray_balance_assets)/meshes/ridgeback/wheel.stl"/>
+      </geometry>
+      <material name="black"/>
+    </visual>
+    <collision>
+      <origin rpy="1.57079632679 0 0" xyz="0 0 0"/>
+      <geometry>
+        <cylinder length="0.079" radius="0.0759"/>
+      </geometry>
+    </collision>
+    <inertial>
+      <origin rpy="0 0 0" xyz="0 0 0"/>
+      <mass value="2.3"/>
+      <inertia ixx="3.3212e-3" ixy="0" ixz="0" iyy="6.6424e-3" iyz="0" izz="3.3212e-3"/>
+    </inertial>
+  </link>
+  <joint name="rear_left_wheel" type="fixed">
+    <parent link="rear_rocker_link"/>
+    <child link="rear_left_wheel_link"/>
+    <origin rpy="0 0 0" xyz="0 0.2755 0"/>
+    <axis xyz="0 1 0"/>
+  </joint>
+  <link name="rear_right_wheel_link">
+    <visual>
+      <origin rpy="1.57079632679 0 0" xyz="0 0 0"/>
+      <geometry>
+        <mesh filename="file://$(find tray_balance_assets)/meshes/ridgeback/wheel.stl"/>
+      </geometry>
+      <material name="black"/>
+    </visual>
+    <collision>
+      <origin rpy="1.57079632679 0 0" xyz="0 0 0"/>
+      <geometry>
+        <cylinder length="0.079" radius="0.0759"/>
+      </geometry>
+    </collision>
+    <inertial>
+      <origin rpy="0 0 0" xyz="0 0 0"/>
+      <mass value="2.3"/>
+      <inertia ixx="3.3212e-3" ixy="0" ixz="0" iyy="6.6424e-3" iyz="0" izz="3.3212e-3"/>
+    </inertial>
+  </link>
+  <joint name="rear_right_wheel" type="fixed">
+    <parent link="rear_rocker_link"/>
+    <child link="rear_right_wheel_link"/>
+    <origin rpy="0 0 0" xyz="0 -0.2755 0"/>
+    <axis xyz="0 1 0"/>
+  </joint>
+  <link name="base_link"/>
+    <!-- 0.01 z-offset is to match the pyb URDF, which requires a small offset to avoid ground collisions. -->
+  <joint name="base_link_joint" type="fixed">
     <origin rpy="0 0 0" xyz="0 0 0.01"/>
-  </joint>
-  <link name="base_link">
-    <inertial>
-      <mass value="0.01"/>
-      <inertia ixx="0.01" ixy="0" ixz="0" iyy="0.01" iyz="0" izz="0.01"/>
-      <origin rpy="0 0 0" xyz="0 0 0"/>
-    </inertial>
-  </link>
-  <joint name="base_link_joint" type="fixed">
-    <origin rpy="0 0 0" xyz="0 0 0"/>
     <parent link="base_link"/>
     <child link="chassis_link"/>
@@ -88,5 +183,5 @@
       <!-- <origin xyz="0 0 0"/> -->
       <geometry>
-        <mesh filename="file:///home/adam/phd/code/mm/tray_balance/catkin_ws/src/tray_balance/tray_balance_assets/meshes/ridgeback/body.stl"/>
+        <mesh filename="file://$(find tray_balance_assets)/meshes/ridgeback/body.stl"/>
       </geometry>
       <material name="black"/>
@@ -124,5 +219,5 @@
       <origin rpy="0 0 3.14159265359" xyz="0 0 0"/>
       <geometry>
-        <mesh filename="file:///home/adam/phd/code/mm/tray_balance/catkin_ws/src/tray_balance/tray_balance_assets/meshes/ridgeback/side-cover.stl"/>
+        <mesh filename="file://$(find tray_balance_assets)/meshes/ridgeback/side-cover.stl"/>
       </geometry>
       <material name="yellow"/>
@@ -133,5 +228,5 @@
       <origin rpy="0 0 0" xyz="0 0 0"/>
       <geometry>
-        <mesh filename="file:///home/adam/phd/code/mm/tray_balance/catkin_ws/src/tray_balance/tray_balance_assets/meshes/ridgeback/side-cover.stl"/>
+        <mesh filename="file://$(find tray_balance_assets)/meshes/ridgeback/side-cover.stl"/>
       </geometry>
       <material name="yellow"/>
@@ -147,5 +242,5 @@
       <origin rpy="0 0 0" xyz="0 0 0"/>
       <geometry>
-        <mesh filename="file:///home/adam/phd/code/mm/tray_balance/catkin_ws/src/tray_balance/tray_balance_assets/meshes/ridgeback/end-cover.stl"/>
+        <mesh filename="file://$(find tray_balance_assets)/meshes/ridgeback/end-cover.stl"/>
       </geometry>
       <material name="black"/>
@@ -161,5 +256,5 @@
       <origin rpy="0 0 3.14159265359" xyz="0 0 0"/>
       <geometry>
-        <mesh filename="file:///home/adam/phd/code/mm/tray_balance/catkin_ws/src/tray_balance/tray_balance_assets/meshes/ridgeback/end-cover.stl"/>
+        <mesh filename="file://$(find tray_balance_assets)/meshes/ridgeback/end-cover.stl"/>
       </geometry>
       <material name="black"/>
@@ -180,5 +275,5 @@
       <origin rpy="0 0 0" xyz="0 0 0"/>
       <geometry>
-        <mesh filename="file:///home/adam/phd/code/mm/tray_balance/catkin_ws/src/tray_balance/tray_balance_assets/meshes/ridgeback/lights.stl"/>
+        <mesh filename="file://$(find tray_balance_assets)/meshes/ridgeback/lights.stl"/>
       </geometry>
       <material name="white"/>
@@ -189,5 +284,5 @@
       <origin rpy="0 0 3.14159265359" xyz="0 0 0"/>
       <geometry>
-        <mesh filename="file:///home/adam/phd/code/mm/tray_balance/catkin_ws/src/tray_balance/tray_balance_assets/meshes/ridgeback/lights.stl"/>
+        <mesh filename="file://$(find tray_balance_assets)/meshes/ridgeback/lights.stl"/>
       </geometry>
       <material name="red"/>
@@ -203,12 +298,12 @@
       <origin rpy="0 0 0" xyz="0 0 0"/>
       <geometry>
-        <mesh filename="file:///home/adam/phd/code/mm/tray_balance/catkin_ws/src/tray_balance/tray_balance_assets/meshes/ridgeback/top.stl"/>
-      </geometry>
-      <material name="black"/>
-    </visual>
-    <collision>
-      <origin rpy="0 0 0" xyz="0 0 0"/>
-      <geometry>
-        <mesh filename="file:///home/adam/phd/code/mm/tray_balance/catkin_ws/src/tray_balance/tray_balance_assets/meshes/ridgeback/top.stl"/>
+        <mesh filename="file://$(find tray_balance_assets)/meshes/ridgeback/top.stl"/>
+      </geometry>
+      <material name="black"/>
+    </visual>
+    <collision>
+      <origin rpy="0 0 0" xyz="0 0 0"/>
+      <geometry>
+        <mesh filename="file://$(find tray_balance_assets)/meshes/ridgeback/top.stl"/>
       </geometry>
     </collision>
@@ -223,5 +318,5 @@
       <origin rpy="0 1.57079632679 0" xyz="0 0 0"/>
       <geometry>
-        <mesh filename="file:///home/adam/phd/code/mm/tray_balance/catkin_ws/src/tray_balance/tray_balance_assets/meshes/ridgeback/axle.stl"/>
+        <mesh filename="file://$(find tray_balance_assets)/meshes/ridgeback/axle.stl"/>
       </geometry>
       <material name="black"/>
@@ -249,5 +344,5 @@
     <visual>
       <geometry>
-        <mesh filename="file:///home/adam/phd/code/mm/tray_balance/catkin_ws/src/tray_balance/tray_balance_assets/meshes/tor11_mech.dae"/>
+        <mesh filename="file://$(find tray_balance_assets)/meshes/tor11_mech.dae"/>
       </geometry>
     </visual>
@@ -271,5 +366,5 @@
     <visual>
       <geometry>
-        <mesh filename="file:///home/adam/phd/code/mm/tray_balance/catkin_ws/src/tray_balance/tray_balance_assets/meshes/ur10/visual/base.dae"/>
+        <mesh filename="file://$(find tray_balance_assets)/meshes/ur10/visual/base.dae"/>
       </geometry>
       <material name="LightGrey">
@@ -279,5 +374,5 @@
     <collision>
       <geometry>
-        <mesh filename="file:///home/adam/phd/code/mm/tray_balance/catkin_ws/src/tray_balance/tray_balance_assets/meshes/ur10/collision/base.stl"/>
+        <mesh filename="file://$(find tray_balance_assets)/meshes/ur10/collision/base.stl"/>
       </geometry>
     </collision>
@@ -299,5 +394,5 @@
     <visual>
       <geometry>
-        <mesh filename="file:///home/adam/phd/code/mm/tray_balance/catkin_ws/src/tray_balance/tray_balance_assets/meshes/ur10/visual/shoulder.dae"/>
+        <mesh filename="file://$(find tray_balance_assets)/meshes/ur10/visual/shoulder.dae"/>
       </geometry>
       <material name="LightGrey">
@@ -307,5 +402,5 @@
     <collision>
       <geometry>
-        <mesh filename="file:///home/adam/phd/code/mm/tray_balance/catkin_ws/src/tray_balance/tray_balance_assets/meshes/ur10/collision/shoulder.stl"/>
+        <mesh filename="file://$(find tray_balance_assets)/meshes/ur10/collision/shoulder.stl"/>
       </geometry>
     </collision>
@@ -327,5 +422,5 @@
     <visual>
       <geometry>
-        <mesh filename="file:///home/adam/phd/code/mm/tray_balance/catkin_ws/src/tray_balance/tray_balance_assets/meshes/ur10/visual/upperarm.dae"/>
+        <mesh filename="file://$(find tray_balance_assets)/meshes/ur10/visual/upperarm.dae"/>
       </geometry>
       <material name="LightGrey">
@@ -335,5 +430,5 @@
     <collision>
       <geometry>
-        <mesh filename="file:///home/adam/phd/code/mm/tray_balance/catkin_ws/src/tray_balance/tray_balance_assets/meshes/ur10/collision/upperarm.stl"/>
+        <mesh filename="file://$(find tray_balance_assets)/meshes/ur10/collision/upperarm.stl"/>
       </geometry>
     </collision>
@@ -355,5 +450,5 @@
     <visual>
       <geometry>
-        <mesh filename="file:///home/adam/phd/code/mm/tray_balance/catkin_ws/src/tray_balance/tray_balance_assets/meshes/ur10/visual/forearm.dae"/>
+        <mesh filename="file://$(find tray_balance_assets)/meshes/ur10/visual/forearm.dae"/>
       </geometry>
       <material name="LightGrey">
@@ -363,5 +458,5 @@
     <collision>
       <geometry>
-        <mesh filename="file:///home/adam/phd/code/mm/tray_balance/catkin_ws/src/tray_balance/tray_balance_assets/meshes/ur10/collision/forearm.stl"/>
+        <mesh filename="file://$(find tray_balance_assets)/meshes/ur10/collision/forearm.stl"/>
       </geometry>
     </collision>
@@ -383,5 +478,5 @@
     <visual>
       <geometry>
-        <mesh filename="file:///home/adam/phd/code/mm/tray_balance/catkin_ws/src/tray_balance/tray_balance_assets/meshes/ur10/visual/wrist1.dae"/>
+        <mesh filename="file://$(find tray_balance_assets)/meshes/ur10/visual/wrist1.dae"/>
       </geometry>
       <material name="LightGrey">
@@ -391,5 +486,5 @@
     <collision>
       <geometry>
-        <mesh filename="file:///home/adam/phd/code/mm/tray_balance/catkin_ws/src/tray_balance/tray_balance_assets/meshes/ur10/collision/wrist1.stl"/>
+        <mesh filename="file://$(find tray_balance_assets)/meshes/ur10/collision/wrist1.stl"/>
       </geometry>
     </collision>
@@ -411,5 +506,5 @@
     <visual>
       <geometry>
-        <mesh filename="file:///home/adam/phd/code/mm/tray_balance/catkin_ws/src/tray_balance/tray_balance_assets/meshes/ur10/visual/wrist2.dae"/>
+        <mesh filename="file://$(find tray_balance_assets)/meshes/ur10/visual/wrist2.dae"/>
       </geometry>
       <material name="LightGrey">
@@ -419,5 +514,5 @@
     <collision>
       <geometry>
-        <mesh filename="file:///home/adam/phd/code/mm/tray_balance/catkin_ws/src/tray_balance/tray_balance_assets/meshes/ur10/collision/wrist2.stl"/>
+        <mesh filename="file://$(find tray_balance_assets)/meshes/ur10/collision/wrist2.stl"/>
       </geometry>
     </collision>
@@ -439,5 +534,5 @@
     <visual>
       <geometry>
-        <mesh filename="file:///home/adam/phd/code/mm/tray_balance/catkin_ws/src/tray_balance/tray_balance_assets/meshes/ur10/visual/wrist3.dae"/>
+        <mesh filename="file://$(find tray_balance_assets)/meshes/ur10/visual/wrist3.dae"/>
       </geometry>
       <material name="LightGrey">
@@ -447,5 +542,5 @@
     <collision>
       <geometry>
-        <mesh filename="file:///home/adam/phd/code/mm/tray_balance/catkin_ws/src/tray_balance/tray_balance_assets/meshes/ur10/collision/wrist3.stl"/>
+        <mesh filename="file://$(find tray_balance_assets)/meshes/ur10/collision/wrist3.stl"/>
       </geometry>
     </collision>
@@ -503,9 +598,4 @@
     </collision>
   </link>
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