Commit message: xacro URDF files to resolve ROS package paths

File: tray_balance_assets/urdf/mm_pyb.urdf.xacro (robot description, xacro)
@@ -1,7 +1,3 @@
-<?xml version="1.0" ?>
-<!-- =================================================================================== -->
-<!-- |    This document was autogenerated by xacro from mm_pyb.urdf.xacro              | -->
-<!-- |    EDITING THIS FILE BY HAND IS NOT RECOMMENDED                                 | -->
-<!-- =================================================================================== -->
+<?xml version="1.0" encoding="utf-8"?>
 <robot name="Thing">
   <material name="dark_grey">
@@ -33,12 +29,12 @@
     </inertial>
   </link>
-  <link name="x_prismatic_link">
-    <inertial>
-      <mass value="0.01"/>
-      <inertia ixx="0.01" ixy="0" ixz="0" iyy="0.01" iyz="0" izz="0.01"/>
-      <origin rpy="0 0 0" xyz="0 0 0"/>
-    </inertial>
-  </link>
-  <joint name="x_to_world_joint" type="prismatic">
+	<link name="x_prismatic_link">
+	 <inertial>
+     <mass value="0.01"/>
+     <inertia ixx="0.01" ixy="0" ixz="0" iyy="0.01" iyz="0" izz="0.01"/>
+     <origin rpy="0 0 0" xyz="0 0 0"/>
+    </inertial>
+  </link>
+	<joint name="x_to_world_joint" type="prismatic">
     <parent link="world_link"/>
     <child link="x_prismatic_link"/>
@@ -47,12 +43,12 @@
     <limit effort="0.0" velocity="1000.0"/>
   </joint>
-  <link name="y_prismatic_link">
-    <inertial>
-      <mass value="0.01"/>
-      <inertia ixx="0.01" ixy="0" ixz="0" iyy="0.01" iyz="0" izz="0.01"/>
-      <origin rpy="0 0 0" xyz="0 0 0"/>
-    </inertial>
-  </link>
-  <joint name="y_to_x_joint" type="prismatic">
+	<link name="y_prismatic_link">
+	 <inertial>
+     <mass value="0.01"/>
+     <inertia ixx="0.01" ixy="0" ixz="0" iyy="0.01" iyz="0" izz="0.01"/>
+     <origin rpy="0 0 0" xyz="0 0 0"/>
+    </inertial>
+  </link>
+	<joint name="y_to_x_joint" type="prismatic">
     <parent link="x_prismatic_link"/>
     <child link="y_prismatic_link"/>
@@ -62,5 +58,5 @@
   </joint>
   <!-- Note the z-offset to raise the base off the ground, to avoid collision issues. Without this, there are vibrations and other artifacts from resolving the ground collision that result in significant error in the balanced object. -->
-  <joint name="base_to_y_joint" type="continuous">
+	<joint name="base_to_y_joint" type="continuous">
     <parent link="y_prismatic_link"/>
     <child link="base_link"/>
@@ -69,8 +65,8 @@
   </joint>
   <link name="base_link">
-    <inertial>
-      <mass value="0.01"/>
-      <inertia ixx="0.01" ixy="0" ixz="0" iyy="0.01" iyz="0" izz="0.01"/>
-      <origin rpy="0 0 0" xyz="0 0 0"/>
+	 <inertial>
+     <mass value="0.01"/>
+     <inertia ixx="0.01" ixy="0" ixz="0" iyy="0.01" iyz="0" izz="0.01"/>
+     <origin rpy="0 0 0" xyz="0 0 0"/>
     </inertial>
   </link>
@@ -88,5 +84,5 @@
       <!-- <origin xyz="0 0 0"/> -->
       <geometry>
-        <mesh filename="file:///home/adam/phd/code/mm/tray_balance/catkin_ws/src/tray_balance/tray_balance_assets/meshes/ridgeback/body.stl"/>
+        <mesh filename="file://$(find tray_balance_assets)/meshes/ridgeback/body.stl"/>
       </geometry>
       <material name="black"/>
@@ -124,5 +120,5 @@
       <origin rpy="0 0 3.14159265359" xyz="0 0 0"/>
       <geometry>
-        <mesh filename="file:///home/adam/phd/code/mm/tray_balance/catkin_ws/src/tray_balance/tray_balance_assets/meshes/ridgeback/side-cover.stl"/>
+        <mesh filename="file://$(find tray_balance_assets)/meshes/ridgeback/side-cover.stl"/>
       </geometry>
       <material name="yellow"/>
@@ -133,5 +129,5 @@
       <origin rpy="0 0 0" xyz="0 0 0"/>
       <geometry>
-        <mesh filename="file:///home/adam/phd/code/mm/tray_balance/catkin_ws/src/tray_balance/tray_balance_assets/meshes/ridgeback/side-cover.stl"/>
+        <mesh filename="file://$(find tray_balance_assets)/meshes/ridgeback/side-cover.stl"/>
       </geometry>
       <material name="yellow"/>
@@ -147,5 +143,5 @@
       <origin rpy="0 0 0" xyz="0 0 0"/>
       <geometry>
-        <mesh filename="file:///home/adam/phd/code/mm/tray_balance/catkin_ws/src/tray_balance/tray_balance_assets/meshes/ridgeback/end-cover.stl"/>
+        <mesh filename="file://$(find tray_balance_assets)/meshes/ridgeback/end-cover.stl"/>
       </geometry>
       <material name="black"/>
@@ -161,5 +157,5 @@
       <origin rpy="0 0 3.14159265359" xyz="0 0 0"/>
       <geometry>
-        <mesh filename="file:///home/adam/phd/code/mm/tray_balance/catkin_ws/src/tray_balance/tray_balance_assets/meshes/ridgeback/end-cover.stl"/>
+        <mesh filename="file://$(find tray_balance_assets)/meshes/ridgeback/end-cover.stl"/>
       </geometry>
       <material name="black"/>
@@ -180,5 +176,5 @@
       <origin rpy="0 0 0" xyz="0 0 0"/>
       <geometry>
-        <mesh filename="file:///home/adam/phd/code/mm/tray_balance/catkin_ws/src/tray_balance/tray_balance_assets/meshes/ridgeback/lights.stl"/>
+        <mesh filename="file://$(find tray_balance_assets)/meshes/ridgeback/lights.stl"/>
       </geometry>
       <material name="white"/>
@@ -189,5 +185,5 @@
       <origin rpy="0 0 3.14159265359" xyz="0 0 0"/>
       <geometry>
-        <mesh filename="file:///home/adam/phd/code/mm/tray_balance/catkin_ws/src/tray_balance/tray_balance_assets/meshes/ridgeback/lights.stl"/>
+        <mesh filename="file://$(find tray_balance_assets)/meshes/ridgeback/lights.stl"/>
       </geometry>
       <material name="red"/>
@@ -203,5 +199,5 @@
       <origin rpy="0 0 0" xyz="0 0 0"/>
       <geometry>
-        <mesh filename="file:///home/adam/phd/code/mm/tray_balance/catkin_ws/src/tray_balance/tray_balance_assets/meshes/ridgeback/top.stl"/>
+        <mesh filename="file://$(find tray_balance_assets)/meshes/ridgeback/top.stl"/>
       </geometry>
       <material name="black"/>
@@ -210,5 +206,5 @@
       <origin rpy="0 0 0" xyz="0 0 0"/>
       <geometry>
-        <mesh filename="file:///home/adam/phd/code/mm/tray_balance/catkin_ws/src/tray_balance/tray_balance_assets/meshes/ridgeback/top.stl"/>
+        <mesh filename="file://$(find tray_balance_assets)/meshes/ridgeback/top.stl"/>
       </geometry>
     </collision>
@@ -223,5 +219,5 @@
       <origin rpy="0 1.57079632679 0" xyz="0 0 0"/>
       <geometry>
-        <mesh filename="file:///home/adam/phd/code/mm/tray_balance/catkin_ws/src/tray_balance/tray_balance_assets/meshes/ridgeback/axle.stl"/>
+        <mesh filename="file://$(find tray_balance_assets)/meshes/ridgeback/axle.stl"/>
       </geometry>
       <material name="black"/>
@@ -249,5 +245,5 @@
     <visual>
       <geometry>
-        <mesh filename="file:///home/adam/phd/code/mm/tray_balance/catkin_ws/src/tray_balance/tray_balance_assets/meshes/tor11_mech.dae"/>
+        <mesh filename="file://$(find tray_balance_assets)/meshes/tor11_mech.dae"/>
       </geometry>
     </visual>
@@ -271,5 +267,5 @@
     <visual>
       <geometry>
-        <mesh filename="file:///home/adam/phd/code/mm/tray_balance/catkin_ws/src/tray_balance/tray_balance_assets/meshes/ur10/visual/base.dae"/>
+        <mesh filename="file://$(find tray_balance_assets)/meshes/ur10/visual/base.dae"/>
       </geometry>
       <material name="LightGrey">
@@ -279,5 +275,5 @@
     <collision>
       <geometry>
-        <mesh filename="file:///home/adam/phd/code/mm/tray_balance/catkin_ws/src/tray_balance/tray_balance_assets/meshes/ur10/collision/base.stl"/>
+        <mesh filename="file://$(find tray_balance_assets)/meshes/ur10/collision/base.stl"/>
       </geometry>
     </collision>
@@ -299,5 +295,5 @@
     <visual>
       <geometry>
-        <mesh filename="file:///home/adam/phd/code/mm/tray_balance/catkin_ws/src/tray_balance/tray_balance_assets/meshes/ur10/visual/shoulder.dae"/>
+        <mesh filename="file://$(find tray_balance_assets)/meshes/ur10/visual/shoulder.dae"/>
       </geometry>
       <material name="LightGrey">
@@ -307,5 +303,5 @@
     <collision>
       <geometry>
-        <mesh filename="file:///home/adam/phd/code/mm/tray_balance/catkin_ws/src/tray_balance/tray_balance_assets/meshes/ur10/collision/shoulder.stl"/>
+        <mesh filename="file://$(find tray_balance_assets)/meshes/ur10/collision/shoulder.stl"/>
       </geometry>
     </collision>
@@ -327,5 +323,5 @@
     <visual>
       <geometry>
-        <mesh filename="file:///home/adam/phd/code/mm/tray_balance/catkin_ws/src/tray_balance/tray_balance_assets/meshes/ur10/visual/upperarm.dae"/>
+        <mesh filename="file://$(find tray_balance_assets)/meshes/ur10/visual/upperarm.dae"/>
       </geometry>
       <material name="LightGrey">
@@ -335,5 +331,5 @@
     <collision>
       <geometry>
-        <mesh filename="file:///home/adam/phd/code/mm/tray_balance/catkin_ws/src/tray_balance/tray_balance_assets/meshes/ur10/collision/upperarm.stl"/>
+        <mesh filename="file://$(find tray_balance_assets)/meshes/ur10/collision/upperarm.stl"/>
       </geometry>
     </collision>
@@ -355,5 +351,5 @@
     <visual>
       <geometry>
-        <mesh filename="file:///home/adam/phd/code/mm/tray_balance/catkin_ws/src/tray_balance/tray_balance_assets/meshes/ur10/visual/forearm.dae"/>
+        <mesh filename="file://$(find tray_balance_assets)/meshes/ur10/visual/forearm.dae"/>
       </geometry>
       <material name="LightGrey">
@@ -363,5 +359,5 @@
     <collision>
       <geometry>
-        <mesh filename="file:///home/adam/phd/code/mm/tray_balance/catkin_ws/src/tray_balance/tray_balance_assets/meshes/ur10/collision/forearm.stl"/>
+        <mesh filename="file://$(find tray_balance_assets)/meshes/ur10/collision/forearm.stl"/>
       </geometry>
     </collision>
@@ -383,5 +379,5 @@
     <visual>
       <geometry>
-        <mesh filename="file:///home/adam/phd/code/mm/tray_balance/catkin_ws/src/tray_balance/tray_balance_assets/meshes/ur10/visual/wrist1.dae"/>
+        <mesh filename="file://$(find tray_balance_assets)/meshes/ur10/visual/wrist1.dae"/>
       </geometry>
       <material name="LightGrey">
@@ -391,5 +387,5 @@
     <collision>
       <geometry>
-        <mesh filename="file:///home/adam/phd/code/mm/tray_balance/catkin_ws/src/tray_balance/tray_balance_assets/meshes/ur10/collision/wrist1.stl"/>
+        <mesh filename="file://$(find tray_balance_assets)/meshes/ur10/collision/wrist1.stl"/>
       </geometry>
     </collision>
@@ -411,5 +407,5 @@
     <visual>
       <geometry>
-        <mesh filename="file:///home/adam/phd/code/mm/tray_balance/catkin_ws/src/tray_balance/tray_balance_assets/meshes/ur10/visual/wrist2.dae"/>
+        <mesh filename="file://$(find tray_balance_assets)/meshes/ur10/visual/wrist2.dae"/>
       </geometry>
       <material name="LightGrey">
@@ -419,5 +415,5 @@
     <collision>
       <geometry>
-        <mesh filename="file:///home/adam/phd/code/mm/tray_balance/catkin_ws/src/tray_balance/tray_balance_assets/meshes/ur10/collision/wrist2.stl"/>
+        <mesh filename="file://$(find tray_balance_assets)/meshes/ur10/collision/wrist2.stl"/>
       </geometry>
     </collision>
@@ -439,5 +435,5 @@
     <visual>
       <geometry>
-        <mesh filename="file:///home/adam/phd/code/mm/tray_balance/catkin_ws/src/tray_balance/tray_balance_assets/meshes/ur10/visual/wrist3.dae"/>
+        <mesh filename="file://$(find tray_balance_assets)/meshes/ur10/visual/wrist3.dae"/>
       </geometry>
       <material name="LightGrey">
@@ -447,5 +443,5 @@
     <collision>
       <geometry>
-        <mesh filename="file:///home/adam/phd/code/mm/tray_balance/catkin_ws/src/tray_balance/tray_balance_assets/meshes/ur10/collision/wrist3.stl"/>
+        <mesh filename="file://$(find tray_balance_assets)/meshes/ur10/collision/wrist3.stl"/>
       </geometry>
     </collision>
@@ -514,10 +510,10 @@
     <origin rpy="0.0 0.0 1.57079632679" xyz="0.01 -0.27 0.375"/>
   </joint>
-  <!-- s = 0.3 -->
-  <!-- h = 0.08660254037844387 -->
-  <!-- r = 0.17320508075688773 -->
-  <!-- s = 0.2 -->
-  <!-- h = 0.0577 -->
-  <!-- r = 0.1155 -->
+<!-- s = 0.3 -->
+<!-- h = 0.08660254037844387 -->
+<!-- r = 0.17320508075688773 -->
+<!-- s = 0.2 -->
+<!-- h = 0.0577 -->
+<!-- r = 0.1155 -->
   <!-- Custom tool for tray balancing -->
   <!-- When oriented forward, the frame has: z forward, x down, y left -->

Commit message: Fix issues with original constraints and recompileLibraries.
* Original constraints were no longer working with Goal 3 and Stack 3.
  This was fixed by adding a small margin to the ZMP constraint.
* recompileLibraries is now set to false for all calls to `.clone()` on
  custom Constraint objects, so that each AD library is compiled at most
  once per run.

File: tray_balance_assets/urdf/mm_ocs2.urdf (robot description, URDF)
Before this commit: robot Thing, 39 links, 38 joints
Links:
- link arch_link: geometry visual mesh filename=file:///home/adam/phd/code/projects/tray_balance/catkin_ws/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
- link axle_link: geometry visual mesh filename=file:///home/adam/phd/code/projects/tray_balance/catkin_ws/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
- link chassis_link: geometry collision box size=1.0 0.8 0.3; visual mesh filename=file:///home/adam/phd/code/projects/tray_balance/catkin_ws/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
- link front_cover_link: geometry visual mesh filename=file:///home/adam/phd/code/projects/tray_balance/catkin_ws/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
- link front_left_wheel_link: geometry collision cylinder length=0.079 radius=0.0759; visual mesh filename=file:///home/adam/phd/code/projects/tray_balance/catkin_ws/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
- link front_lights_link: geometry visual mesh filename=file:///home/adam/phd/code/projects/tray_balance/catkin_ws/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
- link front_right_wheel_link: geometry collision cylinder length=0.079 radius=0.0759; visual mesh filename=file:///home/adam/phd/code/projects/tray_balance/catkin_ws/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
- link front_rocker_link: geometry visual mesh filename=file:///home/adam/phd/code/projects/tray_balance/catkin_ws/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
- link left_side_cover_link: geometry visual mesh filename=file:///home/adam/phd/code/projects/tray_balance/catkin_ws/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
- link rear_cover_link: geometry visual mesh filename=file:///home/adam/phd/code/projects/tray_balance/catkin_ws/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
- link rear_left_wheel_link: geometry collision cylinder length=0.079 radius=0.0759; visual mesh filename=file:///home/adam/phd/code/projects/tray_balance/catkin_ws/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
- link rear_lights_link: geometry visual mesh filename=file:///home/adam/phd/code/projects/tray_balance/catkin_ws/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
- link rear_right_wheel_link: geometry collision cylinder length=0.079 radius=0.0759; visual mesh filename=file:///home/adam/phd/code/projects/tray_balance/catkin_ws/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
- link rear_rocker_link: geometry visual mesh filename=file:///home/adam/phd/code/projects/tray_balance/catkin_ws/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
- link right_side_cover_link: geometry visual mesh filename=file:///home/adam/phd/code/projects/tray_balance/catkin_ws/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
- link top_link: geometry collision mesh filename=file:///home/adam/phd/code/projects/tray_balance/catkin_ws/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; visual mesh filename=file:///home/adam/phd/code/projects/tray_balance/catkin_ws/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
- link ur10_arm_base_link: geometry collision mesh filename=file:///home/adam/phd/code/projects/tray_balance/catkin_ws/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; visual mesh filename=file:///home/adam/phd/code/projects/tray_balance/catkin_ws/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
- link ur10_arm_forearm_link: geometry collision mesh filename=file:///home/adam/phd/code/projects/tray_balance/catkin_ws/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; visual mesh filename=file:///home/adam/phd/code/projects/tray_balance/catkin_ws/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
- link ur10_arm_shoulder_link: geometry collision mesh filename=file:///home/adam/phd/code/projects/tray_balance/catkin_ws/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; visual mesh filename=file:///home/adam/phd/code/projects/tray_balance/catkin_ws/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
- link ur10_arm_upper_arm_link: geometry collision mesh filename=file:///home/adam/phd/code/projects/tray_balance/catkin_ws/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; visual mesh filename=file:///home/adam/phd/code/projects/tray_balance/catkin_ws/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
- link ur10_arm_wrist_1_link: geometry collision mesh filename=file:///home/adam/phd/code/projects/tray_balance/catkin_ws/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; visual mesh filename=file:///home/adam/phd/code/projects/tray_balance/catkin_ws/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
- link ur10_arm_wrist_2_link: geometry collision mesh filename=file:///home/adam/phd/code/projects/tray_balance/catkin_ws/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; visual mesh filename=file:///home/adam/phd/code/projects/tray_balance/catkin_ws/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
- link ur10_arm_wrist_3_link: geometry collision mesh filename=file:///home/adam/phd/code/projects/tray_balance/catkin_ws/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; visual mesh filename=file:///home/adam/phd/code/projects/tray_balance/catkin_ws/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

File: tray_balance_assets/urdf/mm_pyb.urdf (robot description, URDF)
Before this commit: robot Thing, 27 links, 26 joints
Links:
- link arch_link: geometry visual mesh filename=file:///home/adam/phd/code/projects/tray_balance/catkin_ws/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
- link axle_link: geometry visual mesh filename=file:///home/adam/phd/code/projects/tray_balance/catkin_ws/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
- link chassis_link: geometry collision box size=1.0 0.8 0.3; visual mesh filename=file:///home/adam/phd/code/projects/tray_balance/catkin_ws/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
- link front_cover_link: geometry visual mesh filename=file:///home/adam/phd/code/projects/tray_balance/catkin_ws/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
- link front_lights_link: geometry visual mesh filename=file:///home/adam/phd/code/projects/tray_balance/catkin_ws/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
- link left_side_cover_link: geometry visual mesh filename=file:///home/adam/phd/code/projects/tray_balance/catkin_ws/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
- link rear_cover_link: geometry visual mesh filename=file:///home/adam/phd/code/projects/tray_balance/catkin_ws/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
- link rear_lights_link: geometry visual mesh filename=file:///home/adam/phd/code/projects/tray_balance/catkin_ws/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
- link right_side_cover_link: geometry visual mesh filename=file:///home/adam/phd/code/projects/tray_balance/catkin_ws/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
- link top_link: geometry collision mesh filename=file:///home/adam/phd/code/projects/tray_balance/catkin_ws/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; visual mesh filename=file:///home/adam/phd/code/projects/tray_balance/catkin_ws/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
- link ur10_arm_base_link: geometry collision mesh filename=file:///home/adam/phd/code/projects/tray_balance/catkin_ws/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; visual mesh filename=file:///home/adam/phd/code/projects/tray_balance/catkin_ws/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
- link ur10_arm_forearm_link: geometry collision mesh filename=file:///home/adam/phd/code/projects/tray_balance/catkin_ws/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; visual mesh filename=file:///home/adam/phd/code/projects/tray_balance/catkin_ws/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
- link ur10_arm_shoulder_link: geometry collision mesh filename=file:///home/adam/phd/code/projects/tray_balance/catkin_ws/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; visual mesh filename=file:///home/adam/phd/code/projects/tray_balance/catkin_ws/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
- link ur10_arm_upper_arm_link: geometry collision mesh filename=file:///home/adam/phd/code/projects/tray_balance/catkin_ws/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; visual mesh filename=file:///home/adam/phd/code/projects/tray_balance/catkin_ws/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
- link ur10_arm_wrist_1_link: geometry collision mesh filename=file:///home/adam/phd/code/projects/tray_balance/catkin_ws/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; visual mesh filename=file:///home/adam/phd/code/projects/tray_balance/catkin_ws/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
- link ur10_arm_wrist_2_link: geometry collision mesh filename=file:///home/adam/phd/code/projects/tray_balance/catkin_ws/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; visual mesh filename=file:///home/adam/phd/code/projects/tray_balance/catkin_ws/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
- link ur10_arm_wrist_3_link: geometry collision mesh filename=file:///home/adam/phd/code/projects/tray_balance/catkin_ws/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; visual mesh filename=file:///home/adam/phd/code/projects/tray_balance/catkin_ws/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

File: tray_balance_assets/urdf/mm_pyb.urdf.xacro (robot description, xacro)
@@ -568,32 +568,33 @@
     </inertial>
   </link>
-  <link name="robust_sphere1_link">
-    <visual>
-      <origin rpy="0 0 0" xyz="0 0 0.1"/>
-      <geometry>
-        <sphere radius="0.12"/>
-      </geometry>
-      <material name="seethrough"/>
-    </visual>
-  </link>
-  <joint name="robust_sphere1_joint" type="fixed">
-    <origin rpy="0 0 0" xyz="0 0 0"/>
-    <parent link="thing_tool"/>
-    <child link="robust_sphere1_link"/>
-  </joint>
-  <link name="robust_sphere2_link">
-    <visual>
-      <origin rpy="0 0 0" xyz="0 0 0.3"/>
-      <geometry>
-        <sphere radius="0.12"/>
-      </geometry>
-      <material name="seethrough"/>
-    </visual>
-  </link>
-  <joint name="robust_sphere2_joint" type="fixed">
-    <origin rpy="0 0 0" xyz="0 0 0"/>
-    <parent link="thing_tool"/>
-    <child link="robust_sphere2_link"/>
-  </joint>
+  <!-- <link name="robust_sphere1_link"> -->
+  <!--   <visual> -->
+  <!--     <origin rpy="0 0 0" xyz="0 0 0.1"/> -->
+  <!--     <geometry> -->
+  <!--       <sphere radius="0.12"/> -->
+  <!--     </geometry> -->
+  <!--     <material name="seethrough"/> -->
+  <!--   </visual> -->
+  <!-- </link> -->
+  <!-- <joint name="robust_sphere1_joint" type="fixed"> -->
+  <!--   <origin rpy="0 0 0" xyz="0 0 0"/> -->
+  <!--   <parent link="thing_tool"/> -->
+  <!--   <child link="robust_sphere1_link"/> -->
+  <!-- </joint> -->
+  <!--  -->
+  <!-- <link name="robust_sphere2_link"> -->
+  <!--   <visual> -->
+  <!--     <origin rpy="0 0 0" xyz="0 0 0.3"/> -->
+  <!--     <geometry> -->
+  <!--       <sphere radius="0.12"/> -->
+  <!--     </geometry> -->
+  <!--     <material name="seethrough"/> -->
+  <!--   </visual> -->
+  <!-- </link> -->
+  <!-- <joint name="robust_sphere2_joint" type="fixed"> -->
+  <!--   <origin rpy="0 0 0" xyz="0 0 0"/> -->
+  <!--   <parent link="thing_tool"/> -->
+  <!--   <child link="robust_sphere2_link"/> -->
+  <!-- </joint> -->
   <!-- Collision element to protect the balanced objects -->
   <!-- <link name="balanced_object_collision_link"> -->

Commit message: Fix URDFs and config now that arm has been rotated w.r.t. base.

File: tray_balance_assets/urdf/mm_ocs2.urdf (robot description, URDF)
Before this commit: robot Thing, 39 links, 38 joints
Joints:
- joint ur10_arm_base: origin xyz=0.01 -0.27 0.375 rpy=0.0 0.0 1.57079632679 -> xyz=0.01 -0.27 0.375 rpy=0.0 0.0 0.0

File: tray_balance_assets/urdf/mm_ocs2.urdf.xacro (robot description, xacro)
@@ -602,5 +602,5 @@
     <parent link="arch_link"/>
     <child link="ur10_arm_base_link"/>
-    <origin rpy="0.0 0.0 1.57079632679" xyz="0.01 -0.27 0.375"/>
+    <origin rpy="0.0 0.0 0.0" xyz="0.01 -0.27 0.375"/>
   </joint>
   <joint name="tool0_tcp_fixed_joint" type="fixed">

File: tray_balance_assets/urdf/mm_pyb.urdf (robot description, URDF)
Before this commit: robot Thing, 27 links, 26 joints
Joints:
- joint ur10_arm_base: origin xyz=0.01 -0.27 0.375 rpy=0.0 0.0 1.57079632679 -> xyz=0.01 -0.27 0.375 rpy=0.0 0.0 0.0

File: tray_balance_assets/urdf/mm_pyb.urdf.xacro (robot description, xacro)
@@ -511,5 +511,6 @@
     <parent link="arch_link"/>
     <child link="ur10_arm_base_link"/>
-    <origin rpy="0.0 0.0 1.57079632679" xyz="0.01 -0.27 0.375"/>
+    <!-- <origin rpy="0.0 0.0 1.57079632679" xyz="0.01 -0.27 0.375"/> -->
+    <origin rpy="0.0 0.0 0.0" xyz="0.01 -0.27 0.375"/>
   </joint>
 <!-- s = 0.3 -->
