Commit message: Mess about with tray end effector. OCS2 segfault.

File: tray_balance_assets/franka_panda/panda.urdf (robot description, URDF)
Before this commit: robot panda, 13 links, 12 joints
Links:
- removed link panda_grasptarget
- added link tray_link; collision cylinder length=0.02 radius=0.15; visual cylinder length=0.02 radius=0.15
Joints:
- removed joint panda_grasptarget_hand
- added joint tray_joint: type fixed, parent panda_hand, child tray_link, origin xyz=0.0 0.0 0.25 rpy=1.5708 0.0 0.0

Commit message: Single object balance with Panda arm works.

File: tray_balance_assets/franka_panda/panda.urdf (robot description, URDF)
Before this commit: robot panda, 13 links, 12 joints
Joints:
- joint panda_finger_joint1: type prismatic -> fixed
- joint panda_finger_joint2: type prismatic -> fixed
- joint tray_joint: origin xyz=0.0 0.0 0.25 rpy=1.5708 0.0 0.0 -> xyz=0.0 0.0 0.25 rpy=-1.5708 0.0 0.0

Commit message: Reconfigure Panda initial pose to be somewhat less awkward.

File: tray_balance_assets/franka_panda/panda.urdf (robot description, URDF)
Before this commit: robot panda, 13 links, 12 joints
Joints:
- joint tray_joint: origin xyz=0.0 0.0 0.25 rpy=-1.5708 0.0 0.0 -> xyz=0.0 0.0 0.25 rpy=-1.5708 -1.5708 0.0
