Commit message: Add simple script to test velocity joint control of Panda.

File: tray_balance_assets/franka_panda/panda.urdf.xacro (robot description, xacro)
@@ -1,13 +1,9 @@
 <?xml version="1.0" ?>
-<!-- =================================================================================== -->
-<!-- |    This document was autogenerated by xacro from panda.urdf.xacro               | -->
-<!-- |    EDITING THIS FILE BY HAND IS NOT RECOMMENDED                                 | -->
-<!-- =================================================================================== -->
-<robot name="panda">
+<robot name="panda" xmlns:xacro="http://www.ros.org/wiki/xacro">
   <link name="panda_link0">
-    <inertial>
+  	<inertial>
       <origin rpy="0 0 0" xyz="0 0 0.05"/>
-      <mass value="2.9"/>
-      <inertia ixx="0.1" ixy="0" ixz="0" iyy="0.1" iyz="0" izz="0.1"/>
+       <mass value="2.9"/>
+       <inertia ixx="0.1" ixy="0" ixz="0" iyy="0.1" iyz="0" izz="0.1"/>
     </inertial>
     <visual>
@@ -16,6 +12,6 @@
       </geometry>
       <material name="panda_white">
-        <color rgba="1. 1. 1. 1."/>
-      </material>
+    		<color rgba="1. 1. 1. 1."/>
+  		</material>
     </visual>
     <collision>
@@ -27,8 +23,8 @@
   </link>
   <link name="panda_link1">
-    <inertial>
+  	<inertial>
       <origin rpy="0 0 0" xyz="0 -0.04 -0.05"/>
-      <mass value="2.7"/>
-      <inertia ixx="0.1" ixy="0" ixz="0" iyy="0.1" iyz="0" izz="0.1"/>
+       <mass value="2.7"/>
+       <inertia ixx="0.1" ixy="0" ixz="0" iyy="0.1" iyz="0" izz="0.1"/>
     </inertial>
     <visual>
@@ -54,8 +50,8 @@
   </joint>
   <link name="panda_link2">
-    <inertial>
+  	<inertial>
       <origin rpy="0 0 0" xyz="0 -0.04 0.06"/>
-      <mass value="2.73"/>
-      <inertia ixx="0.1" ixy="0" ixz="0" iyy="0.1" iyz="0" izz="0.1"/>
+       <mass value="2.73"/>
+       <inertia ixx="0.1" ixy="0" ixz="0" iyy="0.1" iyz="0" izz="0.1"/>
     </inertial>
     <visual>
@@ -81,8 +77,8 @@
   </joint>
   <link name="panda_link3">
-    <inertial>
+	  <inertial>
       <origin rpy="0 0 0" xyz="0.01 0.01 -0.05"/>
-      <mass value="2.04"/>
-      <inertia ixx="0.1" ixy="0" ixz="0" iyy="0.1" iyz="0" izz="0.1"/>
+       <mass value="2.04"/>
+       <inertia ixx="0.1" ixy="0" ixz="0" iyy="0.1" iyz="0" izz="0.1"/>
     </inertial>
     <visual>
@@ -91,6 +87,6 @@
       </geometry>
       <material name="panda_red">
-        <color rgba="1. 1. 1. 1."/>
-      </material>
+    		<color rgba="1. 1. 1. 1."/>
+  		</material>
     </visual>
     <collision>
@@ -109,8 +105,8 @@
   </joint>
   <link name="panda_link4">
-    <inertial>
+  	<inertial>
       <origin rpy="0 0 0" xyz="-0.03 0.03 0.02"/>
-      <mass value="2.08"/>
-      <inertia ixx="0.1" ixy="0" ixz="0" iyy="0.1" iyz="0" izz="0.1"/>
+       <mass value="2.08"/>
+       <inertia ixx="0.1" ixy="0" ixz="0" iyy="0.1" iyz="0" izz="0.1"/>
     </inertial>
     <visual>
@@ -136,8 +132,8 @@
   </joint>
   <link name="panda_link5">
-    <inertial>
+  	<inertial>
       <origin rpy="0 0 0" xyz="0 0.04 -0.12"/>
-      <mass value="3"/>
-      <inertia ixx="0.1" ixy="0" ixz="0" iyy="0.1" iyz="0" izz="0.1"/>
+       <mass value="3"/>
+       <inertia ixx="0.1" ixy="0" ixz="0" iyy="0.1" iyz="0" izz="0.1"/>
     </inertial>
     <visual>
@@ -163,8 +159,8 @@
   </joint>
   <link name="panda_link6">
-    <inertial>
+  	<inertial>
       <origin rpy="0 0 0" xyz="0.04 0 0"/>
-      <mass value="1.3"/>
-      <inertia ixx="0.1" ixy="0" ixz="0" iyy="0.1" iyz="0" izz="0.1"/>
+       <mass value="1.3"/>
+       <inertia ixx="0.1" ixy="0" ixz="0" iyy="0.1" iyz="0" izz="0.1"/>
     </inertial>
     <visual>
@@ -190,8 +186,8 @@
   </joint>
   <link name="panda_link7">
-    <inertial>
+  	<inertial>
       <origin rpy="0 0 0" xyz="0 0 0.08"/>
-      <mass value=".2"/>
-      <inertia ixx="0.1" ixy="0" ixz="0" iyy="0.1" iyz="0" izz="0.1"/>
+       <mass value=".2"/>
+       <inertia ixx="0.1" ixy="0" ixz="0" iyy="0.1" iyz="0" izz="0.1"/>
     </inertial>
     <visual>
@@ -217,8 +213,8 @@
   </joint>
   <link name="panda_link8">
-    <inertial>
+  	 <inertial>
       <origin rpy="0 0 0" xyz="0 0 0"/>
-      <mass value="0.0"/>
-      <inertia ixx="0.1" ixy="0" ixz="0" iyy="0.1" iyz="0" izz="0.1"/>
+       <mass value="0.0"/>
+       <inertia ixx="0.1" ixy="0" ixz="0" iyy="0.1" iyz="0" izz="0.1"/>
     </inertial>
   </link>
@@ -235,8 +231,8 @@
   </joint>
   <link name="panda_hand">
-    <inertial>
+  	<inertial>
       <origin rpy="0 0 0" xyz="0 0 0.04"/>
-      <mass value=".81"/>
-      <inertia ixx="0.1" ixy="0" ixz="0" iyy="0.1" iyz="0" izz="0.1"/>
+       <mass value=".81"/>
+       <inertia ixx="0.1" ixy="0" ixz="0" iyy="0.1" iyz="0" izz="0.1"/>
     </inertial>
     <visual>
@@ -254,5 +250,5 @@
   </link>
   <link name="panda_leftfinger">
-    <contact>
+       <contact>
       <friction_anchor/>
       <stiffness value="30000.0"/>
@@ -261,8 +257,8 @@
       <lateral_friction value="1.0"/>
     </contact>
-    <inertial>
+  	<inertial>
       <origin rpy="0 0 0" xyz="0 0.01 0.02"/>
-      <mass value="0.1"/>
-      <inertia ixx="0.1" ixy="0" ixz="0" iyy="0.1" iyz="0" izz="0.1"/>
+       <mass value="0.1"/>
+       <inertia ixx="0.1" ixy="0" ixz="0" iyy="0.1" iyz="0" izz="0.1"/>
     </inertial>
     <visual>
@@ -280,5 +276,5 @@
   </link>
   <link name="panda_rightfinger">
-    <contact>
+        <contact>
       <friction_anchor/>
       <stiffness value="30000.0"/>
@@ -287,8 +283,8 @@
       <lateral_friction value="1.0"/>
     </contact>
-    <inertial>
+  	<inertial>
       <origin rpy="0 0 0" xyz="0 -0.01 0.02"/>
-      <mass value="0.1"/>
-      <inertia ixx="0.1" ixy="0" ixz="0" iyy="0.1" iyz="0" izz="0.1"/>
+       <mass value="0.1"/>
+       <inertia ixx="0.1" ixy="0" ixz="0" iyy="0.1" iyz="0" izz="0.1"/>
     </inertial>
     <visual>

File: tray_balance_assets/franka_panda/panda_tray.urdf (robot description, URDF)
Before this commit: robot panda, 12 links, 11 joints
Links:
- added link tray_link; collision cylinder length=0.02 radius=0.15; visual cylinder length=0.02 radius=0.15
Joints:
- added joint tray_joint: type fixed, parent panda_hand, child tray_link, origin xyz=0.0 0.0 0.25 rpy=-1.5708 -1.5708 0.0
