Commit message: Fix robot home position and URDF to actually match reality.

File: tray_balance_assets/thing/xacro/ocs2/mm_ocs2.urdf.xacro (robot description, xacro)
@@ -602,5 +602,5 @@
     <parent link="arch_link"/>
     <child link="ur10_arm_base_link"/>
-    <origin rpy="0.0 0.0 0.0" xyz="0.01 -0.27 0.375"/>
+    <origin rpy="0.0 0.0 3.14159265359" xyz="0.01 -0.27 0.375"/>
   </joint>
 </robot>

File: tray_balance_assets/thing/xacro/pyb/mm_pyb.urdf.xacro (robot description, xacro)
@@ -506,6 +506,5 @@
     <parent link="arch_link"/>
     <child link="ur10_arm_base_link"/>
-    <!-- <origin rpy="0.0 0.0 1.57079632679" xyz="0.01 -0.27 0.375"/> -->
-    <origin rpy="0.0 0.0 0.0" xyz="0.01 -0.27 0.375"/>
+    <origin rpy="0.0 0.0 3.14159265359" xyz="0.01 -0.27 0.375"/>
   </joint>
 </robot>

Commit message: Add 15-deg offset to account for gripper misalignment.

File: tray_balance_assets/thing/xacro/ocs2/mm_ocs2.urdf.xacro (robot description, xacro)
@@ -564,38 +564,26 @@
     </collision>
   </link>
-  <!-- ROS base_link to UR 'Base' Coordinates transform -->
-  <link name="ur10_arm_base"/>
-  <joint name="ur10_arm_base_link-base_fixed_joint" type="fixed">
-    <!-- NOTE: this rotation is only needed as long as base_link itself is
-                 not corrected wrt the real robot (ie: rotated over 180
-                 degrees)
-      -->
-    <origin rpy="0 0 -3.14159265359" xyz="0 0 0"/>
-    <parent link="ur10_arm_base_link"/>
-    <child link="ur10_arm_base"/>
-  </joint>
+  <!-- Frame coincident with all-zeros TCP on UR controller -->
+  <link name="ur10_arm_tool0">
+    <visual>
+      <!-- start halfway along the cylinder -->
+      <origin rpy="0 0 0" xyz="0 0 0.145"/>
+      <geometry>
+        <cylinder length="0.290" radius="0.01"/>
+      </geometry>
+      <material name="black"/>
+    </visual>
+    <collision>
+      <origin rpy="0 0 0" xyz="0 0 0.145"/>
+      <geometry>
+        <cylinder length="0.290" radius="0.01"/>
+      </geometry>
+    </collision>
+  </link>
   <joint name="ur10_arm_wrist_3_link-tool0_fixed_joint" type="fixed">
-    <origin rpy="-1.57079632679 0 0" xyz="0 0.0922 0"/>
+    <origin rpy="-1.57079632679 0.2617993877991494 0" xyz="0 0.0922 0"/>
     <parent link="ur10_arm_wrist_3_link"/>
     <child link="ur10_arm_tool0"/>
   </joint>
-  <!-- Frame coincident with all-zeros TCP on UR controller -->
-  <!-- <link name="ur10_arm_tool0"/> -->
-  <link name="ur10_arm_tool0">
-    <visual>
-      <!-- start halfway along the cylinder -->
-      <origin rpy="0 0 0" xyz="0 0 0.145"/>
-      <geometry>
-        <cylinder length="0.290" radius="0.01"/>
-      </geometry>
-      <material name="black"/>
-    </visual>
-    <collision>
-      <origin rpy="0 0 0" xyz="0 0 0.145"/>
-      <geometry>
-        <cylinder length="0.290" radius="0.01"/>
-      </geometry>
-    </collision>
-  </link>
   <!-- Join arm -->
   <joint name="ur10_arm_base" type="fixed">

File: tray_balance_assets/thing/xacro/pyb/mm_pyb.urdf.xacro (robot description, xacro)
@@ -468,38 +468,27 @@
     </collision>
   </link>
-  <!-- ROS base_link to UR 'Base' Coordinates transform -->
-  <link name="ur10_arm_base"/>
-  <joint name="ur10_arm_base_link-base_fixed_joint" type="fixed">
-    <!-- NOTE: this rotation is only needed as long as base_link itself is
-                 not corrected wrt the real robot (ie: rotated over 180
-                 degrees)
-      -->
-    <origin rpy="0 0 -3.14159265359" xyz="0 0 0"/>
-    <parent link="ur10_arm_base_link"/>
-    <child link="ur10_arm_base"/>
-  </joint>
+  <!-- Frame coincident with all-zeros TCP on UR controller -->
+  <link name="ur10_arm_tool0">
+    <visual>
+      <!-- start halfway along the cylinder -->
+      <origin rpy="0 0 0" xyz="0 0 0.145"/>
+      <geometry>
+        <cylinder length="0.290" radius="0.01"/>
+      </geometry>
+      <material name="black"/>
+    </visual>
+    <collision>
+      <origin rpy="0 0 0" xyz="0 0 0.145"/>
+      <geometry>
+        <cylinder length="0.290" radius="0.01"/>
+      </geometry>
+    </collision>
+  </link>
   <joint name="ur10_arm_wrist_3_link-tool0_fixed_joint" type="fixed">
-    <origin rpy="-1.57079632679 0 0" xyz="0 0.0922 0"/>
+    <!-- The 15-degree offset about the y-axis is to account for the fact that the gripper is actually mounted at this offset. -->
+    <origin rpy="-1.57079632679 0.2617993877991494 0" xyz="0 0.0922 0"/>
     <parent link="ur10_arm_wrist_3_link"/>
     <child link="ur10_arm_tool0"/>
   </joint>
-  <!-- Frame coincident with all-zeros TCP on UR controller -->
-  <!-- <link name="ur10_arm_tool0"/> -->
-  <link name="ur10_arm_tool0">
-    <visual>
-      <!-- start halfway along the cylinder -->
-      <origin rpy="0 0 0" xyz="0 0 0.145"/>
-      <geometry>
-        <cylinder length="0.290" radius="0.01"/>
-      </geometry>
-      <material name="black"/>
-    </visual>
-    <collision>
-      <origin rpy="0 0 0" xyz="0 0 0.145"/>
-      <geometry>
-        <cylinder length="0.290" radius="0.01"/>
-      </geometry>
-    </collision>
-  </link>
   <!-- Join arm -->
   <joint name="ur10_arm_base" type="fixed">
