Commit message: Load UR10 arm from external xacro packages.

File: upright_assets/thing/xacro/end_effector_tray.urdf.xacro (robot description, xacro)
@@ -1,7 +1,7 @@
 <?xml version="1.0" encoding="utf-8"?>
 <robot name="end_effector_tray">
-  <joint name="tool0_tcp_fixed_joint" type="fixed">
+  <joint name="gripper_tool_joint" type="fixed">
     <origin rpy="0 -1.5708 3.14159" xyz="0.0 0.0 0.25"/>
-    <parent link="ur10_arm_tool0"/>
+    <parent link="gripper"/>
     <child link="thing_tool"/>
   </joint>

File: upright_assets/thing/xacro/ocs2/mm_ocs2.urdf.xacro (robot description, xacro)
@@ -1,4 +1,4 @@
 <?xml version="1.0" encoding="utf-8"?>
-<robot name="Thing">
+<robot name="Thing" xmlns:xacro="http://wiki.ros.org/xacro">
   <material name="dark_grey">
     <color rgba="0.2 0.2 0.2 1.0"/>
@@ -358,233 +358,12 @@
     <child link="arch_link"/>
   </joint>
-  <!--
-  Author: Kelsey Hawkins
-  Contributers: Jimmy Da Silva, Ajit Krisshna N L, Muhammad Asif Rana
--->
-  <!-- measured from model -->
-  <link name="ur10_arm_base_link">
-    <visual>
-      <geometry>
-        <mesh filename="file://$(find upright_assets)/thing/meshes/ur10/visual/base.dae"/>
-      </geometry>
-      <material name="LightGrey">
-        <color rgba="0.7 0.7 0.7 1.0"/>
-      </material>
-    </visual>
-    <collision>
-      <geometry>
-        <mesh filename="file://$(find upright_assets)/thing/meshes/ur10/collision/base.stl"/>
-      </geometry>
-    </collision>
-    <inertial>
-      <mass value="4.0"/>
-      <origin rpy="0 0 0" xyz="0.0 0.0 0.0"/>
-      <inertia ixx="0.0061063308908" ixy="0.0" ixz="0.0" iyy="0.0061063308908" iyz="0.0" izz="0.01125"/>
-    </inertial>
-  </link>
-  <joint name="ur10_arm_shoulder_pan_joint" type="revolute">
-    <parent link="ur10_arm_base_link"/>
-    <child link="ur10_arm_shoulder_link"/>
-    <origin rpy="0.0 0.0 0.0" xyz="0.0 0.0 0.1273"/>
-    <axis xyz="0 0 1"/>
-    <limit effort="330.0" lower="-6.28318530718" upper="6.28318530718" velocity="2.16"/>
-    <dynamics damping="0.0" friction="0.0"/>
-  </joint>
-  <link name="ur10_arm_shoulder_link">
-    <visual>
-      <geometry>
-        <mesh filename="file://$(find upright_assets)/thing/meshes/ur10/visual/shoulder.dae"/>
-      </geometry>
-      <material name="LightGrey">
-        <color rgba="0.7 0.7 0.7 1.0"/>
-      </material>
-    </visual>
-    <collision>
-      <geometry>
-        <mesh filename="file://$(find upright_assets)/thing/meshes/ur10/collision/shoulder.stl"/>
-      </geometry>
-    </collision>
-    <inertial>
-      <mass value="7.778"/>
-      <origin rpy="0 0 0" xyz="0.0 0.0 0.0"/>
-      <inertia ixx="0.0314743125769" ixy="0.0" ixz="0.0" iyy="0.0314743125769" iyz="0.0" izz="0.021875625"/>
-    </inertial>
-  </link>
-  <joint name="ur10_arm_shoulder_lift_joint" type="revolute">
-    <parent link="ur10_arm_shoulder_link"/>
-    <child link="ur10_arm_upper_arm_link"/>
-    <origin rpy="0.0 1.57079632679 0.0" xyz="0.0 0.220941 0.0"/>
-    <axis xyz="0 1 0"/>
-    <limit effort="330.0" lower="-6.28318530718" upper="6.28318530718" velocity="2.16"/>
-    <dynamics damping="0.0" friction="0.0"/>
-  </joint>
-  <link name="ur10_arm_upper_arm_link">
-    <visual>
-      <geometry>
-        <mesh filename="file://$(find upright_assets)/thing/meshes/ur10/visual/upperarm.dae"/>
-      </geometry>
-      <material name="LightGrey">
-        <color rgba="0.7 0.7 0.7 1.0"/>
-      </material>
-    </visual>
-    <collision>
-      <geometry>
-        <mesh filename="file://$(find upright_assets)/thing/meshes/ur10/collision/upperarm.stl"/>
-      </geometry>
-    </collision>
-    <inertial>
-      <mass value="12.93"/>
-      <origin rpy="0 0 0" xyz="0.0 -0.045 0.306"/>
-      <inertia ixx="0.421753803798" ixy="0.0" ixz="0.0" iyy="0.421753803798" iyz="0.0" izz="0.036365625"/>
-    </inertial>
-  </link>
-  <joint name="ur10_arm_elbow_joint" type="revolute">
-    <parent link="ur10_arm_upper_arm_link"/>
-    <child link="ur10_arm_forearm_link"/>
-    <origin rpy="0.0 0.0 0.0" xyz="0.0 -0.1719 0.612"/>
-    <axis xyz="0 1 0"/>
-    <limit effort="150.0" lower="-3.14159265359" upper="3.14159265359" velocity="3.15"/>
-    <dynamics damping="0.0" friction="0.0"/>
-  </joint>
-  <link name="ur10_arm_forearm_link">
-    <visual>
-      <geometry>
-        <mesh filename="file://$(find upright_assets)/thing/meshes/ur10/visual/forearm.dae"/>
-      </geometry>
-      <material name="LightGrey">
-        <color rgba="0.7 0.7 0.7 1.0"/>
-      </material>
-    </visual>
-    <collision>
-      <geometry>
-        <mesh filename="file://$(find upright_assets)/thing/meshes/ur10/collision/forearm.stl"/>
-      </geometry>
-    </collision>
-    <inertial>
-      <mass value="3.87"/>
-      <origin rpy="0 0 0" xyz="0.0 0.0 0.28615"/>
-      <inertia ixx="0.111069694097" ixy="0.0" ixz="0.0" iyy="0.111069694097" iyz="0.0" izz="0.010884375"/>
-    </inertial>
-  </link>
-  <joint name="ur10_arm_wrist_1_joint" type="revolute">
-    <parent link="ur10_arm_forearm_link"/>
-    <child link="ur10_arm_wrist_1_link"/>
-    <origin rpy="0.0 1.57079632679 0.0" xyz="0.0 0.0 0.5723"/>
-    <axis xyz="0 1 0"/>
-    <limit effort="54.0" lower="-6.28318530718" upper="6.28318530718" velocity="3.2"/>
-    <dynamics damping="0.0" friction="0.0"/>
-  </joint>
-  <link name="ur10_arm_wrist_1_link">
-    <visual>
-      <geometry>
-        <mesh filename="file://$(find upright_assets)/thing/meshes/ur10/visual/wrist1.dae"/>
-      </geometry>
-      <material name="LightGrey">
-        <color rgba="0.7 0.7 0.7 1.0"/>
-      </material>
-    </visual>
-    <collision>
-      <geometry>
-        <mesh filename="file://$(find upright_assets)/thing/meshes/ur10/collision/wrist1.stl"/>
-      </geometry>
-    </collision>
-    <inertial>
-      <mass value="1.96"/>
-      <origin rpy="0 0 0" xyz="0.0 0.1149 0.0"/>
-      <inertia ixx="0.0051082479567" ixy="0.0" ixz="0.0" iyy="0.0051082479567" iyz="0.0" izz="0.0055125"/>
-    </inertial>
-  </link>
-  <joint name="ur10_arm_wrist_2_joint" type="revolute">
-    <parent link="ur10_arm_wrist_1_link"/>
-    <child link="ur10_arm_wrist_2_link"/>
-    <origin rpy="0.0 0.0 0.0" xyz="0.0 0.1149 0.0"/>
-    <axis xyz="0 0 1"/>
-    <limit effort="54.0" lower="-6.28318530718" upper="6.28318530718" velocity="3.2"/>
-    <dynamics damping="0.0" friction="0.0"/>
-  </joint>
-  <link name="ur10_arm_wrist_2_link">
-    <visual>
-      <geometry>
-        <mesh filename="file://$(find upright_assets)/thing/meshes/ur10/visual/wrist2.dae"/>
-      </geometry>
-      <material name="LightGrey">
-        <color rgba="0.7 0.7 0.7 1.0"/>
-      </material>
-    </visual>
-    <collision>
-      <geometry>
-        <mesh filename="file://$(find upright_assets)/thing/meshes/ur10/collision/wrist2.stl"/>
-      </geometry>
-    </collision>
-    <inertial>
-      <mass value="1.96"/>
-      <origin rpy="0 0 0" xyz="0.0 0.0 0.1157"/>
-      <inertia ixx="0.0051082479567" ixy="0.0" ixz="0.0" iyy="0.0051082479567" iyz="0.0" izz="0.0055125"/>
-    </inertial>
-  </link>
-  <joint name="ur10_arm_wrist_3_joint" type="revolute">
-    <parent link="ur10_arm_wrist_2_link"/>
-    <child link="ur10_arm_wrist_3_link"/>
-    <origin rpy="0.0 0.0 0.0" xyz="0.0 0.0 0.1157"/>
-    <axis xyz="0 1 0"/>
-    <limit effort="54.0" lower="-6.28318530718" upper="6.28318530718" velocity="3.2"/>
-    <dynamics damping="0.0" friction="0.0"/>
-  </joint>
-  <link name="ur10_arm_wrist_3_link">
-    <visual>
-      <geometry>
-        <mesh filename="file://$(find upright_assets)/thing/meshes/ur10/visual/wrist3.dae"/>
-      </geometry>
-      <material name="LightGrey">
-        <color rgba="0.7 0.7 0.7 1.0"/>
-      </material>
-    </visual>
-    <collision>
-      <geometry>
-        <mesh filename="file://$(find upright_assets)/thing/meshes/ur10/collision/wrist3.stl"/>
-      </geometry>
-    </collision>
-    <inertial>
-      <mass value="0.202"/>
-      <origin rpy="1.57079632679 0 0" xyz="0.0 0.07695 0.0"/>
-      <inertia ixx="0.000117921661165" ixy="0.0" ixz="0.0" iyy="0.000117921661165" iyz="0.0" izz="0.000204525"/>
-    </inertial>
-  </link>
-  <joint name="ur10_arm_ee_fixed_joint" type="fixed">
-    <parent link="ur10_arm_wrist_3_link"/>
-    <child link="ur10_arm_ee_link"/>
-    <origin rpy="0.0 0.0 1.57079632679" xyz="0.0 0.0922 0.0"/>
-  </joint>
-  <link name="ur10_arm_ee_link">
-    <collision>
-      <geometry>
-        <box size="0.01 0.01 0.01"/>
-      </geometry>
-      <origin rpy="0 0 0" xyz="-0.01 0 0"/>
-    </collision>
-  </link>
-  <!-- Frame coincident with all-zeros TCP on UR controller -->
-  <link name="ur10_arm_tool0">
-    <visual>
-      <!-- start halfway along the cylinder -->
-      <origin rpy="0 0 0" xyz="0 0 0.145"/>
-      <geometry>
-        <cylinder length="0.290" radius="0.01"/>
-      </geometry>
-      <material name="black"/>
-    </visual>
-    <collision>
-      <origin rpy="0 0 0" xyz="0 0 0.145"/>
-      <geometry>
-        <cylinder length="0.290" radius="0.01"/>
-      </geometry>
-    </collision>
-  </link>
-  <joint name="ur10_arm_wrist_3_link-tool0_fixed_joint" type="fixed">
-    <origin rpy="-1.57079632679 0.2617993877991494 0" xyz="0 0.0922 0"/>
-    <parent link="ur10_arm_wrist_3_link"/>
-    <child link="ur10_arm_tool0"/>
-  </joint>
-  <!-- Join arm -->
+  <!-- UR10 arm -->
+  <xacro:include filename="$(find ur_description)/urdf/inc/ur10_macro.xacro"/>
+  <xacro:ur10_robot
+    prefix="ur10_arm_"
+    visual_parameters_file="$(find upright_assets)/config/ur10/visual_parameters.yaml"
+    kinematics_parameters_file="$(find upright_assets)/config/ur10/calibration.yaml"
+  />
+  <!-- Join arm to the base -->
   <joint name="ur10_arm_base" type="fixed">
     <parent link="arch_link"/>
@@ -592,3 +371,49 @@
     <origin rpy="0.0 0.0 3.14159265359" xyz="0.01 -0.27 0.375"/>
   </joint>
+  <!-- Frame coincident with all-zeros TCP on UR controller -->
+  <link name="gripper">
+    <visual>
+      <!-- start halfway along the cylinder -->
+      <origin rpy="0 0 0" xyz="0 0 0.145"/>
+      <geometry>
+        <cylinder length="0.290" radius="0.01"/>
+      </geometry>
+      <material name="black"/>
+    </visual>
+    <collision>
+      <origin rpy="0 0 0" xyz="0 0 0.145"/>
+      <geometry>
+        <cylinder length="0.290" radius="0.01"/>
+      </geometry>
+    </collision>
+  </link>
+  <joint name="tool_gripper_joint" type="fixed">
+    <!-- The 15-degree offset about the z-axis is to account for the fact that the gripper is actually mounted at this offset. -->
+    <origin rpy="0 0 0.2617993877991494" xyz="0 0.0 0"/>
+    <parent link="ur10_arm_tool0"/>
+    <child link="gripper"/>
+  </joint>
+  <!-- &#60;&#33;&#45;&#45; Frame coincident with all-zeros TCP on UR controller &#45;&#45;&#62; -->
+  <!-- <link name="ur10_arm_tool0"> -->
+  <!--   <visual> -->
+  <!--     &#60;&#33;&#45;&#45; start halfway along the cylinder &#45;&#45;&#62; -->
+  <!--     <origin rpy="0 0 0" xyz="0 0 0.145"/> -->
+  <!--     <geometry> -->
+  <!--       <cylinder length="0.290" radius="0.01"/> -->
+  <!--     </geometry> -->
+  <!--     <material name="black"/> -->
+  <!--   </visual> -->
+  <!--   <collision> -->
+  <!--     <origin rpy="0 0 0" xyz="0 0 0.145"/> -->
+  <!--     <geometry> -->
+  <!--       <cylinder length="0.290" radius="0.01"/> -->
+  <!--     </geometry> -->
+  <!--   </collision> -->
+  <!-- </link> -->
+  <!--  -->
+  <!-- <joint name="ur10_arm_wrist_3_link-tool0_fixed_joint" type="fixed"> -->
+  <!--   <origin rpy="-1.57079632679 0.2617993877991494 0" xyz="0 0.0922 0"/> -->
+  <!--   <parent link="ur10_arm_wrist_3_link"/> -->
+  <!--   <child link="ur10_arm_tool0"/> -->
+  <!-- </joint> -->
 </robot>

File: upright_assets/thing/xacro/pyb/mm_pyb_old.urdf.xacro (robot description, xacro)
@@ -1,4 +1,4 @@
 <?xml version="1.0" encoding="utf-8"?>
-<robot name="Thing" xmlns:xacro="http://wiki.ros.org/xacro">
+<robot name="Thing">
   <material name="dark_grey">
     <color rgba="0.2 0.2 0.2 1.0"/>
@@ -251,4 +251,9 @@
       </material>
     </visual>
+    <!-- <collision> -->
+    <!-- 	<geometry> -->
+    <!-- 		<mesh filename="package://mm_description/thing/meshes/tor11_mech.dae" /> -->
+    <!-- 	</geometry> -->
+    <!-- </collision> -->
   </link>
   <joint name="arch_joint" type="fixed">
@@ -257,12 +262,234 @@
     <child link="arch_link"/>
   </joint>
-  <!-- UR10 arm -->
-  <xacro:include filename="$(find ur_description)/urdf/inc/ur10_macro.xacro"/>
-  <xacro:ur10_robot
-    prefix="ur10_arm_"
-    visual_parameters_file="$(find upright_assets)/config/ur10/visual_parameters.yaml"
-    kinematics_parameters_file="$(find upright_assets)/config/ur10/calibration.yaml"
-  />
-  <!-- Join arm to the base -->
+  <!--
+  Author: Kelsey Hawkins
+  Contributers: Jimmy Da Silva, Ajit Krisshna N L, Muhammad Asif Rana
+-->
+  <!-- measured from model -->
+  <link name="ur10_arm_base_link">
+    <visual>
+      <geometry>
+        <mesh filename="file://$(find upright_assets)/thing/meshes/ur10/visual/base.dae"/>
+      </geometry>
+      <material name="LightGrey">
+        <color rgba="0.7 0.7 0.7 1.0"/>
+      </material>
+    </visual>
+    <collision>
+      <geometry>
+        <mesh filename="file://$(find upright_assets)/thing/meshes/ur10/collision/base.stl"/>
+      </geometry>
+    </collision>
+    <inertial>
+      <mass value="4.0"/>
+      <origin rpy="0 0 0" xyz="0.0 0.0 0.0"/>
+      <inertia ixx="0.0061063308908" ixy="0.0" ixz="0.0" iyy="0.0061063308908" iyz="0.0" izz="0.01125"/>
+    </inertial>
+  </link>
+  <joint name="ur10_arm_shoulder_pan_joint" type="revolute">
+    <parent link="ur10_arm_base_link"/>
+    <child link="ur10_arm_shoulder_link"/>
+    <origin rpy="0.0 0.0 0.0" xyz="0.0 0.0 0.1273"/>
+    <axis xyz="0 0 1"/>
+    <limit effort="330.0" lower="-6.28318530718" upper="6.28318530718" velocity="2.16"/>
+    <dynamics damping="0.0" friction="0.0"/>
+  </joint>
+  <link name="ur10_arm_shoulder_link">
+    <visual>
+      <geometry>
+        <mesh filename="file://$(find upright_assets)/thing/meshes/ur10/visual/shoulder.dae"/>
+      </geometry>
+      <material name="LightGrey">
+        <color rgba="0.7 0.7 0.7 1.0"/>
+      </material>
+    </visual>
+    <collision>
+      <geometry>
+        <mesh filename="file://$(find upright_assets)/thing/meshes/ur10/collision/shoulder.stl"/>
+      </geometry>
+    </collision>
+    <inertial>
+      <mass value="7.778"/>
+      <origin rpy="0 0 0" xyz="0.0 0.0 0.0"/>
+      <inertia ixx="0.0314743125769" ixy="0.0" ixz="0.0" iyy="0.0314743125769" iyz="0.0" izz="0.021875625"/>
+    </inertial>
+  </link>
+  <joint name="ur10_arm_shoulder_lift_joint" type="revolute">
+    <parent link="ur10_arm_shoulder_link"/>
+    <child link="ur10_arm_upper_arm_link"/>
+    <origin rpy="0.0 1.57079632679 0.0" xyz="0.0 0.220941 0.0"/>
+    <axis xyz="0 1 0"/>
+    <limit effort="330.0" lower="-6.28318530718" upper="6.28318530718" velocity="2.16"/>
+    <dynamics damping="0.0" friction="0.0"/>
+  </joint>
+  <link name="ur10_arm_upper_arm_link">
+    <visual>
+      <geometry>
+        <mesh filename="file://$(find upright_assets)/thing/meshes/ur10/visual/upperarm.dae"/>
+      </geometry>
+      <material name="LightGrey">
+        <color rgba="0.7 0.7 0.7 1.0"/>
+      </material>
+    </visual>
+    <collision>
+      <geometry>
+        <mesh filename="file://$(find upright_assets)/thing/meshes/ur10/collision/upperarm.stl"/>
+      </geometry>
+    </collision>
+    <inertial>
+      <mass value="12.93"/>
+      <origin rpy="0 0 0" xyz="0.0 -0.045 0.306"/>
+      <inertia ixx="0.421753803798" ixy="0.0" ixz="0.0" iyy="0.421753803798" iyz="0.0" izz="0.036365625"/>
+    </inertial>
+  </link>
+  <joint name="ur10_arm_elbow_joint" type="revolute">
+    <parent link="ur10_arm_upper_arm_link"/>
+    <child link="ur10_arm_forearm_link"/>
+    <origin rpy="0.0 0.0 0.0" xyz="0.0 -0.1719 0.612"/>
+    <axis xyz="0 1 0"/>
+    <limit effort="150.0" lower="-3.14159265359" upper="3.14159265359" velocity="3.15"/>
+    <dynamics damping="0.0" friction="0.0"/>
+  </joint>
+  <link name="ur10_arm_forearm_link">
+    <visual>
+      <geometry>
+        <mesh filename="file://$(find upright_assets)/thing/meshes/ur10/visual/forearm.dae"/>
+      </geometry>
+      <material name="LightGrey">
+        <color rgba="0.7 0.7 0.7 1.0"/>
+      </material>
+    </visual>
+    <collision>
+      <geometry>
+        <mesh filename="file://$(find upright_assets)/thing/meshes/ur10/collision/forearm.stl"/>
+      </geometry>
+    </collision>
+    <inertial>
+      <mass value="3.87"/>
+      <origin rpy="0 0 0" xyz="0.0 0.0 0.28615"/>
+      <inertia ixx="0.111069694097" ixy="0.0" ixz="0.0" iyy="0.111069694097" iyz="0.0" izz="0.010884375"/>
+    </inertial>
+  </link>
+  <joint name="ur10_arm_wrist_1_joint" type="revolute">
+    <parent link="ur10_arm_forearm_link"/>
+    <child link="ur10_arm_wrist_1_link"/>
+    <origin rpy="0.0 1.57079632679 0.0" xyz="0.0 0.0 0.5723"/>
+    <axis xyz="0 1 0"/>
+    <limit effort="54.0" lower="-6.28318530718" upper="6.28318530718" velocity="3.2"/>
+    <dynamics damping="0.0" friction="0.0"/>
+  </joint>
+  <link name="ur10_arm_wrist_1_link">
+    <visual>
+      <geometry>
+        <mesh filename="file://$(find upright_assets)/thing/meshes/ur10/visual/wrist1.dae"/>
+      </geometry>
+      <material name="LightGrey">
+        <color rgba="0.7 0.7 0.7 1.0"/>
+      </material>
+    </visual>
+    <collision>
+      <geometry>
+        <mesh filename="file://$(find upright_assets)/thing/meshes/ur10/collision/wrist1.stl"/>
+      </geometry>
+    </collision>
+    <inertial>
+      <mass value="1.96"/>
+      <origin rpy="0 0 0" xyz="0.0 0.1149 0.0"/>
+      <inertia ixx="0.0051082479567" ixy="0.0" ixz="0.0" iyy="0.0051082479567" iyz="0.0" izz="0.0055125"/>
+    </inertial>
+  </link>
+  <joint name="ur10_arm_wrist_2_joint" type="revolute">
+    <parent link="ur10_arm_wrist_1_link"/>
+    <child link="ur10_arm_wrist_2_link"/>
+    <origin rpy="0.0 0.0 0.0" xyz="0.0 0.1149 0.0"/>
+    <axis xyz="0 0 1"/>
+    <limit effort="54.0" lower="-6.28318530718" upper="6.28318530718" velocity="3.2"/>
+    <dynamics damping="0.0" friction="0.0"/>
+  </joint>
+  <link name="ur10_arm_wrist_2_link">
+    <visual>
+      <geometry>
+        <mesh filename="file://$(find upright_assets)/thing/meshes/ur10/visual/wrist2.dae"/>
+      </geometry>
+      <material name="LightGrey">
+        <color rgba="0.7 0.7 0.7 1.0"/>
+      </material>
+    </visual>
+    <collision>
+      <geometry>
+        <mesh filename="file://$(find upright_assets)/thing/meshes/ur10/collision/wrist2.stl"/>
+      </geometry>
+    </collision>
+    <inertial>
+      <mass value="1.96"/>
+      <origin rpy="0 0 0" xyz="0.0 0.0 0.1157"/>
+      <inertia ixx="0.0051082479567" ixy="0.0" ixz="0.0" iyy="0.0051082479567" iyz="0.0" izz="0.0055125"/>
+    </inertial>
+  </link>
+  <joint name="ur10_arm_wrist_3_joint" type="revolute">
+    <parent link="ur10_arm_wrist_2_link"/>
+    <child link="ur10_arm_wrist_3_link"/>
+    <origin rpy="0.0 0.0 0.0" xyz="0.0 0.0 0.1157"/>
+    <axis xyz="0 1 0"/>
+    <limit effort="54.0" lower="-6.28318530718" upper="6.28318530718" velocity="3.2"/>
+    <dynamics damping="0.0" friction="0.0"/>
+  </joint>
+  <link name="ur10_arm_wrist_3_link">
+    <visual>
+      <geometry>
+        <mesh filename="file://$(find upright_assets)/thing/meshes/ur10/visual/wrist3.dae"/>
+      </geometry>
+      <material name="LightGrey">
+        <color rgba="0.7 0.7 0.7 1.0"/>
+      </material>
+    </visual>
+    <collision>
+      <geometry>
+        <mesh filename="file://$(find upright_assets)/thing/meshes/ur10/collision/wrist3.stl"/>
+      </geometry>
+    </collision>
+    <inertial>
+      <mass value="0.202"/>
+      <origin rpy="1.57079632679 0 0" xyz="0.0 0.07695 0.0"/>
+      <inertia ixx="0.000117921661165" ixy="0.0" ixz="0.0" iyy="0.000117921661165" iyz="0.0" izz="0.000204525"/>
+    </inertial>
+  </link>
+  <joint name="ur10_arm_ee_fixed_joint" type="fixed">
+    <parent link="ur10_arm_wrist_3_link"/>
+    <child link="ur10_arm_ee_link"/>
+    <origin rpy="0.0 0.0 1.57079632679" xyz="0.0 0.0922 0.0"/>
+  </joint>
+  <link name="ur10_arm_ee_link">
+    <collision>
+      <geometry>
+        <box size="0.01 0.01 0.01"/>
+      </geometry>
+      <origin rpy="0 0 0" xyz="-0.01 0 0"/>
+    </collision>
+  </link>
+  <!-- Frame coincident with all-zeros TCP on UR controller -->
+  <link name="ur10_arm_tool0">
+    <visual>
+      <!-- start halfway along the cylinder -->
+      <origin rpy="0 0 0" xyz="0 0 0.145"/>
+      <geometry>
+        <cylinder length="0.290" radius="0.01"/>
+      </geometry>
+      <material name="black"/>
+    </visual>
+    <collision>
+      <origin rpy="0 0 0" xyz="0 0 0.145"/>
+      <geometry>
+        <cylinder length="0.290" radius="0.01"/>
+      </geometry>
+    </collision>
+  </link>
+  <joint name="ur10_arm_wrist_3_link-tool0_fixed_joint" type="fixed">
+    <!-- The 15-degree offset about the y-axis is to account for the fact that the gripper is actually mounted at this offset. -->
+    <origin rpy="-1.57079632679 0.2617993877991494 0" xyz="0 0.0922 0"/>
+    <parent link="ur10_arm_wrist_3_link"/>
+    <child link="ur10_arm_tool0"/>
+  </joint>
+  <!-- Join arm -->
   <joint name="ur10_arm_base" type="fixed">
     <parent link="arch_link"/>
@@ -270,26 +497,3 @@
     <origin rpy="0.0 0.0 3.14159265359" xyz="0.01 -0.27 0.375"/>
   </joint>
-  <!-- Frame coincident with all-zeros TCP on UR controller -->
-  <link name="gripper">
-    <visual>
-      <!-- start halfway along the cylinder -->
-      <origin rpy="0 0 0" xyz="0 0 0.145"/>
-      <geometry>
-        <cylinder length="0.290" radius="0.01"/>
-      </geometry>
-      <material name="black"/>
-    </visual>
-    <collision>
-      <origin rpy="0 0 0" xyz="0 0 0.145"/>
-      <geometry>
-        <cylinder length="0.290" radius="0.01"/>
-      </geometry>
-    </collision>
-  </link>
-  <joint name="tool_gripper_joint" type="fixed">
-    <!-- The 15-degree offset about the z-axis is to account for the fact that the gripper is actually mounted at this offset. -->
-    <origin rpy="0 0 0.2617993877991494" xyz="0 0.0 0"/>
-    <parent link="ur10_arm_tool0"/>
-    <child link="gripper"/>
-  </joint>
 </robot>
