Commit message: OCS2 and PyBullet mostly share the same URDF xacro stuff.

File: upright_assets/thing/xacro/end_effector_fingers.urdf.xacro (robot description, xacro)
@@ -1,7 +1,7 @@
 <?xml version="1.0" encoding="utf-8"?>
 <robot name="end_effector_fingers">
-  <joint name="tool0_tcp_fixed_joint" type="fixed">
+  <joint name="gripper_tool_joint" type="fixed">
     <origin rpy="0.0 0.0 3.14159" xyz="0.0 0.0 0.290"/>
-    <parent link="ur10_arm_tool0"/>
+    <parent link="gripper"/>
     <child link="thing_tool"/>
   </joint>

File: upright_assets/thing/xacro/mm.urdf.xacro (robot description, xacro)
@@ -22,46 +22,4 @@
     <color rgba="0.0 0.0 0.0 0.25"/>
   </material>
-  <link name="world_link">
-    <inertial>
-      <mass value="0"/>
-      <inertia ixx="0.2125" ixy="-0.005" ixz="0.0225" iyy="0.205" iyz="0.045" izz="0.0125"/>
-      <origin rpy="0 0 0" xyz="0 0 0"/>
-    </inertial>
-  </link>
-	<link name="x_prismatic_link">
-	 <inertial>
-     <mass value="0.01"/>
-     <inertia ixx="0.01" ixy="0" ixz="0" iyy="0.01" iyz="0" izz="0.01"/>
-     <origin rpy="0 0 0" xyz="0 0 0"/>
-    </inertial>
-  </link>
-	<joint name="x_to_world_joint" type="prismatic">
-    <parent link="world_link"/>
-    <child link="x_prismatic_link"/>
-    <axis xyz="1 0 0"/>
-    <origin rpy="0 0 0" xyz="0 0 0"/>
-    <limit effort="0.0" velocity="1000.0"/>
-  </joint>
-	<link name="y_prismatic_link">
-	 <inertial>
-     <mass value="0.01"/>
-     <inertia ixx="0.01" ixy="0" ixz="0" iyy="0.01" iyz="0" izz="0.01"/>
-     <origin rpy="0 0 0" xyz="0 0 0"/>
-    </inertial>
-  </link>
-	<joint name="y_to_x_joint" type="prismatic">
-    <parent link="x_prismatic_link"/>
-    <child link="y_prismatic_link"/>
-    <axis xyz="0 1 0"/>
-    <origin rpy="0 0 0" xyz="0 0 0"/>
-    <limit effort="0.0" velocity="1000.0"/>
-  </joint>
-  <!-- Note the z-offset to raise the base off the ground, to avoid collision issues. Without this, there are vibrations and other artifacts from resolving the ground collision that result in significant error in the balanced object. -->
-	<joint name="base_to_y_joint" type="continuous">
-    <parent link="y_prismatic_link"/>
-    <child link="base_link"/>
-    <axis xyz="0 0 1"/>
-    <origin rpy="0 0 0" xyz="0 0 0.01"/>
-  </joint>
   <link name="base_link">
 	 <inertial>

File: upright_assets/thing/xacro/ocs2/mm_ocs2_fingers.urdf.xacro (robot description, xacro)
@@ -1,5 +1,5 @@
 <?xml version="1.0" ?>
-<robot name="mm_pyb_tray" xmlns:xacro="http://www.ros.org/wiki/xacro">
-  <xacro:include filename="mm_ocs2.urdf.xacro" />
+<robot name="mm_ocs2_fingers" xmlns:xacro="http://www.ros.org/wiki/xacro">
+  <xacro:include filename="../mm.urdf.xacro" />
   <xacro:include filename="../end_effector_fingers.urdf.xacro" />
 </robot>

File: upright_assets/thing/xacro/ocs2/mm_ocs2_tray.urdf.xacro (robot description, xacro)
@@ -1,5 +1,5 @@
 <?xml version="1.0" ?>
-<robot name="mm_pyb_tray" xmlns:xacro="http://www.ros.org/wiki/xacro">
-  <xacro:include filename="mm_ocs2.urdf.xacro" />
+<robot name="mm_ocs2_tray" xmlns:xacro="http://www.ros.org/wiki/xacro">
+  <xacro:include filename="../mm.urdf.xacro" />
   <xacro:include filename="../end_effector_tray.urdf.xacro" />
 </robot>

File: upright_assets/thing/xacro/pyb/mm_pyb_fingers.urdf.xacro (robot description, xacro)
@@ -1,5 +1,6 @@
 <?xml version="1.0" ?>
-<robot name="mm_pyb_tray" xmlns:xacro="http://www.ros.org/wiki/xacro">
-  <xacro:include filename="mm_pyb.urdf.xacro" />
+<robot name="mm_pyb_fingers" xmlns:xacro="http://www.ros.org/wiki/xacro">
+  <xacro:include filename="base_joints.urdf.xacro" />
+  <xacro:include filename="../mm.urdf.xacro" />
   <xacro:include filename="../end_effector_fingers.urdf.xacro" />
 </robot>

File: upright_assets/thing/xacro/pyb/mm_pyb_tray.urdf.xacro (robot description, xacro)
@@ -1,5 +1,6 @@
 <?xml version="1.0" ?>
 <robot name="mm_pyb_tray" xmlns:xacro="http://www.ros.org/wiki/xacro">
-  <xacro:include filename="mm_pyb.urdf.xacro" />
+  <xacro:include filename="base_joints.urdf.xacro" />
+  <xacro:include filename="../mm.urdf.xacro" />
   <xacro:include filename="../end_effector_tray.urdf.xacro" />
 </robot>
