Commit message: Basic MPC works on the real robot now.

File: upright_assets/thing/xacro/mm.urdf.xacro (robot description, xacro)
@@ -168,36 +168,4 @@
     </collision>
   </link>
-  <joint name="axle_joint" type="fixed">
-    <origin rpy="0 0 0" xyz="0 0 0.05"/>
-    <parent link="chassis_link"/>
-    <child link="axle_link"/>
-  </joint>
-  <link name="axle_link">
-    <visual>
-      <origin rpy="0 1.57079632679 0" xyz="0 0 0"/>
-      <geometry>
-        <mesh filename="file://$(find upright_assets)/thing/meshes/ridgeback/axle.stl"/>
-      </geometry>
-      <material name="black"/>
-    </visual>
-  </link>
-  <link name="imu_link">
-    <inertial>
-      <mass value="0.001"/>
-      <origin rpy="0 0 0" xyz="0 0 0"/>
-      <inertia ixx="1e-09" ixy="0.0" ixz="0.0" iyy="1e-09" iyz="0.0" izz="1e-09"/>
-    </inertial>
-  </link>
-  <joint name="imu_joint" type="fixed">
-    <parent link="chassis_link"/>
-    <child link="imu_link"/>
-    <origin rpy="0 0 0" xyz="0.2085 -0.2902 0.1681"/>
-  </joint>
-  <link name="mid_mount"/>
-  <joint name="mid_mount_joint" type="fixed">
-    <parent link="base_link"/>
-    <child link="mid_mount"/>
-    <origin rpy="0 0 0" xyz="0 0 0.28"/>
-  </joint>
   <link name="arch_link">
     <visual>

File: upright_assets/thing/xacro/ros/ridgeback_wheels.urdf.xacro (robot description, xacro)
@@ -15,10 +15,4 @@
   <xacro:property name="imu_offset_z" value="0.1681" />
   <xacro:property name="dummy_inertia" value="1e-09"/>
-  <material name="dark_grey"><color rgba="0.2 0.2 0.2 1.0" /></material>
-  <material name="light_grey"><color rgba="0.4 0.4 0.4 1.0" /></material>
-  <material name="red"><color rgba="0.8 0.0 0.0 1.0" /></material>
-  <material name="white"><color rgba="0.9 0.9 0.9 1.0" /></material>
-  <material name="yellow"><color rgba="0.8 0.8 0.0 1.0" /></material>
-  <material name="black"><color rgba="0.15 0.15 0.15 1.0" /></material>
   <xacro:macro name="wheel" params="prefix side *joint_pose">
     <link name="${prefix}_${side}_wheel_link">

Commit message: Bringing back static obstacle avoidance.
There is a convenience Pinocchio geometry interface in Python for quick
experimenting and sanity checking.

File: upright_assets/thing/xacro/mm.urdf.xacro (robot description, xacro)
@@ -20,5 +20,5 @@
   </material>
   <material name="seethrough">
-    <color rgba="0.0 0.0 0.0 0.25"/>
+    <color rgba="1.0 0.0 0.0 0.25"/>
   </material>
   <link name="base_link">
@@ -36,9 +36,4 @@
   <link name="chassis_link">
     <visual>
-      <!-- <origin rpy="0 0 0" xyz="0 0 0.15"/> -->
-      <!-- <geometry> -->
-      <!--   <box size="1.0 0.8 0.3"/> -->
-      <!-- </geometry> -->
-      <!-- <origin xyz="0 0 0"/> -->
       <geometry>
         <mesh filename="file://$(find upright_assets)/thing/meshes/ridgeback/body.stl"/>
@@ -47,13 +42,8 @@
     </visual>
     <collision>
-      <!-- simpler collision geometry for speed -->
-      <origin rpy="0 0 0" xyz="0 0 0.15"/>
-      <geometry>
-        <box size="1.0 0.8 0.3"/>
-      </geometry>
-      <!-- <origin xyz="0 0 0"/> -->
-      <!-- <geometry> -->
-      <!--   <mesh filename="file://$(find upright_assets)/thing/meshes/ridgeback/body&#45;collision.stl"/> -->
-      <!-- </geometry> -->
+      <origin xyz="0 0 0"/>
+      <geometry>
+        <mesh filename="file://$(find upright_assets)/thing/meshes/ridgeback/body-collision.stl"/>
+      </geometry>
     </collision>
     <inertial>
@@ -180,4 +170,5 @@
   <joint name="arch_joint" type="fixed">
     <origin rpy="0 0 1.57079632679" xyz="0 0 0.278"/>
+    <!-- <origin rpy="-1.57079632679 0 1.57079632679" xyz="0 0 0.278"/> -->
     <parent link="top_link"/>
     <child link="arch_link"/>

File: upright_assets/thing/xacro/ocs2/mm_ocs2_tray.urdf.xacro (robot description, xacro)
@@ -3,3 +3,4 @@
   <xacro:include filename="../mm.urdf.xacro" />
   <xacro:include filename="../end_effector_tray.urdf.xacro" />
+  <xacro:include filename="../collision_links.urdf.xacro" />
 </robot>

File: upright_assets/thing/xacro/pyb/mm_pyb_tray.urdf.xacro (robot description, xacro)
@@ -4,3 +4,4 @@
   <xacro:include filename="../mm.urdf.xacro" />
   <xacro:include filename="../end_effector_tray.urdf.xacro" />
+  <xacro:include filename="../visual_collision_links.urdf.xacro" />
 </robot>

File: upright_assets/thing/xacro/visual_collision_links.urdf.xacro (robot description, xacro)
@@ -1,36 +1,10 @@
 <?xml version="1.0" encoding="utf-8"?>
 <robot name="collision_links">
-  <material name="seethrough">
-    <color rgba="1.0 0.0 0.0 0.5"/>
-  </material>
-  <!-- Collision element to protect the balanced objects -->
-  <!-- This configuration is used for both obstacle avoidance tasks -->
-  <!-- <link name="balanced_object_collision_link"> -->
-  <!--   <collision> -->
-  <!--     <origin rpy="0 0 0" xyz="0 0 0.1"/> -->
-  <!--     <geometry> -->
-  <!--       <cylinder length="0.25" radius="0.25"/> -->
-  <!--     </geometry> -->
-  <!--   </collision> -->
-  <!--   <visual> -->
-  <!--     <origin rpy="0 0 0" xyz="0 0 0.1"/> -->
-  <!--     <geometry> -->
-  <!--       <cylinder length="0.25" radius="0.25"/> -->
-  <!--     </geometry> -->
-  <!--     <material name="seethrough"/> -->
-  <!--   </visual> -->
-  <!-- </link> -->
   <!-- This configuration is used for the single- and multi-object balancing tasks -->
   <link name="balanced_object_collision_link">
-    <collision>
-      <origin rpy="0 0 0" xyz="0 0 0.02"/>
+    <visual>
+      <origin rpy="0 0 0" xyz="0 0 0"/>
       <geometry>
-        <cylinder length="0.1" radius="0.25"/>
-      </geometry>
-    </collision>
-    <visual>
-      <origin rpy="0 0 0" xyz="0 0 0.02"/>
-      <geometry>
-        <cylinder length="0.1" radius="0.25"/>
+        <sphere radius="0.2"/>
       </geometry>
       <material name="seethrough"/>
@@ -38,5 +12,5 @@
   </link>
   <joint name="balanced_object_collision_joint" type="fixed">
-    <origin rpy="0 0 0" xyz="0 0 0"/>
+    <origin rpy="0 0 0" xyz="0 0 0.05"/>
     <parent link="thing_tool"/>
     <child link="balanced_object_collision_link"/>
@@ -44,10 +18,4 @@
   <!-- Collision sphere for the shoulder -->
   <link name="shoulder_collision_link">
-    <collision>
-      <origin rpy="0 0 0" xyz="0 0 0"/>
-      <geometry>
-        <sphere radius="0.15"/>
-      </geometry>
-    </collision>
     <visual>
       <origin rpy="0 0 0" xyz="0 0 0"/>
@@ -65,12 +33,6 @@
   <!-- Collision cylinder for the upper arm link -->
   <link name="upper_arm_collision_link">
-    <collision>
-      <origin rpy="0 0 0" xyz="0 -0.05 0.325"/>
-      <geometry>
-        <cylinder length="0.65" radius="0.06"/>
-      </geometry>
-    </collision>
     <visual>
-      <origin rpy="0 0 0" xyz="0 -0.05 0.325"/>
+      <origin rpy="0 0 0" xyz="0 0 0"/>
       <geometry>
         <cylinder length="0.65" radius="0.06"/>
@@ -80,5 +42,5 @@
   </link>
   <joint name="upper_arm_collision_joint" type="fixed">
-    <origin rpy="0 0 0" xyz="0 0 0"/>
+    <origin rpy="0 1.5708 0" xyz="-0.325 0 0.18"/>
     <parent link="ur10_arm_upper_arm_link"/>
     <child link="upper_arm_collision_link"/>
@@ -86,12 +48,6 @@
   <!-- Collision sphere for the elbow -->
   <link name="elbow_collision_link">
-    <collision>
-      <origin rpy="0 0 0" xyz="0 0.06 0"/>
-      <geometry>
-        <sphere radius="0.15"/>
-      </geometry>
-    </collision>
     <visual>
-      <origin rpy="0 0 0" xyz="0 0.06 0"/>
+      <origin rpy="0 0 0" xyz="0 0 0"/>
       <geometry>
         <sphere radius="0.15"/>
@@ -101,5 +57,5 @@
   </link>
   <joint name="elbow_collision_joint" type="fixed">
-    <origin rpy="0 0 0" xyz="0 0 0"/>
+    <origin rpy="0 0 0" xyz="0 0 0.12"/>
     <parent link="ur10_arm_forearm_link"/>
     <child link="elbow_collision_link"/>
@@ -107,13 +63,8 @@
   <!-- Collision cylinder for the forearm link -->
   <!-- For use as an end effector (i.e. to compute its position for the dynamic obstacle task), we must specify the origin of the link using the <joint> rather than inside the <link> itself. Otherwise, this should not be done, as it (oddly, and unexpectedly) changes the behaviour. -->
+  <!-- the above is because the origin used for the EE is the joint frame -->
   <link name="forearm_collision_link">
-    <collision>
-      <origin rpy="0 0 0" xyz="0 0 0.3"/>
-      <geometry>
-        <cylinder length="0.6" radius="0.06"/>
-      </geometry>
-    </collision>
     <visual>
-      <origin rpy="0 0 0" xyz="0 0 0.3"/>
+      <origin rpy="0 0 0" xyz="0 0 0"/>
       <geometry>
         <cylinder length="0.6" radius="0.06"/>
@@ -123,5 +74,5 @@
   </link>
   <joint name="forearm_collision_joint" type="fixed">
-    <origin rpy="0 0 0" xyz="0 0 0"/>
+    <origin rpy="0 1.5708 0" xyz="-0.3 0 0.05"/>
     <parent link="ur10_arm_forearm_link"/>
     <child link="forearm_collision_link"/>
@@ -129,10 +80,4 @@
   <!-- Collision sphere for the wrist -->
   <link name="wrist_collision_link">
-    <collision>
-      <origin rpy="0 0 0" xyz="0 0 0"/>
-      <geometry>
-        <sphere radius="0.15"/>
-      </geometry>
-    </collision>
     <visual>
       <origin rpy="0 0 0" xyz="0 0 0"/>
@@ -151,5 +96,5 @@
   <link name="base_collision_link">
     <visual>
-      <origin rpy="0 0 0" xyz="0 0 0.15"/>
+      <origin rpy="0 0 0" xyz="0 0 0"/>
       <geometry>
         <box size="1.0 0.8 0.3"/>
@@ -157,13 +102,7 @@
       <material name="seethrough"/>
     </visual>
-    <collision>
-      <origin rpy="0 0 0" xyz="0 0 0.15"/>
-      <geometry>
-        <box size="1.0 0.8 0.3"/>
-      </geometry>
-    </collision>
   </link>
   <joint name="base_collision_joint" type="fixed">
-    <origin rpy="0 0 0" xyz="0 0 0.01"/>
+    <origin rpy="0 0 0" xyz="0 0 0.16"/>
     <parent link="base_link"/>
     <child link="base_collision_link"/>
@@ -177,13 +116,7 @@
       <material name="seethrough"/>
     </visual>
-    <collision>
-      <origin rpy="0 0 0" xyz="0 0 0"/>
-      <geometry>
-        <sphere radius="0.15"/>
-      </geometry>
-    </collision>
   </link>
   <joint name="forearm_collision_sphere_joint1" type="fixed">
-    <origin rpy="0 0 0" xyz="0 0 0.2"/>
+    <origin rpy="0 1.5708 0" xyz="-0.2 0 0.06"/>
     <parent link="ur10_arm_forearm_link"/>
     <child link="forearm_collision_sphere_link1"/>
@@ -197,15 +130,8 @@
       <material name="seethrough"/>
     </visual>
-    <collision>
-      <origin rpy="0 0 0" xyz="0 0 0"/>
-      <geometry>
-        <sphere radius="0.15"/>
-      </geometry>
-    </collision>
   </link>
   <joint name="forearm_collision_sphere_joint2" type="fixed">
-    <origin rpy="0 0 0" xyz="0 0 0.4"/>
+    <origin rpy="0 1.5708 0" xyz="-0.4 0 0.06"/>
     <parent link="ur10_arm_forearm_link"/>
-    <child link="forearm_collision_sphere_link2"/>
-  </joint>
+    <child link="forearm_collision_sphere_link2"/> </joint>
 </robot>
