Commit message: Static collision avoidance is working

File: upright_assets/thing/xacro/obstacles.urdf.xacro (robot description, xacro)
@@ -113,14 +113,18 @@
   <link name="table3_link">
     <visual>
-      <origin rpy="0 0 0" xyz="3.5 0.0 0.375"/>
-      <geometry>
-        <cylinder length="0.75" radius="0.5"/>
-      </geometry>
-      <material name="table_color"/>
-    </visual>
-    <collision>
-      <origin rpy="0 0 0" xyz="3.5 0.0 0.375"/>
-      <geometry>
-        <cylinder length="0.75" radius="0.5"/>
+      <!-- <origin rpy="0 0 0" xyz="3.5 0.0 0.375"/> -->
+      <origin rpy="0 0 0" xyz="0 0 0"/>
+      <geometry>
+        <cylinder length="0.75" radius="0.5"/>
+        <!-- <sphere radius="0.75"/> -->
+      </geometry>
+      <material name="table_color"/>
+    </visual>
+    <collision>
+      <!-- <origin rpy="0 0 0" xyz="3.5 0.0 0.375"/> -->
+      <origin rpy="0 0 0" xyz="0 0 0"/>
+      <geometry>
+        <cylinder length="0.75" radius="0.5"/>
+        <!-- <sphere radius="0.75"/> -->
       </geometry>
     </collision>
@@ -129,5 +133,6 @@
     <parent link="obstacle_base_link"/>
     <child link="table3_link"/>
-    <origin rpy="0 0 0" xyz="0 0 0"/>
+    <origin rpy="0 0 0" xyz="3.5 0.0 0.375"/>
+    <!-- <origin rpy="0 0 0" xyz="0 0 0"/> -->
   </joint>
   <link name="chair3_1_link">

Commit message: Clean up obstacle constraint code.

File: upright_assets/thing/xacro/obstacles.urdf.xacro (robot description, xacro)
@@ -113,18 +113,14 @@
   <link name="table3_link">
     <visual>
-      <!-- <origin rpy="0 0 0" xyz="3.5 0.0 0.375"/> -->
       <origin rpy="0 0 0" xyz="0 0 0"/>
       <geometry>
         <cylinder length="0.75" radius="0.5"/>
-        <!-- <sphere radius="0.75"/> -->
-      </geometry>
-      <material name="table_color"/>
-    </visual>
-    <collision>
-      <!-- <origin rpy="0 0 0" xyz="3.5 0.0 0.375"/> -->
+      </geometry>
+      <material name="table_color"/>
+    </visual>
+    <collision>
       <origin rpy="0 0 0" xyz="0 0 0"/>
       <geometry>
         <cylinder length="0.75" radius="0.5"/>
-        <!-- <sphere radius="0.75"/> -->
       </geometry>
     </collision>
@@ -134,5 +130,4 @@
     <child link="table3_link"/>
     <origin rpy="0 0 0" xyz="3.5 0.0 0.375"/>
-    <!-- <origin rpy="0 0 0" xyz="0 0 0"/> -->
   </joint>
   <link name="chair3_1_link">
