Commit message: Simulate with calibrated transform.

File: upright_assets/thing/xacro/collision_links.urdf.xacro (robot description, xacro)
@@ -19,5 +19,5 @@
   <joint name="balanced_object_collision_joint" type="fixed">
     <origin rpy="0 0 0" xyz="0 0 0.05"/>
-    <parent link="thing_tool"/>
+    <parent link="gripped_object"/>
     <child link="balanced_object_collision_link"/>
   </joint>

File: upright_assets/thing/xacro/ocs2/thing_ocs2_tray.urdf.xacro (robot description, xacro)
@@ -2,5 +2,6 @@
 <robot name="mm_ocs2_tray" xmlns:xacro="http://www.ros.org/wiki/xacro">
   <xacro:include filename="$(find mobile_manipulation_central)/urdf/xacro/thing_no_wheels.urdf.xacro" />
-  <xacro:include filename="../end_effector_tray.urdf.xacro" />
+  <!-- <xacro:include filename="../end_effector_tray.urdf.xacro" /> -->
+  <xacro:include filename="../end_effector_gripped_object.urdf.xacro" />
   <xacro:include filename="../collision_links.urdf.xacro" />
 </robot>

File: upright_assets/thing/xacro/pyb/thing_pyb_tray.urdf.xacro (robot description, xacro)
@@ -3,5 +3,6 @@
   <xacro:include filename="base_joints.urdf.xacro" />
   <xacro:include filename="$(find mobile_manipulation_central)/urdf/xacro/thing_no_wheels.urdf.xacro" />
-  <xacro:include filename="../end_effector_tray.urdf.xacro" />
+  <!-- <xacro:include filename="../end_effector_tray.urdf.xacro" /> -->
+  <xacro:include filename="../end_effector_gripped_object.urdf.xacro" />
   <xacro:include filename="../visual_collision_links.urdf.xacro" />
 </robot>

File: upright_assets/thing/xacro/visual_collision_links.urdf.xacro (robot description, xacro)
@@ -13,5 +13,5 @@
   <joint name="balanced_object_collision_joint" type="fixed">
     <origin rpy="0 0 0" xyz="0 0 0.05"/>
-    <parent link="thing_tool"/>
+    <parent link="gripped_object"/>
     <child link="balanced_object_collision_link"/>
   </joint>

Commit message: Experiments with static obstacles.

File: upright_assets/thing/xacro/collision_links.urdf.xacro (robot description, xacro)
@@ -23,5 +23,5 @@
     <origin rpy="0 0 0" xyz="0 0 0"/>
     <geometry>
-      <sphere radius="0.2"/>
+      <sphere radius="0.21"/>
     </geometry>
   </xacro:collision_link>
@@ -68,6 +68,5 @@
     <child link="elbow_collision_link"/>
   </joint>
-  <!-- Collision sphere for the wrist -->
-  <xacro:collision_link name="wrist_collision_link">
+  <xacro:collision_link name="wrist1_collision_link">
     <origin rpy="0 0 0" xyz="0 0 0"/>
     <geometry>
@@ -75,8 +74,20 @@
     </geometry>
   </xacro:collision_link>
-  <joint name="wrist_collision_joint" type="fixed">
+  <joint name="wrist1_collision_joint" type="fixed">
+    <origin rpy="0 0 0" xyz="0 0 -0.05"/>
+    <parent link="ur10_arm_wrist_1_link"/>
+    <child link="wrist1_collision_link"/>
+  </joint>
+  <!-- Collision sphere for the wrist -->
+  <xacro:collision_link name="wrist3_collision_link">
+    <origin rpy="0 0 0" xyz="0 0 0"/>
+    <geometry>
+      <sphere radius="0.15"/>
+    </geometry>
+  </xacro:collision_link>
+  <joint name="wrist3_collision_joint" type="fixed">
     <origin rpy="0 0 0" xyz="0 0 0"/>
     <parent link="ur10_arm_wrist_3_link"/>
-    <child link="wrist_collision_link"/>
+    <child link="wrist3_collision_link"/>
   </joint>
   <!-- Collision rectangle for the base -->

File: upright_assets/thing/xacro/obstacles/simple.urdf.xacro (robot description, xacro)
@@ -25,5 +25,5 @@
   <link name="obstacle_base_link"></link>
   <xacro:obstacle_link name="sphere1_link" material="red">
-    <origin rpy="0 0 0" xyz="1.5 0.75 0.25"/>
+    <origin rpy="0 0 0" xyz="0 -1 0.25"/>
     <geometry>
       <sphere radius="0.25"/>
@@ -31,5 +31,5 @@
   </xacro:obstacle_link>
   <xacro:obstacle_link name="sphere2_link" material="red">
-    <origin rpy="0 0 0" xyz="1.5 0.75 0.75"/>
+    <origin rpy="0 0 0" xyz="0 -1 0.75"/>
     <geometry>
       <sphere radius="0.25"/>

Commit message: Dynamic obstacle tuning; resurrect inertial alignment cost/constraint.

File: upright_assets/thing/xacro/collision_links.urdf.xacro (robot description, xacro)
@@ -23,10 +23,10 @@
     <origin rpy="0 0 0" xyz="0 0 0"/>
     <geometry>
-      <sphere radius="0.21"/>
+      <!-- <sphere radius="0.21"/> -->
+      <box size="0.23 0.3 0.2" />
     </geometry>
   </xacro:collision_link>
   <joint name="balanced_object_collision_joint" type="fixed">
-    <!-- <origin rpy="0 0 0" xyz="0 0 0.05"/> -->
-    <origin rpy="0 0 0" xyz="0.1 0.13 0"/>
+    <origin rpy="0 0 0" xyz="0.1 0.13 0.036"/>
     <parent link="gripped_object"/>
     <child link="balanced_object_collision_link"/>

Commit message: Implement relaxed alignment constraint.

File: upright_assets/thing/xacro/collision_links.urdf.xacro (robot description, xacro)
@@ -19,14 +19,26 @@
     </link>
   </xacro:macro>
-  <!-- This configuration is used for the single- and multi-object balancing tasks -->
+  <!-- Original box tray -->
+  <!-- <xacro:collision_link name="balanced_object_collision_link"> -->
+  <!--   <origin rpy="0 0 0" xyz="0 0 0"/> -->
+  <!--   <geometry> -->
+      <!-- <sphere radius="0.21"/> -->
+  <!--     <box size="0.23 0.3 0.2" /> -->
+  <!--   </geometry> -->
+  <!-- </xacro:collision_link> -->
+  <!-- <joint name="balanced_object_collision_joint" type="fixed"> -->
+  <!--   <origin rpy="0 0 0" xyz="0.1 0.13 0.036"/> -->
+  <!--   <parent link="gripped_object"/> -->
+  <!--   <child link="balanced_object_collision_link"/> -->
+  <!-- </joint> -->
+  <!-- New round tray -->
   <xacro:collision_link name="balanced_object_collision_link">
     <origin rpy="0 0 0" xyz="0 0 0"/>
     <geometry>
-      <!-- <sphere radius="0.21"/> -->
-      <box size="0.23 0.3 0.2" />
+      <sphere radius="0.2"/>
     </geometry>
   </xacro:collision_link>
   <joint name="balanced_object_collision_joint" type="fixed">
-    <origin rpy="0 0 0" xyz="0.1 0.13 0.036"/>
+    <origin rpy="0 0 0" xyz="0.09 0.12 0.03"/>
     <parent link="gripped_object"/>
     <child link="balanced_object_collision_link"/>

File: upright_assets/thing/xacro/end_effectors/gripped_object.urdf.xacro (robot description, xacro)
@@ -6,8 +6,14 @@
     <child link="gripped_object"/>
   </joint>
+  <!-- <xacro:macro name="gripped_object_geometry"> -->
+  <!--   <origin rpy="0 0 0" xyz="0.1 0.13 -0.032"/> -->
+  <!--   <geometry> -->
+  <!--     <box size="0.23 0.3 0.064" /> -->
+  <!--   </geometry> -->
+  <!-- </xacro:macro> -->
   <xacro:macro name="gripped_object_geometry">
-    <origin rpy="0 0 0" xyz="0.1 0.13 -0.032"/>
+    <origin rpy="0 0 0" xyz="0.09 0.12 -0.035"/>
     <geometry>
-      <box size="0.23 0.3 0.064" />
+      <cylinder length="0.01" radius="0.178" />
     </geometry>
   </xacro:macro>

Commit message: Revise obstacles and poses for experiments.

File: upright_assets/thing/xacro/collision_links.urdf.xacro (robot description, xacro)
@@ -57,15 +57,15 @@
   </joint>
   <!-- Collision cylinder for the upper arm link -->
-  <xacro:collision_link name="upper_arm_collision_link">
-    <origin rpy="0 0 0" xyz="0 0 0"/>
-    <geometry>
-      <cylinder length="0.65" radius="0.06"/>
-    </geometry>
-  </xacro:collision_link>
-  <joint name="upper_arm_collision_joint" type="fixed">
-    <origin rpy="0 1.5708 0" xyz="-0.325 0 0.18"/>
-    <parent link="ur10_arm_upper_arm_link"/>
-    <child link="upper_arm_collision_link"/>
-  </joint>
+  <!-- <xacro:collision_link name="upper_arm_collision_link"> -->
+  <!--   <origin rpy="0 0 0" xyz="0 0 0"/> -->
+  <!--   <geometry> -->
+  <!--     <cylinder length="0.65" radius="0.06"/> -->
+  <!--   </geometry> -->
+  <!-- </xacro:collision_link> -->
+  <!-- <joint name="upper_arm_collision_joint" type="fixed"> -->
+  <!--   <origin rpy="0 1.5708 0" xyz="-0.325 0 0.18"/> -->
+  <!--   <parent link="ur10_arm_upper_arm_link"/> -->
+  <!--   <child link="upper_arm_collision_link"/> -->
+  <!-- </joint> -->
   <!-- Collision sphere for the elbow -->
   <xacro:collision_link name="elbow_collision_link">
@@ -103,28 +103,30 @@
     <child link="wrist3_collision_link"/>
   </joint>
-  <!-- Collision rectangle for the base -->
+  <!-- Collision sphere for the base -->
   <xacro:collision_link name="base_collision_link">
     <origin rpy="0 0 0" xyz="0 0 0"/>
     <geometry>
-      <box size="1.0 0.8 0.3"/>
+      <!-- <box size="1.0 0.8 0.3"/> -->
+      <sphere radius="0.5"/>
     </geometry>
   </xacro:collision_link>
   <joint name="base_collision_joint" type="fixed">
-    <origin rpy="0 0 0" xyz="0 0 0.16"/>
+    <!-- <origin rpy="0 0 0" xyz="0 0 0.16"/> -->
+    <origin rpy="0 0 0" xyz="0 0 0"/>
     <parent link="base_link"/>
     <child link="base_collision_link"/>
   </joint>
   <!-- Collision cylinder for the forearm link -->
-  <xacro:collision_link name="forearm_collision_link">
-    <origin rpy="0 0 0" xyz="0 0 0"/>
-    <geometry>
-      <cylinder length="0.6" radius="0.06"/>
-    </geometry>
-  </xacro:collision_link>
-  <joint name="forearm_collision_joint" type="fixed">
-    <origin rpy="0 1.5708 0" xyz="-0.3 0 0.05"/>
-    <parent link="ur10_arm_forearm_link"/>
-    <child link="forearm_collision_link"/>
-  </joint>
+  <!-- <xacro:collision_link name="forearm_collision_link"> -->
+  <!--   <origin rpy="0 0 0" xyz="0 0 0"/> -->
+  <!--   <geometry> -->
+  <!--     <cylinder length="0.6" radius="0.06"/> -->
+  <!--   </geometry> -->
+  <!-- </xacro:collision_link> -->
+  <!-- <joint name="forearm_collision_joint" type="fixed"> -->
+  <!--   <origin rpy="0 1.5708 0" xyz="-0.3 0 0.05"/> -->
+  <!--   <parent link="ur10_arm_forearm_link"/> -->
+  <!--   <child link="forearm_collision_link"/> -->
+  <!-- </joint> -->
   <!-- Alternatively we can use collision spheres -->
   <xacro:collision_link name="forearm_collision_sphere_link1">

File: upright_assets/thing/xacro/obstacles/simple.urdf.xacro (robot description, xacro)
@@ -24,12 +24,37 @@
   </xacro:macro>
   <link name="obstacle_base_link"></link>
-  <xacro:obstacle_link name="sphere1_link" material="red">
-    <origin rpy="0 0 0" xyz="0 -1 0.25"/>
+  <!-- IMPORTANT: collision avoidance is much more numerically stable for the solver when the collision objects are spheres. Make everything a sphere! -->
+  <xacro:obstacle_link name="sphere1_bottom_link" material="red">
+    <origin rpy="0 0 0" xyz="-1 -0.75 0.25"/>
     <geometry>
       <sphere radius="0.25"/>
     </geometry>
   </xacro:obstacle_link>
-  <xacro:obstacle_link name="sphere2_link" material="red">
-    <origin rpy="0 0 0" xyz="0 -1 0.75"/>
+  <xacro:obstacle_link name="sphere1_top_link" material="red">
+    <origin rpy="0 0 0" xyz="-1 -0.75 0.75"/>
+    <geometry>
+      <sphere radius="0.25"/>
+    </geometry>
+  </xacro:obstacle_link>
+  <xacro:obstacle_link name="sphere2_bottom_link" material="red">
+    <origin rpy="0 0 0" xyz="0.5 0 0.25"/>
+    <geometry>
+      <sphere radius="0.25"/>
+    </geometry>
+  </xacro:obstacle_link>
+  <xacro:obstacle_link name="sphere2_top_link" material="red">
+    <origin rpy="0 0 0" xyz="0.5 0 0.75"/>
+    <geometry>
+      <sphere radius="0.25"/>
+    </geometry>
+  </xacro:obstacle_link>
+  <xacro:obstacle_link name="sphere3_bottom_link" material="red">
+    <origin rpy="0 0 0" xyz="-1.5 1 0.25"/>
+    <geometry>
+      <sphere radius="0.25"/>
+    </geometry>
+  </xacro:obstacle_link>
+  <xacro:obstacle_link name="sphere3_top_link" material="red">
+    <origin rpy="0 0 0" xyz="-1.5 1 0.75"/>
     <geometry>
       <sphere radius="0.25"/>

Commit message: A lot of config for experiments.

File: upright_assets/thing/xacro/collision_links.urdf.xacro (robot description, xacro)
@@ -19,5 +19,5 @@
     </link>
   </xacro:macro>
-  <!-- Original box tray -->
+  <!-- Box tray -->
   <!-- <xacro:collision_link name="balanced_object_collision_link"> -->
   <!--   <origin rpy="0 0 0" xyz="0 0 0"/> -->
@@ -32,13 +32,25 @@
   <!--   <child link="balanced_object_collision_link"/> -->
   <!-- </joint> -->
-  <!-- New round tray -->
+  <!-- Restaurant tray -->
+  <!-- <xacro:collision_link name="balanced_object_collision_link"> -->
+  <!--   <origin rpy="0 0 0" xyz="0 0 0"/> -->
+  <!--   <geometry> -->
+  <!--     <sphere radius="0.2"/> -->
+  <!--   </geometry> -->
+  <!-- </xacro:collision_link> -->
+  <!-- <joint name="balanced_object_collision_joint" type="fixed"> -->
+  <!--   <origin rpy="0 0 0" xyz="0.09 0.12 0.03"/> -->
+  <!--   <parent link="gripped_object"/> -->
+  <!--   <child link="balanced_object_collision_link"/> -->
+  <!-- </joint> -->
+  <!-- Wood tray -->
   <xacro:collision_link name="balanced_object_collision_link">
     <origin rpy="0 0 0" xyz="0 0 0"/>
     <geometry>
-      <sphere radius="0.2"/>
+      <sphere radius="0.21"/>
     </geometry>
   </xacro:collision_link>
   <joint name="balanced_object_collision_joint" type="fixed">
-    <origin rpy="0 0 0" xyz="0.09 0.12 0.03"/>
+    <origin rpy="0 0 0" xyz="0 0 0.02"/>
     <parent link="gripped_object"/>
     <child link="balanced_object_collision_link"/>

File: upright_assets/thing/xacro/end_effectors/gripped_object.urdf.xacro (robot description, xacro)
@@ -6,4 +6,12 @@
     <child link="gripped_object"/>
   </joint>
+  <!-- Wood tray -->
+  <xacro:macro name="gripped_object_geometry">
+    <origin rpy="0 0 0" xyz="0 0 -0.01"/>
+    <geometry>
+      <box size="0.285 0.285 0.02" />
+    </geometry>
+  </xacro:macro>
+  <!-- Box tray -->
   <!-- <xacro:macro name="gripped_object_geometry"> -->
   <!--   <origin rpy="0 0 0" xyz="0.1 0.13 -0.032"/> -->
@@ -12,10 +20,11 @@
   <!--   </geometry> -->
   <!-- </xacro:macro> -->
-  <xacro:macro name="gripped_object_geometry">
-    <origin rpy="0 0 0" xyz="0.064 0.127 -0.005"/>
-    <geometry>
-      <cylinder length="0.01" radius="0.178" />
-    </geometry>
-  </xacro:macro>
+  <!-- Restaurant tray -->
+  <!-- <xacro:macro name="gripped_object_geometry"> -->
+  <!--   <origin rpy="0 0 0" xyz="0.064 0.127 -0.005"/> -->
+  <!--   <geometry> -->
+  <!--     <cylinder length="0.01" radius="0.178" /> -->
+  <!--   </geometry> -->
+  <!-- </xacro:macro> -->
   <!-- Extra link for the gripped object, which must be calibrated. -->
   <link name="gripped_object">

File: upright_assets/thing/xacro/obstacles/simple.urdf.xacro (robot description, xacro)
@@ -26,5 +26,5 @@
   <!-- IMPORTANT: collision avoidance is much more numerically stable for the solver when the collision objects are spheres. Make everything a sphere! -->
   <xacro:obstacle_link name="sphere1_bottom_link" material="red">
-    <origin rpy="0 0 0" xyz="0 -0.75 0.25"/>
+    <origin rpy="0 0 0" xyz="0 0.25 0.25"/>
     <geometry>
       <sphere radius="0.25"/>
@@ -32,5 +32,5 @@
   </xacro:obstacle_link>
   <xacro:obstacle_link name="sphere1_top_link" material="red">
-    <origin rpy="0 0 0" xyz="0 -0.75 0.75"/>
+    <origin rpy="0 0 0" xyz="0 0.25 0.75"/>
     <geometry>
       <sphere radius="0.25"/>
@@ -38,5 +38,5 @@
   </xacro:obstacle_link>
   <xacro:obstacle_link name="sphere2_bottom_link" material="red">
-    <origin rpy="0 0 0" xyz="1.5 0 0.25"/>
+    <origin rpy="0 0 0" xyz="1.5 1 0.25"/>
     <geometry>
       <sphere radius="0.25"/>
@@ -44,5 +44,5 @@
   </xacro:obstacle_link>
   <xacro:obstacle_link name="sphere2_top_link" material="red">
-    <origin rpy="0 0 0" xyz="1.5 0 0.75"/>
+    <origin rpy="0 0 0" xyz="1.5 1 0.75"/>
     <geometry>
       <sphere radius="0.25"/>
@@ -50,5 +50,5 @@
   </xacro:obstacle_link>
   <xacro:obstacle_link name="sphere3_bottom_link" material="red">
-    <origin rpy="0 0 0" xyz="-0.5 1 0.25"/>
+    <origin rpy="0 0 0" xyz="-0.5 2 0.25"/>
     <geometry>
       <sphere radius="0.25"/>
@@ -56,5 +56,5 @@
   </xacro:obstacle_link>
   <xacro:obstacle_link name="sphere3_top_link" material="red">
-    <origin rpy="0 0 0" xyz="-0.5 1 0.75"/>
+    <origin rpy="0 0 0" xyz="-0.5 2 0.75"/>
     <geometry>
       <sphere radius="0.25"/>
@@ -62,5 +62,5 @@
   </xacro:obstacle_link>
   <xacro:obstacle_link name="sphere3_middle_link" material="red">
-    <origin rpy="0 0 0" xyz="-0.5 1 0.5"/>
+    <origin rpy="0 0 0" xyz="-0.5 2 0.5"/>
     <geometry>
       <sphere radius="0.25"/>

Commit message: Tune projectile avoidance.

File: upright_assets/thing/xacro/collision_links.urdf.xacro (robot description, xacro)
@@ -19,34 +19,10 @@
     </link>
   </xacro:macro>
-  <!-- Box tray -->
-  <!-- <xacro:collision_link name="balanced_object_collision_link"> -->
-  <!--   <origin rpy="0 0 0" xyz="0 0 0"/> -->
-  <!--   <geometry> -->
-      <!-- <sphere radius="0.21"/> -->
-  <!--     <box size="0.23 0.3 0.2" /> -->
-  <!--   </geometry> -->
-  <!-- </xacro:collision_link> -->
-  <!-- <joint name="balanced_object_collision_joint" type="fixed"> -->
-  <!--   <origin rpy="0 0 0" xyz="0.1 0.13 0.036"/> -->
-  <!--   <parent link="gripped_object"/> -->
-  <!--   <child link="balanced_object_collision_link"/> -->
-  <!-- </joint> -->
-  <!-- Restaurant tray -->
-  <!-- <xacro:collision_link name="balanced_object_collision_link"> -->
-  <!--   <origin rpy="0 0 0" xyz="0 0 0"/> -->
-  <!--   <geometry> -->
-  <!--     <sphere radius="0.2"/> -->
-  <!--   </geometry> -->
-  <!-- </xacro:collision_link> -->
-  <!-- <joint name="balanced_object_collision_joint" type="fixed"> -->
-  <!--   <origin rpy="0 0 0" xyz="0.09 0.12 0.03"/> -->
-  <!--   <parent link="gripped_object"/> -->
-  <!--   <child link="balanced_object_collision_link"/> -->
-  <!-- </joint> -->
   <!-- Wood tray -->
   <xacro:collision_link name="balanced_object_collision_link">
-    <origin rpy="0 0 0" xyz="0 0 0"/>
+    <origin rpy="0 0 0" xyz="0 0 0.05"/>
     <geometry>
-      <sphere radius="0.21"/>
+      <!-- <sphere radius="0.21"/> -->
+      <sphere radius="0.25"/>
     </geometry>
   </xacro:collision_link>
@@ -56,4 +32,15 @@
     <child link="balanced_object_collision_link"/>
   </joint>
+  <!-- <xacro:collision_link name="balanced_object_collision_link_large"> -->
+  <!--   <origin rpy="0 0 0" xyz="0 0 0"/> -->
+  <!--   <geometry> -->
+  <!--     <sphere radius="0.36"/> -->
+  <!--   </geometry> -->
+  <!-- </xacro:collision_link> -->
+  <!-- <joint name="balanced_object_collision_joint_large" type="fixed"> -->
+  <!--   <origin rpy="0 0 0" xyz="0 0 0.02"/> -->
+  <!--   <parent link="gripped_object"/> -->
+  <!--   <child link="balanced_object_collision_link_large"/> -->
+  <!-- </joint> -->
   <!-- Collision sphere for the shoulder -->
   <xacro:collision_link name="shoulder_collision_link">

Commit message: Fix offset of object collision sphere.
All offsets are specified in the joint rather than the link (which this
was not before).

File: upright_assets/thing/xacro/collision_links.urdf.xacro (robot description, xacro)
@@ -21,5 +21,5 @@
   <!-- Wood tray -->
   <xacro:collision_link name="balanced_object_collision_link">
-    <origin rpy="0 0 0" xyz="0 0 0.05"/>
+    <origin rpy="0 0 0" xyz="0 0 0"/>
     <geometry>
       <!-- <sphere radius="0.21"/> -->
@@ -28,5 +28,5 @@
   </xacro:collision_link>
   <joint name="balanced_object_collision_joint" type="fixed">
-    <origin rpy="0 0 0" xyz="0 0 0.02"/>
+    <origin rpy="0 0 0" xyz="0 0 0.07"/>
     <parent link="gripped_object"/>
     <child link="balanced_object_collision_link"/>

Commit message: Organize paper simulation code.

File: upright_assets/thing/xacro/collision_links.urdf.xacro (robot description, xacro)
@@ -3,5 +3,8 @@
   <!-- Set false to not include <collision> blocks, which is useful if we just want to visualize in a simulator. -->
   <xacro:arg name="use_collision" default="true"/>
-  <xacro:property name="material" value="seethrough"/>
+  <material name="obstacle_material">
+    <color rgba="1.0 0.0 0.0 0.25"/>
+  </material>
+  <xacro:property name="material" value="obstacle_material"/>
   <xacro:macro name="collision_link" params="name *origin *geometry">
     <link name="${name}">
@@ -32,15 +35,4 @@
     <child link="balanced_object_collision_link"/>
   </joint>
-  <!-- <xacro:collision_link name="balanced_object_collision_link_large"> -->
-  <!--   <origin rpy="0 0 0" xyz="0 0 0"/> -->
-  <!--   <geometry> -->
-  <!--     <sphere radius="0.36"/> -->
-  <!--   </geometry> -->
-  <!-- </xacro:collision_link> -->
-  <!-- <joint name="balanced_object_collision_joint_large" type="fixed"> -->
-  <!--   <origin rpy="0 0 0" xyz="0 0 0.02"/> -->
-  <!--   <parent link="gripped_object"/> -->
-  <!--   <child link="balanced_object_collision_link_large"/> -->
-  <!-- </joint> -->
   <!-- Collision sphere for the shoulder -->
   <xacro:collision_link name="shoulder_collision_link">
@@ -55,28 +47,16 @@
     <child link="shoulder_collision_link"/>
   </joint>
-  <!-- Collision cylinder for the upper arm link -->
-  <!-- <xacro:collision_link name="upper_arm_collision_link"> -->
+  <!-- Collision sphere for the elbow -->
+  <!-- <xacro:collision_link name="elbow_collision_link"> -->
   <!--   <origin rpy="0 0 0" xyz="0 0 0"/> -->
   <!--   <geometry> -->
-  <!--     <cylinder length="0.65" radius="0.06"/> -->
+  <!--     <sphere radius="0.15"/> -->
   <!--   </geometry> -->
   <!-- </xacro:collision_link> -->
-  <!-- <joint name="upper_arm_collision_joint" type="fixed"> -->
-  <!--   <origin rpy="0 1.5708 0" xyz="-0.325 0 0.18"/> -->
-  <!--   <parent link="ur10_arm_upper_arm_link"/> -->
-  <!--   <child link="upper_arm_collision_link"/> -->
+  <!-- <joint name="elbow_collision_joint" type="fixed"> -->
+  <!--   <origin rpy="0 0 0" xyz="0 0 0.12"/> -->
+  <!--   <parent link="ur10_arm_forearm_link"/> -->
+  <!--   <child link="elbow_collision_link"/> -->
   <!-- </joint> -->
-  <!-- Collision sphere for the elbow -->
-  <xacro:collision_link name="elbow_collision_link">
-    <origin rpy="0 0 0" xyz="0 0 0"/>
-    <geometry>
-      <sphere radius="0.15"/>
-    </geometry>
-  </xacro:collision_link>
-  <joint name="elbow_collision_joint" type="fixed">
-    <origin rpy="0 0 0" xyz="0 0 0.12"/>
-    <parent link="ur10_arm_forearm_link"/>
-    <child link="elbow_collision_link"/>
-  </joint>
   <xacro:collision_link name="wrist1_collision_link">
     <origin rpy="0 0 0" xyz="0 0 0"/>
@@ -116,17 +96,4 @@
     <child link="base_collision_link"/>
   </joint>
-  <!-- Collision cylinder for the forearm link -->
-  <!-- <xacro:collision_link name="forearm_collision_link"> -->
-  <!--   <origin rpy="0 0 0" xyz="0 0 0"/> -->
-  <!--   <geometry> -->
-  <!--     <cylinder length="0.6" radius="0.06"/> -->
-  <!--   </geometry> -->
-  <!-- </xacro:collision_link> -->
-  <!-- <joint name="forearm_collision_joint" type="fixed"> -->
-  <!--   <origin rpy="0 1.5708 0" xyz="-0.3 0 0.05"/> -->
-  <!--   <parent link="ur10_arm_forearm_link"/> -->
-  <!--   <child link="forearm_collision_link"/> -->
-  <!-- </joint> -->
-  <!-- Alternatively we can use collision spheres -->
   <xacro:collision_link name="forearm_collision_sphere_link1">
     <origin rpy="0 0 0" xyz="0 0 0"/>

File: upright_assets/thing/xacro/obstacles/simple.urdf.xacro (robot description, xacro)
@@ -2,5 +2,5 @@
 <robot name="obstacles" xmlns:xacro="http://wiki.ros.org/xacro">
   <material name="red">
-    <color rgba="1.0 0.0 0.0 1.0"/>
+    <color rgba="0.0 0.0 1.0 1.0"/>
   </material>
   <!-- It is convenient to use a macro to avoid accidental mismatches between visual and collision geometry -->
