Commit message: WIP: projectile waypoint planning logic

File: upright_assets/thing/xacro/collision_links.urdf.xacro (robot description, xacro)
@@ -46,4 +46,15 @@
     <parent link="ur10_arm_upper_arm_link"/>
     <child link="shoulder_collision_link"/>
+  </joint>
+  <xacro:collision_link name="upper_arm_collision_link1">
+    <origin rpy="0 0 0" xyz="0 0 0"/>
+    <geometry>
+      <sphere radius="0.15"/>
+    </geometry>
+  </xacro:collision_link>
+  <joint name="upper_arm_collision_joint1" type="fixed">
+    <origin rpy="0 0 0" xyz="0 0 0.2"/>
+    <parent link="ur10_arm_upper_arm_link"/>
+    <child link="upper_arm_collision_link1"/>
   </joint>
   <!-- Collision sphere for the elbow -->

Commit message: Tuning and generalizing the projectile path constraints.

File: upright_assets/thing/xacro/collision_links.urdf.xacro (robot description, xacro)
@@ -32,7 +32,20 @@
   <joint name="balanced_object_collision_joint" type="fixed">
     <origin rpy="0 0 0" xyz="0 0 0.07"/>
+    <!-- <origin rpy="0 0 0" xyz="0 0 0"/> -->
     <parent link="gripped_object"/>
     <child link="balanced_object_collision_link"/>
   </joint>
+  <!-- Extra collision link for just the bottle. -->
+  <!-- <xacro:collision_link name="bottle_collision_link"> -->
+  <!--   <origin rpy="0 0 0" xyz="0 0 0"/> -->
+  <!--   <geometry> -->
+  <!--     <sphere radius="0.10"/> -->
+  <!--   </geometry> -->
+  <!-- </xacro:collision_link> -->
+  <!-- <joint name="bottle_collision_joint" type="fixed"> -->
+  <!--   <origin rpy="0 0 0" xyz="0.035 -0.035 0.2"/> -->
+  <!--   <parent link="gripped_object"/> -->
+  <!--   <child link="bottle_collision_link"/> -->
+  <!-- </joint> -->
   <!-- Collision sphere for the shoulder -->
   <xacro:collision_link name="shoulder_collision_link">

Commit message: A bit of clean up.

File: upright_assets/thing/xacro/collision_links.urdf.xacro (robot description, xacro)
@@ -5,4 +5,5 @@
   <material name="obstacle_material">
     <color rgba="1.0 0.0 0.0 0.25"/>
+    <!-- <color rgba="1.0 0.0 0.0 1.0"/> -->
   </material>
   <xacro:property name="material" value="obstacle_material"/>
@@ -60,15 +61,37 @@
     <child link="shoulder_collision_link"/>
   </joint>
-  <xacro:collision_link name="upper_arm_collision_link1">
-    <origin rpy="0 0 0" xyz="0 0 0"/>
-    <geometry>
-      <sphere radius="0.15"/>
-    </geometry>
-  </xacro:collision_link>
-  <joint name="upper_arm_collision_joint1" type="fixed">
-    <origin rpy="0 0 0" xyz="0 0 0.2"/>
-    <parent link="ur10_arm_upper_arm_link"/>
-    <child link="upper_arm_collision_link1"/>
-  </joint>
+  <!-- <xacro:collision_link name="upper_arm_collision_link1"> -->
+  <!--   <origin rpy="0 0 0" xyz="0 0 0"/> -->
+  <!--   <geometry> -->
+  <!--     <sphere radius="0.1"/> -->
+  <!--   </geometry> -->
+  <!-- </xacro:collision_link> -->
+  <!-- <joint name="upper_arm_collision_joint1" type="fixed"> -->
+  <!--   <origin rpy="0 0 0" xyz="0 0 0.2"/> -->
+  <!--   <parent link="ur10_arm_upper_arm_link"/> -->
+  <!--   <child link="upper_arm_collision_link1"/> -->
+  <!-- </joint> -->
+  <!-- <xacro:collision_link name="upper_arm_collision_link2"> -->
+  <!--   <origin rpy="0 0 0" xyz="0 0 0"/> -->
+  <!--   <geometry> -->
+  <!--     <sphere radius="0.1"/> -->
+  <!--   </geometry> -->
+  <!-- </xacro:collision_link> -->
+  <!-- <joint name="upper_arm_collision_joint2" type="fixed"> -->
+  <!--   <origin rpy="0 0 0" xyz="-0.2 0 0.2"/> -->
+  <!--   <parent link="ur10_arm_upper_arm_link"/> -->
+  <!--   <child link="upper_arm_collision_link2"/> -->
+  <!-- </joint> -->
+  <!-- <xacro:collision_link name="upper_arm_collision_link3"> -->
+  <!--   <origin rpy="0 0 0" xyz="0 0 0"/> -->
+  <!--   <geometry> -->
+  <!--     <sphere radius="0.1"/> -->
+  <!--   </geometry> -->
+  <!-- </xacro:collision_link> -->
+  <!-- <joint name="upper_arm_collision_joint3" type="fixed"> -->
+  <!--   <origin rpy="0 0 0" xyz="-0.4 0 0.2"/> -->
+  <!--   <parent link="ur10_arm_upper_arm_link"/> -->
+  <!--   <child link="upper_arm_collision_link3"/> -->
+  <!-- </joint> -->
   <!-- Collision sphere for the elbow -->
   <!-- <xacro:collision_link name="elbow_collision_link"> -->

File: upright_assets/thing/xacro/obstacles/simple.urdf.xacro (robot description, xacro)
@@ -3,4 +3,7 @@
   <material name="red">
     <color rgba="0.0 0.0 1.0 1.0"/>
+  </material>
+  <material name="green">
+    <color rgba="0.0 1.0 0.0 1.0"/>
   </material>
   <!-- It is convenient to use a macro to avoid accidental mismatches between visual and collision geometry -->
@@ -24,4 +27,11 @@
   </xacro:macro>
   <link name="obstacle_base_link"></link>
+  <!-- For the experimental setup figure. -->
+  <!-- <xacro:obstacle_link name="sudden_obstacle_link" material="green"> -->
+  <!--   <origin rpy="0 0 0" xyz="1.25 1.5 0.25"/> -->
+  <!--   <geometry> -->
+  <!--     <sphere radius="0.25"/> -->
+  <!--   </geometry> -->
+  <!-- </xacro:obstacle_link> -->
   <!-- IMPORTANT: collision avoidance is much more numerically stable for the solver when the collision objects are spheres. Make everything a sphere! -->
   <xacro:obstacle_link name="sphere1_bottom_link" material="red">
