Commit message: Clean up obstacle constraints.

File: upright_assets/thing/xacro/obstacles/simple.urdf.xacro (robot description, xacro)
@@ -4,29 +4,35 @@
     <color rgba="1.0 0.0 0.0 1.0"/>
   </material>
-  <!-- It is convenient to use a macro to avoid mismatches accidental between visual and collision geometry -->
+  <!-- It is convenient to use a macro to avoid accidental mismatches between visual and collision geometry -->
   <xacro:macro name="obstacle_link" params="name material *origin *geometry">
     <link name="${name}">
       <collision>
-        <xacro:insert_block name="origin" />
+        <origin rpy="0 0 0" xyz="0 0 0"/>
         <xacro:insert_block name="geometry" />
       </collision>
       <visual>
-        <xacro:insert_block name="origin" />
+        <origin rpy="0 0 0" xyz="0 0 0"/>
         <xacro:insert_block name="geometry" />
         <material name="${material}"/>
       </visual>
     </link>
+    <joint name="${name}_joint" type="fixed">
+      <parent link="obstacle_base_link"/>
+      <child link="${name}"/>
+      <xacro:insert_block name="origin" />
+    </joint>
   </xacro:macro>
   <link name="obstacle_base_link"></link>
   <xacro:obstacle_link name="sphere1_link" material="red">
-    <origin rpy="0 0 0" xyz="0 0 0"/>
+    <origin rpy="0 0 0" xyz="1.5 0.75 0.25"/>
     <geometry>
-      <sphere radius="0.5"/>
+      <sphere radius="0.25"/>
     </geometry>
   </xacro:obstacle_link>
-  <joint name="table1_link_joint" type="fixed">
-    <parent link="obstacle_base_link"/>
-    <child link="sphere1_link"/>
-    <origin rpy="0 0 0" xyz="1.5 1.0 0.375"/>
-  </joint>
+  <xacro:obstacle_link name="sphere2_link" material="red">
+    <origin rpy="0 0 0" xyz="1.5 0.75 0.75"/>
+    <geometry>
+      <sphere radius="0.25"/>
+    </geometry>
+  </xacro:obstacle_link>
 </robot>

Commit message: Start configs for experiments; implement base pose for fixed base.

File: upright_assets/thing/xacro/obstacles/simple.urdf.xacro (robot description, xacro)
@@ -61,3 +61,9 @@
     </geometry>
   </xacro:obstacle_link>
+  <xacro:obstacle_link name="sphere3_middle_link" material="red">
+    <origin rpy="0 0 0" xyz="-1.5 1 0.5"/>
+    <geometry>
+      <sphere radius="0.25"/>
+    </geometry>
+  </xacro:obstacle_link>
 </robot>

Commit message: Adjust starting point of base to (x, y) = (-1, 0)

File: upright_assets/thing/xacro/obstacles/simple.urdf.xacro (robot description, xacro)
@@ -26,5 +26,5 @@
   <!-- IMPORTANT: collision avoidance is much more numerically stable for the solver when the collision objects are spheres. Make everything a sphere! -->
   <xacro:obstacle_link name="sphere1_bottom_link" material="red">
-    <origin rpy="0 0 0" xyz="-1 -0.75 0.25"/>
+    <origin rpy="0 0 0" xyz="0 -0.75 0.25"/>
     <geometry>
       <sphere radius="0.25"/>
@@ -32,5 +32,5 @@
   </xacro:obstacle_link>
   <xacro:obstacle_link name="sphere1_top_link" material="red">
-    <origin rpy="0 0 0" xyz="-1 -0.75 0.75"/>
+    <origin rpy="0 0 0" xyz="0 -0.75 0.75"/>
     <geometry>
       <sphere radius="0.25"/>
@@ -38,5 +38,5 @@
   </xacro:obstacle_link>
   <xacro:obstacle_link name="sphere2_bottom_link" material="red">
-    <origin rpy="0 0 0" xyz="0.5 0 0.25"/>
+    <origin rpy="0 0 0" xyz="1.5 0 0.25"/>
     <geometry>
       <sphere radius="0.25"/>
@@ -44,5 +44,5 @@
   </xacro:obstacle_link>
   <xacro:obstacle_link name="sphere2_top_link" material="red">
-    <origin rpy="0 0 0" xyz="0.5 0 0.75"/>
+    <origin rpy="0 0 0" xyz="1.5 0 0.75"/>
     <geometry>
       <sphere radius="0.25"/>
@@ -50,5 +50,5 @@
   </xacro:obstacle_link>
   <xacro:obstacle_link name="sphere3_bottom_link" material="red">
-    <origin rpy="0 0 0" xyz="-1.5 1 0.25"/>
+    <origin rpy="0 0 0" xyz="-0.5 1 0.25"/>
     <geometry>
       <sphere radius="0.25"/>
@@ -56,5 +56,5 @@
   </xacro:obstacle_link>
   <xacro:obstacle_link name="sphere3_top_link" material="red">
-    <origin rpy="0 0 0" xyz="-1.5 1 0.75"/>
+    <origin rpy="0 0 0" xyz="-0.5 1 0.75"/>
     <geometry>
       <sphere radius="0.25"/>
@@ -62,5 +62,5 @@
   </xacro:obstacle_link>
   <xacro:obstacle_link name="sphere3_middle_link" material="red">
-    <origin rpy="0 0 0" xyz="-1.5 1 0.5"/>
+    <origin rpy="0 0 0" xyz="-0.5 1 0.5"/>
     <geometry>
       <sphere radius="0.25"/>

Commit message: Adjust some experiment parameters.

File: upright_assets/thing/xacro/obstacles/simple.urdf.xacro (robot description, xacro)
@@ -37,6 +37,18 @@
     </geometry>
   </xacro:obstacle_link>
+  <xacro:obstacle_link name="sphere1_middle_link" material="red">
+    <origin rpy="0 0 0" xyz="0 0.25 0.5"/>
+    <geometry>
+      <sphere radius="0.25"/>
+    </geometry>
+  </xacro:obstacle_link>
   <xacro:obstacle_link name="sphere2_bottom_link" material="red">
     <origin rpy="0 0 0" xyz="1.5 1 0.25"/>
+    <geometry>
+      <sphere radius="0.25"/>
+    </geometry>
+  </xacro:obstacle_link>
+  <xacro:obstacle_link name="sphere2_middle_link" material="red">
+    <origin rpy="0 0 0" xyz="1.5 1 0.5"/>
     <geometry>
       <sphere radius="0.25"/>
