Commit message: Implement Ridgeback-only configuration.
More generally, there is now the ability to lock artitrary arm joints.

File: upright_assets/thing/xacro/end_effectors/gripped_object.urdf.xacro (robot description, xacro)
@@ -13,5 +13,5 @@
   <!-- </xacro:macro> -->
   <xacro:macro name="gripped_object_geometry">
-    <origin rpy="0 0 0" xyz="0.09 0.12 -0.035"/>
+    <origin rpy="0 0 0" xyz="0.09 0.115 -0.035"/>
     <geometry>
       <cylinder length="0.01" radius="0.178" />

Commit message: Improve calibration, add more config options for tracking.

File: upright_assets/thing/xacro/end_effectors/gripped_object.urdf.xacro (robot description, xacro)
@@ -13,5 +13,5 @@
   <!-- </xacro:macro> -->
   <xacro:macro name="gripped_object_geometry">
-    <origin rpy="0 0 0" xyz="0.09 0.115 -0.035"/>
+    <origin rpy="0 0 0" xyz="0.064 0.127 -0.005"/>
     <geometry>
       <cylinder length="0.01" radius="0.178" />

Commit message: More descriptive names for calibrated transforms.

File: upright_assets/thing/xacro/end_effectors/gripped_object.urdf.xacro (robot description, xacro)
@@ -2,5 +2,5 @@
 <robot name="end_effector_gripped_object" xmlns:xacro="http://wiki.ros.org/xacro">
   <joint name="gripped_object_joint" type="fixed">
-    <xacro:transformed_origin name="T2" />
+    <xacro:transformed_origin name="ee_to_tray_transform" />
     <parent link="gripper"/>
     <child link="gripped_object"/>
@@ -13,18 +13,4 @@
     </geometry>
   </xacro:macro>
-  <!-- Box tray -->
-  <!-- <xacro:macro name="gripped_object_geometry"> -->
-  <!--   <origin rpy="0 0 0" xyz="0.1 0.13 -0.032"/> -->
-  <!--   <geometry> -->
-  <!--     <box size="0.23 0.3 0.064" /> -->
-  <!--   </geometry> -->
-  <!-- </xacro:macro> -->
-  <!-- Restaurant tray -->
-  <!-- <xacro:macro name="gripped_object_geometry"> -->
-  <!--   <origin rpy="0 0 0" xyz="0.064 0.127 -0.005"/> -->
-  <!--   <geometry> -->
-  <!--     <cylinder length="0.01" radius="0.178" /> -->
-  <!--   </geometry> -->
-  <!-- </xacro:macro> -->
   <!-- Extra link for the gripped object, which must be calibrated. -->
   <link name="gripped_object">

Commit message: Rename ee_to_tray_transform -> gripped_object_transform.
This is a generic name that matches the underlying infrastructure in
mobile_manipulation_central.

Also changed the recompile_libraries option to true, as it is confusing
when things don't work because it's false and you don't remember this is
the case.

File: upright_assets/thing/xacro/end_effectors/gripped_object.urdf.xacro (robot description, xacro)
@@ -2,5 +2,5 @@
 <robot name="end_effector_gripped_object" xmlns:xacro="http://wiki.ros.org/xacro">
   <joint name="gripped_object_joint" type="fixed">
-    <xacro:transformed_origin name="ee_to_tray_transform" />
+    <xacro:transformed_origin name="gripped_object_transform" />
     <parent link="gripper"/>
     <child link="gripped_object"/>
@@ -29,3 +29,18 @@
     </inertial>
   </link>
+  <!-- The visual_balance link/joint is visual-only and just provides a visual reference for an object that stays in place w.r.t. the tray. -->
+  <!-- For debugging purposes only! -->
+  <joint name="visual_balance_joint" type="fixed">
+    <parent link="gripped_object"/>
+    <child link="visual_balance_link"/>
+    <origin rpy="0 0 0" xyz="0 0 0.2"/>
+  </joint>
+  <link name="visual_balance_link">
+    <visual>
+      <geometry>
+        <box size="0.1 0.1 0.1" />
+      </geometry>
+      <material name="black"/>
+    </visual>
+  </link>
 </robot>

Commit message: Add xacro arg to show/hide the extra visual balance link.

File: upright_assets/thing/xacro/end_effectors/gripped_object.urdf.xacro (robot description, xacro)
@@ -1,4 +1,5 @@
 <?xml version="1.0" encoding="utf-8"?>
 <robot name="end_effector_gripped_object" xmlns:xacro="http://wiki.ros.org/xacro">
+  <xacro:arg name="show_balance_link" default="true"/>
   <joint name="gripped_object_joint" type="fixed">
     <xacro:transformed_origin name="gripped_object_transform" />
@@ -30,17 +31,18 @@
   </link>
   <!-- The visual_balance link/joint is visual-only and just provides a visual reference for an object that stays in place w.r.t. the tray. -->
-  <!-- For debugging purposes only! -->
-  <joint name="visual_balance_joint" type="fixed">
-    <parent link="gripped_object"/>
-    <child link="visual_balance_link"/>
-    <origin rpy="0 0 0" xyz="0 0 0.2"/>
-  </joint>
-  <link name="visual_balance_link">
-    <visual>
-      <geometry>
-        <box size="0.1 0.1 0.1" />
-      </geometry>
-      <material name="black"/>
-    </visual>
-  </link>
+  <xacro:if value="$(arg show_balance_link)">
+    <joint name="visual_balance_joint" type="fixed">
+      <parent link="gripped_object"/>
+      <child link="visual_balance_link"/>
+      <origin rpy="0 0 0" xyz="0 0 0.2"/>
+    </joint>
+    <link name="visual_balance_link">
+      <visual>
+        <geometry>
+          <box size="0.1 0.1 0.1" />
+        </geometry>
+        <material name="black"/>
+      </visual>
+    </link>
+  </xacro:if>
 </robot>
